Commit message: L/r launch files and xacro for UR10 and SR hand

File: urdf/srhand_ur10arm.urdf.xacro (robot description, xacro)
@@ -1,3 +1,3 @@
- <robot xmlns:xacro="http://ros.org/wiki/xacro">
+ <robot xmlns:xacro="http://ros.org/wiki/xacro" name="ur10srh">
   <!--<xacro:include filename="$(find ur_description)/urdf/gazebo.urdf.xacro" />-->
   <xacro:include filename="$(find ur_description)/urdf/ur10.urdf.xacro" />
@@ -5,16 +5,16 @@
   <joint name="world_joint" type="fixed">
     <parent link="world" />
-    <child link = "ra_base_link" />
+    <child link = "$(arg prefix)a_base_link" />
     <origin xyz="0.0 0.0 0.0" rpy="0.0 0.0 0.0" />
   </joint>
-  <xacro:ur10_robot prefix="ra_" joint_limited="false"/>
+  <xacro:ur10_robot prefix="$(arg prefix)a_" joint_limited="false"/>
   <xacro:include filename="$(find sr_description)/materials.urdf.xacro" />
   <xacro:include filename="$(find sr_description)/hand/xacro/full_hand.urdf.xacro" />
   <xacro:include filename="$(find sr_description)/other/xacro/gazebo/gazebo.urdf.xacro" />
-  <xacro:shadowhand muscletrans="false" muscle="false" bio="true" ubi="false" eli="false" reflect="1.0" prefix="rh_" />
-  <joint name="right_arm_to_right_hand" type="fixed">
-    <parent link="ra_ee_link" />
-    <child link = "rh_forearm" />
-    <origin xyz="0.012 0.0 0.0" rpy="${pi/2.0} 0.0 ${pi/2.0}" />
-  </joint>
+  <xacro:shadowhand muscletrans="false" muscle="false" bio="true" ubi="false" eli="false" reflect="1.0" prefix="$(arg prefix)h_" />
+    <joint name="arm_to_hand" type="fixed">
+      <parent link="$(arg prefix)a_ee_link" />
+      <child link = "$(arg prefix)h_forearm" />
+      <origin xyz="0.012 0.0 0.0" rpy="${pi/2.0} 0.0 ${pi/2.0}" />
+    </joint>
  </robot>

Commit message: test

File: urdf/srhand_ur10arm.urdf.xacro (robot description, xacro)
@@ -5,15 +5,15 @@
   <joint name="world_joint" type="fixed">
     <parent link="world" />
-    <child link = "$(arg prefix)a_base_link" />
+    <child link = "ra_base_link" />
     <origin xyz="0.0 0.0 0.0" rpy="0.0 0.0 0.0" />
   </joint>
-  <xacro:ur10_robot prefix="$(arg prefix)a_" joint_limited="false"/>
+  <xacro:ur10_robot prefix="ra_" joint_limited="false"/>
   <xacro:include filename="$(find sr_description)/materials.urdf.xacro" />
   <xacro:include filename="$(find sr_description)/hand/xacro/full_hand.urdf.xacro" />
   <xacro:include filename="$(find sr_description)/other/xacro/gazebo/gazebo.urdf.xacro" />
-  <xacro:shadowhand muscletrans="false" muscle="false" bio="true" ubi="false" eli="false" reflect="1.0" prefix="$(arg prefix)h_" />
+  <xacro:shadowhand muscletrans="false" muscle="false" bio="true" ubi="false" eli="false" reflect="1.0" prefix="rh_" />
     <joint name="arm_to_hand" type="fixed">
-      <parent link="$(arg prefix)a_ee_link" />
-      <child link = "$(arg prefix)h_forearm" />
+      <parent link="ra_ee_link" />
+      <child link = "rh_forearm" />
       <origin xyz="0.012 0.0 0.0" rpy="${pi/2.0} 0.0 ${pi/2.0}" />
     </joint>

Commit message: ur10srh moveit config

File: urdf/srhand_ur10arm.urdf.xacro (robot description, xacro)
@@ -12,6 +12,6 @@
   <xacro:include filename="$(find sr_description)/hand/xacro/full_hand.urdf.xacro" />
   <xacro:include filename="$(find sr_description)/other/xacro/gazebo/gazebo.urdf.xacro" />
-  <xacro:shadowhand muscletrans="false" muscle="false" bio="true" ubi="false" eli="false" reflect="1.0" prefix="rh_" />
-    <joint name="arm_to_hand" type="fixed">
+  <xacro:shadowhand muscletrans="false" muscle="false" bio="false" ubi="false" eli="false" reflect="1.0" prefix="rh_" />
+    <joint name="right_arm_to_right_hand" type="fixed">
       <parent link="ra_ee_link" />
       <child link = "rh_forearm" />
