Commit message: Fix pending things after merge

File: urdf/left_srhand_ur10_joint_limited.urdf.xacro (robot description, xacro)
@@ -5,15 +5,15 @@
   <joint name="world_joint" type="fixed">
     <parent link="world" />
-    <child link = "$(arg prefix)a_base_link" />
+    <child link = "la_base_link" />
     <origin xyz="0.0 0.0 0.0" rpy="0.0 0.0 0.0" />
   </joint>
-  <xacro:ur10_robot prefix="$(arg prefix)a_" joint_limited="true"/>
+  <xacro:ur10_robot prefix="la_" joint_limited="true"/>
   <xacro:include filename="$(find sr_description)/materials.urdf.xacro" />
   <xacro:include filename="$(find sr_description)/hand/xacro/full_hand.urdf.xacro" />
   <xacro:include filename="$(find sr_description)/other/xacro/gazebo/gazebo.urdf.xacro" />
-  <xacro:shadowhand muscletrans="false" muscle="false" bio="true" ubi="false" eli="false" reflect="1.0" prefix="$(arg prefix)h_" />
+  <xacro:shadowhand muscletrans="false" muscle="false" bio="false" ubi="false" eli="false" reflect="-1.0" prefix="lh_" />
     <joint name="arm_to_hand" type="fixed">
-      <parent link="$(arg prefix)a_ee_link" />
-      <child link = "$(arg prefix)h_forearm" />
+      <parent link="la_ee_link" />
+      <child link = "lh_forearm" />
       <origin xyz="0.012 0.0 0.0" rpy="${pi/2.0} ${pi} ${pi/2.0}" />
     </joint>
