Commit message: setting the hand face down + adding opened and pack default pose for the hand

File: urdf/for_moveit/srhand_ur10arm.urdf.xacro (robot description, xacro)
@@ -16,5 +16,5 @@
       <parent link="ra_ee_link" />
       <child link = "rh_forearm" />
-      <origin xyz="0.012 0.0 0.0" rpy="${pi/2.0} 0.0 ${pi/2.0}" />
+      <origin xyz="0.012 0.0 0.0" rpy="${pi/2.0} ${pi} ${pi/2.0}" />
     </joint>
  </robot>

File: urdf/srhand_ur10arm.urdf.xacro (robot description, xacro)
@@ -16,5 +16,5 @@
       <parent link="$(arg prefix)a_ee_link" />
       <child link = "$(arg prefix)h_forearm" />
-      <origin xyz="0.012 0.0 0.0" rpy="${pi/2.0} 0.0 ${pi/2.0}" />
+      <origin xyz="0.012 0.0 0.0" rpy="${pi/2.0} ${pi} ${pi/2.0}" />
     </joint>
  </robot>
