Commit message: fixing coding style

File: sr_multi_description/urdf/for_moveit/srhand_ur10arm.urdf.xacro (robot description, xacro)
@@ -1,20 +1,21 @@
- <robot xmlns:xacro="http://ros.org/wiki/xacro" name="ur10srh">
-  <!--<xacro:include filename="$(find ur_description)/urdf/gazebo.urdf.xacro" />-->
-  <xacro:include filename="$(find ur_description)/urdf/ur10.urdf.xacro" />
-  <link name="world" />
-  <joint name="world_joint" type="fixed">
-    <parent link="world" />
-    <child link = "ra_base_link" />
-    <origin xyz="0.0 0.0 0.0" rpy="0.0 0.0 0.0" />
-  </joint>
-  <xacro:ur10_robot prefix="ra_" joint_limited="false"/>
-  <xacro:include filename="$(find sr_description)/materials.urdf.xacro" />
-  <xacro:include filename="$(find sr_description)/hand/xacro/full_hand.urdf.xacro" />
-  <xacro:include filename="$(find sr_description)/other/xacro/gazebo/gazebo.urdf.xacro" />
-  <xacro:shadowhand muscletrans="false" muscle="false" bio="true" bt_sp="false" ubi="false" eli="false" reflect="1.0" prefix="rh_" />
+<robot xmlns:xacro="http://ros.org/wiki/xacro" name="ur10srh">
+    <!--<xacro:include filename="$(find ur_description)/urdf/gazebo.urdf.xacro" />-->
+    <xacro:include filename="$(find ur_description)/urdf/ur10.urdf.xacro"/>
+    <link name="world"/>
+    <joint name="world_joint" type="fixed">
+        <parent link="world"/>
+        <child link="ra_base_link"/>
+        <origin xyz="0.0 0.0 0.0" rpy="0.0 0.0 0.0"/>
+    </joint>
+    <xacro:ur10_robot prefix="ra_" joint_limited="false"/>
+    <xacro:include filename="$(find sr_description)/materials.urdf.xacro"/>
+    <xacro:include filename="$(find sr_description)/hand/xacro/full_hand.urdf.xacro"/>
+    <xacro:include filename="$(find sr_description)/other/xacro/gazebo/gazebo.urdf.xacro"/>
+    <xacro:shadowhand muscletrans="false" muscle="false" bio="true" bt_sp="false" ubi="false" eli="false" reflect="1.0"
+                      prefix="rh_"/>
     <joint name="arm_to_hand" type="fixed">
-      <parent link="ra_ee_link" />
-      <child link = "rh_forearm" />
-      <origin xyz="0.012 0.0 0.0" rpy="${pi/2.0} ${pi} ${pi/2.0}" />
+        <parent link="ra_ee_link"/>
+        <child link="rh_forearm"/>
+        <origin xyz="0.012 0.0 0.0" rpy="${pi/2.0} ${pi} ${pi/2.0}"/>
     </joint>
- </robot>
+</robot>

File: sr_multi_description/urdf/left_srhand_ur10.urdf.xacro (robot description, xacro)
@@ -1,20 +1,21 @@
- <robot xmlns:xacro="http://ros.org/wiki/xacro" name="ur10srh">
-  <!--<xacro:include filename="$(find ur_description)/urdf/gazebo.urdf.xacro" />-->
-  <xacro:include filename="$(find ur_description)/urdf/ur10.urdf.xacro" />
-  <link name="world" />
-  <joint name="world_joint" type="fixed">
-    <parent link="world" />
-    <child link = "la_base_link" />
-    <origin xyz="0.0 0.0 0.0" rpy="0.0 0.0 0.0" />
-  </joint>
-  <xacro:ur10_robot prefix="la_" joint_limited="false"/>
-  <xacro:include filename="$(find sr_description)/materials.urdf.xacro" />
-  <xacro:include filename="$(find sr_description)/hand/xacro/full_hand.urdf.xacro" />
-  <xacro:include filename="$(find sr_description)/other/xacro/gazebo/gazebo.urdf.xacro" />
-  <xacro:shadowhand muscletrans="false" muscle="false" bio="false" bt_sp="false" ubi="false" eli="false" reflect="-1.0" prefix="lh_" />
+<robot xmlns:xacro="http://ros.org/wiki/xacro" name="ur10srh">
+    <!--<xacro:include filename="$(find ur_description)/urdf/gazebo.urdf.xacro" />-->
+    <xacro:include filename="$(find ur_description)/urdf/ur10.urdf.xacro"/>
+    <link name="world"/>
+    <joint name="world_joint" type="fixed">
+        <parent link="world"/>
+        <child link="la_base_link"/>
+        <origin xyz="0.0 0.0 0.0" rpy="0.0 0.0 0.0"/>
+    </joint>
+    <xacro:ur10_robot prefix="la_" joint_limited="false"/>
+    <xacro:include filename="$(find sr_description)/materials.urdf.xacro"/>
+    <xacro:include filename="$(find sr_description)/hand/xacro/full_hand.urdf.xacro"/>
+    <xacro:include filename="$(find sr_description)/other/xacro/gazebo/gazebo.urdf.xacro"/>
+    <xacro:shadowhand muscletrans="false" muscle="false" bio="false" bt_sp="false" ubi="false" eli="false"
+                      reflect="-1.0" prefix="lh_"/>
     <joint name="arm_to_hand" type="fixed">
-      <parent link="la_ee_link" />
-      <child link = "lh_forearm" />
-      <origin xyz="0.012 0.0 0.0" rpy="${pi/2.0} ${pi} ${pi/2.0}" />
+        <parent link="la_ee_link"/>
+        <child link="lh_forearm"/>
+        <origin xyz="0.012 0.0 0.0" rpy="${pi/2.0} ${pi} ${pi/2.0}"/>
     </joint>
- </robot>
+</robot>

File: sr_multi_description/urdf/left_srhand_ur10_joint_limited.urdf.xacro (robot description, xacro)
@@ -1,20 +1,21 @@
- <robot xmlns:xacro="http://ros.org/wiki/xacro" name="ur10srh">
-  <!--<xacro:include filename="$(find ur_description)/urdf/gazebo.urdf.xacro" />-->
-  <xacro:include filename="$(find ur_description)/urdf/ur10.urdf.xacro" />
-  <link name="world" />
-  <joint name="world_joint" type="fixed">
-    <parent link="world" />
-    <child link = "la_base_link" />
-    <origin xyz="0.0 0.0 0.0" rpy="0.0 0.0 0.0" />
-  </joint>
-  <xacro:ur10_robot prefix="la_" joint_limited="true"/>
-  <xacro:include filename="$(find sr_description)/materials.urdf.xacro" />
-  <xacro:include filename="$(find sr_description)/hand/xacro/full_hand.urdf.xacro" />
-  <xacro:include filename="$(find sr_description)/other/xacro/gazebo/gazebo.urdf.xacro" />
-  <xacro:shadowhand muscletrans="false" muscle="false" bio="false" bt_sp="false" ubi="false" eli="false" reflect="-1.0" prefix="lh_" />
+<robot xmlns:xacro="http://ros.org/wiki/xacro" name="ur10srh">
+    <!--<xacro:include filename="$(find ur_description)/urdf/gazebo.urdf.xacro" />-->
+    <xacro:include filename="$(find ur_description)/urdf/ur10.urdf.xacro"/>
+    <link name="world"/>
+    <joint name="world_joint" type="fixed">
+        <parent link="world"/>
+        <child link="la_base_link"/>
+        <origin xyz="0.0 0.0 0.0" rpy="0.0 0.0 0.0"/>
+    </joint>
+    <xacro:ur10_robot prefix="la_" joint_limited="true"/>
+    <xacro:include filename="$(find sr_description)/materials.urdf.xacro"/>
+    <xacro:include filename="$(find sr_description)/hand/xacro/full_hand.urdf.xacro"/>
+    <xacro:include filename="$(find sr_description)/other/xacro/gazebo/gazebo.urdf.xacro"/>
+    <xacro:shadowhand muscletrans="false" muscle="false" bio="false" bt_sp="false" ubi="false" eli="false"
+                      reflect="-1.0" prefix="lh_"/>
     <joint name="arm_to_hand" type="fixed">
-      <parent link="la_ee_link" />
-      <child link = "lh_forearm" />
-      <origin xyz="0.012 0.0 0.0" rpy="${pi/2.0} ${pi} ${pi/2.0}" />
+        <parent link="la_ee_link"/>
+        <child link="lh_forearm"/>
+        <origin xyz="0.012 0.0 0.0" rpy="${pi/2.0} ${pi} ${pi/2.0}"/>
     </joint>
- </robot>
+</robot>

File: sr_multi_description/urdf/right_srhand_ur10.urdf.xacro (robot description, xacro)
@@ -1,20 +1,21 @@
- <robot xmlns:xacro="http://ros.org/wiki/xacro" name="ur10srh">
-  <!--<xacro:include filename="$(find ur_description)/urdf/gazebo.urdf.xacro" />-->
-  <xacro:include filename="$(find ur_description)/urdf/ur10.urdf.xacro" />
-  <link name="world" />
-  <joint name="world_joint" type="fixed">
-    <parent link="world" />
-    <child link = "ra_base_link" />
-    <origin xyz="0.0 0.0 0.0" rpy="0.0 0.0 0.0" />
-  </joint>
-  <xacro:ur10_robot prefix="ra_" joint_limited="false"/>
-  <xacro:include filename="$(find sr_description)/materials.urdf.xacro" />
-  <xacro:include filename="$(find sr_description)/hand/xacro/full_hand.urdf.xacro" />
-  <xacro:include filename="$(find sr_description)/other/xacro/gazebo/gazebo.urdf.xacro" />
-  <xacro:shadowhand muscletrans="false" muscle="false" bio="false" bt_sp="false" ubi="false" eli="false" reflect="1.0" prefix="rh_" />
+<robot xmlns:xacro="http://ros.org/wiki/xacro" name="ur10srh">
+    <!--<xacro:include filename="$(find ur_description)/urdf/gazebo.urdf.xacro" />-->
+    <xacro:include filename="$(find ur_description)/urdf/ur10.urdf.xacro"/>
+    <link name="world"/>
+    <joint name="world_joint" type="fixed">
+        <parent link="world"/>
+        <child link="ra_base_link"/>
+        <origin xyz="0.0 0.0 0.0" rpy="0.0 0.0 0.0"/>
+    </joint>
+    <xacro:ur10_robot prefix="ra_" joint_limited="false"/>
+    <xacro:include filename="$(find sr_description)/materials.urdf.xacro"/>
+    <xacro:include filename="$(find sr_description)/hand/xacro/full_hand.urdf.xacro"/>
+    <xacro:include filename="$(find sr_description)/other/xacro/gazebo/gazebo.urdf.xacro"/>
+    <xacro:shadowhand muscletrans="false" muscle="false" bio="false" bt_sp="false" ubi="false" eli="false" reflect="1.0"
+                      prefix="rh_"/>
     <joint name="arm_to_hand" type="fixed">
-      <parent link="ra_ee_link" />
-      <child link = "rh_forearm" />
-      <origin xyz="0.012 0.0 0.0" rpy="${pi/2.0} ${pi} ${pi/2.0}" />
+        <parent link="ra_ee_link"/>
+        <child link="rh_forearm"/>
+        <origin xyz="0.012 0.0 0.0" rpy="${pi/2.0} ${pi} ${pi/2.0}"/>
     </joint>
- </robot>
+</robot>

File: sr_multi_description/urdf/right_srhand_ur10_biotacs.urdf.xacro (robot description, xacro)
@@ -1,20 +1,21 @@
- <robot xmlns:xacro="http://ros.org/wiki/xacro" name="ur10srh">
-  <!--<xacro:include filename="$(find ur_description)/urdf/gazebo.urdf.xacro" />-->
-  <xacro:include filename="$(find ur_description)/urdf/ur10.urdf.xacro" />
-  <link name="world" />
-  <joint name="world_joint" type="fixed">
-    <parent link="world" />
-    <child link = "ra_base_link" />
-    <origin xyz="0.0 0.0 0.0" rpy="0.0 0.0 0.0" />
-  </joint>
-  <xacro:ur10_robot prefix="ra_" joint_limited="false"/>
-  <xacro:include filename="$(find sr_description)/materials.urdf.xacro" />
-  <xacro:include filename="$(find sr_description)/hand/xacro/full_hand.urdf.xacro" />
-  <xacro:include filename="$(find sr_description)/other/xacro/gazebo/gazebo.urdf.xacro" />
-  <xacro:shadowhand muscletrans="false" muscle="false" bio="true" bt_sp="false" ubi="false" eli="false" reflect="1.0" prefix="rh_" />
+<robot xmlns:xacro="http://ros.org/wiki/xacro" name="ur10srh">
+    <!--<xacro:include filename="$(find ur_description)/urdf/gazebo.urdf.xacro" />-->
+    <xacro:include filename="$(find ur_description)/urdf/ur10.urdf.xacro"/>
+    <link name="world"/>
+    <joint name="world_joint" type="fixed">
+        <parent link="world"/>
+        <child link="ra_base_link"/>
+        <origin xyz="0.0 0.0 0.0" rpy="0.0 0.0 0.0"/>
+    </joint>
+    <xacro:ur10_robot prefix="ra_" joint_limited="false"/>
+    <xacro:include filename="$(find sr_description)/materials.urdf.xacro"/>
+    <xacro:include filename="$(find sr_description)/hand/xacro/full_hand.urdf.xacro"/>
+    <xacro:include filename="$(find sr_description)/other/xacro/gazebo/gazebo.urdf.xacro"/>
+    <xacro:shadowhand muscletrans="false" muscle="false" bio="true" bt_sp="false" ubi="false" eli="false" reflect="1.0"
+                      prefix="rh_"/>
     <joint name="arm_to_hand" type="fixed">
-      <parent link="ra_ee_link" />
-      <child link = "rh_forearm" />
-      <origin xyz="0.012 0.0 0.0" rpy="${pi/2.0} ${pi} ${pi/2.0}" />
+        <parent link="ra_ee_link"/>
+        <child link="rh_forearm"/>
+        <origin xyz="0.012 0.0 0.0" rpy="${pi/2.0} ${pi} ${pi/2.0}"/>
     </joint>
- </robot>
+</robot>

File: sr_multi_description/urdf/right_srhand_ur10_joint_limited.urdf.xacro (robot description, xacro)
@@ -1,20 +1,21 @@
- <robot xmlns:xacro="http://ros.org/wiki/xacro" name="ur10srh">
-  <!--<xacro:include filename="$(find ur_description)/urdf/gazebo.urdf.xacro" />-->
-  <xacro:include filename="$(find ur_description)/urdf/ur10.urdf.xacro" />
-  <link name="world" />
-  <joint name="world_joint" type="fixed">
-    <parent link="world" />
-    <child link = "ra_base_link" />
-    <origin xyz="0.0 0.0 0.0" rpy="0.0 0.0 0.0" />
-  </joint>
-  <xacro:ur10_robot prefix="ra_" joint_limited="true"/>
-  <xacro:include filename="$(find sr_description)/materials.urdf.xacro" />
-  <xacro:include filename="$(find sr_description)/hand/xacro/full_hand.urdf.xacro" />
-  <xacro:include filename="$(find sr_description)/other/xacro/gazebo/gazebo.urdf.xacro" />
-  <xacro:shadowhand muscletrans="false" muscle="false" bio="false" bt_sp="false" ubi="false" eli="false" reflect="1.0" prefix="rh_" />
+<robot xmlns:xacro="http://ros.org/wiki/xacro" name="ur10srh">
+    <!--<xacro:include filename="$(find ur_description)/urdf/gazebo.urdf.xacro" />-->
+    <xacro:include filename="$(find ur_description)/urdf/ur10.urdf.xacro"/>
+    <link name="world"/>
+    <joint name="world_joint" type="fixed">
+        <parent link="world"/>
+        <child link="ra_base_link"/>
+        <origin xyz="0.0 0.0 0.0" rpy="0.0 0.0 0.0"/>
+    </joint>
+    <xacro:ur10_robot prefix="ra_" joint_limited="true"/>
+    <xacro:include filename="$(find sr_description)/materials.urdf.xacro"/>
+    <xacro:include filename="$(find sr_description)/hand/xacro/full_hand.urdf.xacro"/>
+    <xacro:include filename="$(find sr_description)/other/xacro/gazebo/gazebo.urdf.xacro"/>
+    <xacro:shadowhand muscletrans="false" muscle="false" bio="false" bt_sp="false" ubi="false" eli="false" reflect="1.0"
+                      prefix="rh_"/>
     <joint name="arm_to_hand" type="fixed">
-      <parent link="ra_ee_link" />
-      <child link = "rh_forearm" />
-      <origin xyz="0.012 0.0 0.0" rpy="${pi/2.0} ${pi} ${pi/2.0}" />
+        <parent link="ra_ee_link"/>
+        <child link="rh_forearm"/>
+        <origin xyz="0.012 0.0 0.0" rpy="${pi/2.0} ${pi} ${pi/2.0}"/>
     </joint>
- </robot>
+</robot>

File: sr_multi_description/urdf/right_srhand_ur10_joint_limited_biotacs.urdf.xacro (robot description, xacro)
@@ -1,20 +1,21 @@
- <robot xmlns:xacro="http://ros.org/wiki/xacro" name="ur10srh">
-  <!--<xacro:include filename="$(find ur_description)/urdf/gazebo.urdf.xacro" />-->
-  <xacro:include filename="$(find ur_description)/urdf/ur10.urdf.xacro" />
-  <link name="world" />
-  <joint name="world_joint" type="fixed">
-    <parent link="world" />
-    <child link = "ra_base_link" />
-    <origin xyz="0.0 0.0 0.0" rpy="0.0 0.0 0.0" />
-  </joint>
-  <xacro:ur10_robot prefix="ra_" joint_limited="true"/>
-  <xacro:include filename="$(find sr_description)/materials.urdf.xacro" />
-  <xacro:include filename="$(find sr_description)/hand/xacro/full_hand.urdf.xacro" />
-  <xacro:include filename="$(find sr_description)/other/xacro/gazebo/gazebo.urdf.xacro" />
-  <xacro:shadowhand muscletrans="false" muscle="false" bio="true" bt_sp="false" ubi="false" eli="false" reflect="1.0" prefix="rh_" />
+<robot xmlns:xacro="http://ros.org/wiki/xacro" name="ur10srh">
+    <!--<xacro:include filename="$(find ur_description)/urdf/gazebo.urdf.xacro" />-->
+    <xacro:include filename="$(find ur_description)/urdf/ur10.urdf.xacro"/>
+    <link name="world"/>
+    <joint name="world_joint" type="fixed">
+        <parent link="world"/>
+        <child link="ra_base_link"/>
+        <origin xyz="0.0 0.0 0.0" rpy="0.0 0.0 0.0"/>
+    </joint>
+    <xacro:ur10_robot prefix="ra_" joint_limited="true"/>
+    <xacro:include filename="$(find sr_description)/materials.urdf.xacro"/>
+    <xacro:include filename="$(find sr_description)/hand/xacro/full_hand.urdf.xacro"/>
+    <xacro:include filename="$(find sr_description)/other/xacro/gazebo/gazebo.urdf.xacro"/>
+    <xacro:shadowhand muscletrans="false" muscle="false" bio="true" bt_sp="false" ubi="false" eli="false" reflect="1.0"
+                      prefix="rh_"/>
     <joint name="arm_to_hand" type="fixed">
-      <parent link="ra_ee_link" />
-      <child link = "rh_forearm" />
-      <origin xyz="0.012 0.0 0.0" rpy="${pi/2.0} ${pi} ${pi/2.0}" />
+        <parent link="ra_ee_link"/>
+        <child link="rh_forearm"/>
+        <origin xyz="0.012 0.0 0.0" rpy="${pi/2.0} ${pi} ${pi/2.0}"/>
     </joint>
- </robot>
+</robot>

Commit message: rotate hand on arm in urdf

File: sr_multi_description/urdf/for_moveit/srhand_ur10arm.urdf.xacro (robot description, xacro)
@@ -17,5 +17,5 @@
         <parent link="ra_ee_link"/>
         <child link="rh_forearm"/>
-        <origin xyz="0.012 0.0 0.0" rpy="${pi/2.0} ${pi} ${pi/2.0}"/>
+        <origin xyz="0.012 0.0 0.0" rpy="${pi/2.0} ${0.0} ${pi/2.0}"/>
     </joint>
 </robot>

File: sr_multi_description/urdf/left_srhand_ur10.urdf.xacro (robot description, xacro)
@@ -17,5 +17,5 @@
         <parent link="la_ee_link"/>
         <child link="lh_forearm"/>
-        <origin xyz="0.012 0.0 0.0" rpy="${pi/2.0} ${pi} ${pi/2.0}"/>
+        <origin xyz="0.012 0.0 0.0" rpy="${pi/2.0} ${0.0} ${pi/2.0}"/>
     </joint>
 </robot>

File: sr_multi_description/urdf/left_srhand_ur10_joint_limited.urdf.xacro (robot description, xacro)
@@ -17,5 +17,5 @@
         <parent link="la_ee_link"/>
         <child link="lh_forearm"/>
-        <origin xyz="0.012 0.0 0.0" rpy="${pi/2.0} ${pi} ${pi/2.0}"/>
+        <origin xyz="0.012 0.0 0.0" rpy="${pi/2.0} ${0.0} ${pi/2.0}"/>
     </joint>
 </robot>

File: sr_multi_description/urdf/left_srhand_ur5.urdf.xacro (robot description, xacro)
@@ -17,5 +17,5 @@
         <parent link="la_ee_link"/>
         <child link="lh_forearm"/>
-        <origin xyz="0.012 0.0 0.0" rpy="${pi/2.0} ${pi} ${pi/2.0}"/>
+        <origin xyz="0.012 0.0 0.0" rpy="${pi/2.0} ${0.0} ${pi/2.0}"/>
     </joint>
 </robot>

File: sr_multi_description/urdf/left_srhand_ur5_joint_limited.urdf.xacro (robot description, xacro)
@@ -17,5 +17,5 @@
         <parent link="la_ee_link"/>
         <child link="lh_forearm"/>
-        <origin xyz="0.012 0.0 0.0" rpy="${pi/2.0} ${pi} ${pi/2.0}"/>
+        <origin xyz="0.012 0.0 0.0" rpy="${pi/2.0} ${0.0} ${pi/2.0}"/>
     </joint>
 </robot>

File: sr_multi_description/urdf/right_srhand_extra_lite_ur5_joint_limited.urdf.xacro (robot description, xacro)
@@ -17,5 +17,5 @@
         <parent link="ra_ee_link"/>
         <child link="rh_forearm"/>
-        <origin xyz="0.012 0.0 0.0" rpy="${pi/2.0} ${pi} ${pi/2.0}"/>
+        <origin xyz="0.012 0.0 0.0" rpy="${pi/2.0} ${0.0} ${pi/2.0}"/>
     </joint>
 </robot>

File: sr_multi_description/urdf/right_srhand_lite_ur10_joint_limited.urdf.xacro (robot description, xacro)
@@ -17,5 +17,5 @@
         <parent link="ra_ee_link"/>
         <child link="rh_forearm"/>
-        <origin xyz="0.012 0.0 0.0" rpy="${pi/2.0} ${pi} ${pi/2.0}"/>
+        <origin xyz="0.012 0.0 0.0" rpy="${pi/2.0} ${0.0} ${pi/2.0}"/>
     </joint>
 </robot>

File: sr_multi_description/urdf/right_srhand_lite_ur5.urdf.xacro (robot description, xacro)
@@ -17,5 +17,5 @@
         <parent link="ra_ee_link"/>
         <child link="rh_forearm"/>
-        <origin xyz="0.012 0.0 0.0" rpy="${pi/2.0} ${pi} ${pi/2.0}"/>
+        <origin xyz="0.012 0.0 0.0" rpy="${pi/2.0} ${0.0} ${pi/2.0}"/>
     </joint>
 </robot>

File: sr_multi_description/urdf/right_srhand_lite_ur5_joint_limited.urdf.xacro (robot description, xacro)
@@ -17,5 +17,5 @@
         <parent link="ra_ee_link"/>
         <child link="rh_forearm"/>
-        <origin xyz="0.012 0.0 0.0" rpy="${pi/2.0} ${pi} ${pi/2.0}"/>
+        <origin xyz="0.012 0.0 0.0" rpy="${pi/2.0} ${0.0} ${pi/2.0}"/>
     </joint>
 </robot>

File: sr_multi_description/urdf/right_srhand_ur10.urdf.xacro (robot description, xacro)
@@ -17,5 +17,5 @@
         <parent link="ra_ee_link"/>
         <child link="rh_forearm"/>
-        <origin xyz="0.012 0.0 0.0" rpy="${pi/2.0} ${pi} ${pi/2.0}"/>
+        <origin xyz="0.012 0.0 0.0" rpy="${pi/2.0} ${0.0} ${pi/2.0}"/>
     </joint>
 </robot>

File: sr_multi_description/urdf/right_srhand_ur10_biotacs.urdf.xacro (robot description, xacro)
@@ -17,5 +17,5 @@
         <parent link="ra_ee_link"/>
         <child link="rh_forearm"/>
-        <origin xyz="0.012 0.0 0.0" rpy="${pi/2.0} ${pi} ${pi/2.0}"/>
+        <origin xyz="0.012 0.0 0.0" rpy="${pi/2.0} ${0.0} ${pi/2.0}"/>
     </joint>
 </robot>

File: sr_multi_description/urdf/right_srhand_ur10_bt_sp_biotacs.urdf.xacro (robot description, xacro)
@@ -17,5 +17,5 @@
         <parent link="ra_ee_link"/>
         <child link="rh_forearm"/>
-        <origin xyz="0.012 0.0 0.0" rpy="${pi/2.0} ${pi} ${pi/2.0}"/>
+        <origin xyz="0.012 0.0 0.0" rpy="${pi/2.0} ${0.0} ${pi/2.0}"/>
     </joint>
 </robot>

File: sr_multi_description/urdf/right_srhand_ur10_joint_limited.urdf.xacro (robot description, xacro)
@@ -17,5 +17,5 @@
         <parent link="ra_ee_link"/>
         <child link="rh_forearm"/>
-        <origin xyz="0.012 0.0 0.0" rpy="${pi/2.0} ${pi} ${pi/2.0}"/>
+        <origin xyz="0.012 0.0 0.0" rpy="${pi/2} ${0.0} ${pi/2}"/>
     </joint>
 </robot>

File: sr_multi_description/urdf/right_srhand_ur10_joint_limited_biotacs.urdf.xacro (robot description, xacro)
@@ -17,5 +17,5 @@
         <parent link="ra_ee_link"/>
         <child link="rh_forearm"/>
-        <origin xyz="0.012 0.0 0.0" rpy="${pi/2.0} ${pi} ${pi/2.0}"/>
+        <origin xyz="0.012 0.0 0.0" rpy="${pi/2.0} ${0.0} ${pi/2.0}"/>
     </joint>
 </robot>

File: sr_multi_description/urdf/right_srhand_ur5.urdf.xacro (robot description, xacro)
@@ -17,5 +17,5 @@
         <parent link="ra_ee_link"/>
         <child link="rh_forearm"/>
-        <origin xyz="0.012 0.0 0.0" rpy="${pi/2.0} ${pi} ${pi/2.0}"/>
+        <origin xyz="0.012 0.0 0.0" rpy="${pi/2.0} ${0.0} ${pi/2.0}"/>
     </joint>
 </robot>

File: sr_multi_description/urdf/right_srhand_ur5_joint_limited.urdf.xacro (robot description, xacro)
@@ -17,5 +17,5 @@
         <parent link="ra_ee_link"/>
         <child link="rh_forearm"/>
-        <origin xyz="0.012 0.0 0.0" rpy="${pi/2.0} ${pi} ${pi/2.0}"/>
+        <origin xyz="0.012 0.0 0.0" rpy="${pi/2.0} ${0.0} ${pi/2.0}"/>
     </joint>
 </robot>
