Commit message: proposed changed to add initial position to xacro

File: sr_multi_description/urdf/right_srhand_ur10_joint_limited.urdf.xacro (robot description, xacro)
@@ -6,5 +6,10 @@
         <parent link="world"/>
         <child link="ra_base_link"/>
-        <origin xyz="0.0 0.0 0.0" rpy="0.0 0.0 0.0"/>
+        <xacro:if value="$(arg initial_z)">
+        	<origin xyz="0.0 0.0 $(arg initial_z)" rpy="0.0 0.0 0.0"/>
+		</xacro:if>
+        <xacro:if value="$(arg initial_z)">
+        	<origin xyz="0.0 0.0 0.0" rpy="0.0 0.0 0.0"/>
+		</xacro:if>
     </joint>
     <xacro:ur10_robot prefix="ra_" joint_limited="true"/>

Commit message: fixed urdf

File: sr_multi_description/urdf/right_srhand_ur10_joint_limited.urdf.xacro (robot description, xacro)
@@ -3,13 +3,14 @@
     <xacro:include filename="$(find ur_description)/urdf/ur10.urdf.xacro"/>
     <link name="world"/>
+    <xacro:arg name="initial_z" default="0.0"/>
     <joint name="world_joint" type="fixed">
         <parent link="world"/>
         <child link="ra_base_link"/>
         <xacro:if value="$(arg initial_z)">
-        	<origin xyz="0.0 0.0 $(arg initial_z)" rpy="0.0 0.0 0.0"/>
-		</xacro:if>
-        <xacro:if value="$(arg initial_z)">
-        	<origin xyz="0.0 0.0 0.0" rpy="0.0 0.0 0.0"/>
-		</xacro:if>
+            <origin xyz="0.0 0.0 $(arg initial_z)" rpy="0.0 0.0 0.0"/>
+        </xacro:if>
+        <xacro:unless value="$(arg initial_z)">
+            <origin xyz="0.0 0.0 0.0" rpy="0.0 0.0 0.0"/>
+        </xacro:unless>
     </joint>
     <xacro:ur10_robot prefix="ra_" joint_limited="true"/>
