Commit message: Fixed xacro condition

File: sr_multi_description/urdf/right_srhand_ur10.urdf.xacro (robot description, xacro)
@@ -7,10 +7,5 @@
         <parent link="world"/>
         <child link="ra_base_link"/>
-        <xacro:if value="$(arg initial_z)">
-            <origin xyz="0.0 0.0 $(arg initial_z)" rpy="0.0 0.0 0.0"/>
-        </xacro:if>
-        <xacro:unless value="$(arg initial_z)">
-            <origin xyz="0.0 0.0 0.0" rpy="0.0 0.0 0.0"/>
-        </xacro:unless>
+        <origin xyz="0.0 0.0 $(arg initial_z)" rpy="0.0 0.0 0.0"/>
     </joint>
     <xacro:ur10_robot prefix="ra_" joint_limited="false"/>

File: sr_multi_description/urdf/right_srhand_ur10_joint_limited.urdf.xacro (robot description, xacro)
@@ -7,10 +7,5 @@
         <parent link="world"/>
         <child link="ra_base_link"/>
-        <xacro:if value="$(arg initial_z)">
-            <origin xyz="0.0 0.0 $(arg initial_z)" rpy="0.0 0.0 0.0"/>
-        </xacro:if>
-        <xacro:unless value="$(arg initial_z)">
-            <origin xyz="0.0 0.0 0.0" rpy="0.0 0.0 0.0"/>
-        </xacro:unless>
+        <origin xyz="0.0 0.0 $(arg initial_z)" rpy="0.0 0.0 0.0"/>
     </joint>
     <xacro:ur10_robot prefix="ra_" joint_limited="true"/>
