Commit message: Refactoring initial_z

File: sr_multi_description/urdf/left_srhand_ur10_joint_limited.urdf.xacro (robot description, xacro)
@@ -7,9 +7,5 @@
         <parent link="world"/>
         <child link="la_base_link"/>
-        <xacro:if value="$(arg initial_z)">
-            <origin xyz="0.0 0.0 $(arg initial_z)" rpy="0.0 0.0 0.0"/>
-        </xacro:if>
-        <xacro:unless value="$(arg initial_z)">
-            <origin xyz="0.0 0.0 0.0" rpy="0.0 0.0 0.0"/>
+        <origin xyz="0.0 0.0 $(arg initial_z)" rpy="0.0 0.0 0.0"/>
         </xacro:unless>
     </joint>

File: sr_multi_moveit/sr_box_ur10_moveit_config/config/ur10_with_box.urdf.xacro (robot description, xacro)
@@ -14,10 +14,5 @@
       <parent link="world"/>
       <child link="ra_base_link"/>
-      <xacro:if value="$(arg initial_z)">
-          <origin xyz="0.0 0.0 $(arg initial_z)" rpy="0.0 0.0 0.0"/>
-      </xacro:if>
-      <xacro:unless value="$(arg initial_z)">
-          <origin xyz="0.0 0.0 0.0" rpy="0.0 0.0 0.0"/>
-      </xacro:unless>
+      <origin xyz="0.0 0.0 $(arg initial_z)" rpy="0.0 0.0 0.0"/>
   </joint>
   <!-- Box representation of hand -->
