Commit message: rotating 180 degrees the wrist

File: sr_multi_description/urdf/right_srhand_ur10_bt_sp_biotacs.urdf.xacro (robot description, xacro)
@@ -18,5 +18,5 @@
         <parent link="ra_ee_link"/>
         <child link="rh_forearm"/>
-        <origin xyz="0.012 0.0 0.0" rpy="${pi/2.0} ${0.0} ${pi/2.0}"/>
+        <origin xyz="0.012 0.0 0.0" rpy="${pi/2.0} ${-pi} ${pi/2.0}"/>
     </joint>
 </robot>
