Commit message: roating wrist on all xacros

File: sr_multi_description/urdf/both_srhand_two_ur10_two_hands.urdf.xacro (robot description, xacro)
@@ -24,5 +24,5 @@
         <parent link="ra_ee_link"/>
         <child link="rh_forearm"/>
-        <origin xyz="0.012 0.0 0.0" rpy="${pi/2.0} ${0.0} ${pi/2.0}"/>
+        <origin xyz="0.012 0.0 0.0" rpy="${pi/2.0} ${-pi} ${pi/2.0}"/>
     </joint>
     <xacro:shadowhand muscletrans="false" muscle="false" bio="false" bt_sp="false" ubi="false" eli="false" reflect="1.0" prefix="lh_" lf="true" cable_mesh="true"/>
@@ -30,5 +30,5 @@
         <parent link="la_ee_link"/>
         <child link="lh_forearm"/>
-        <origin xyz="0.012 0.0 0.0" rpy="${pi/2.0} ${0.0} ${pi/2.0}"/>
+        <origin xyz="0.012 0.0 0.0" rpy="${pi/2.0} ${-pi} ${pi/2.0}"/>
     </joint>
 </robot>

File: sr_multi_description/urdf/left_srhand_ur10.urdf.xacro (robot description, xacro)
@@ -18,5 +18,5 @@
         <parent link="la_ee_link"/>
         <child link="lh_forearm"/>
-        <origin xyz="0.012 0.0 0.0" rpy="${pi/2.0} ${0.0} ${pi/2.0}"/>
+        <origin xyz="0.012 0.0 0.0" rpy="${pi/2.0} ${-pi} ${pi/2.0}"/>
     </joint>
 </robot>

File: sr_multi_description/urdf/left_srhand_ur10_joint_limited.urdf.xacro (robot description, xacro)
@@ -19,5 +19,5 @@
         <parent link="la_ee_link"/>
         <child link="lh_forearm"/>
-        <origin xyz="0.012 0.0 0.0" rpy="${pi/2.0} ${0.0} ${pi/2.0}"/>
+        <origin xyz="0.012 0.0 0.0" rpy="${pi/2.0} ${-pi} ${pi/2.0}"/>
     </joint>
 </robot>

File: sr_multi_description/urdf/left_srhand_ur5.urdf.xacro (robot description, xacro)
@@ -18,5 +18,5 @@
         <parent link="la_ee_link"/>
         <child link="lh_forearm"/>
-        <origin xyz="0.012 0.0 0.0" rpy="${pi/2.0} ${0.0} ${pi/2.0}"/>
+        <origin xyz="0.012 0.0 0.0" rpy="${pi/2.0} ${-pi} ${pi/2.0}"/>
     </joint>
 </robot>

File: sr_multi_description/urdf/left_srhand_ur5_joint_limited.urdf.xacro (robot description, xacro)
@@ -18,5 +18,5 @@
         <parent link="la_ee_link"/>
         <child link="lh_forearm"/>
-        <origin xyz="0.012 0.0 0.0" rpy="${pi/2.0} ${0.0} ${pi/2.0}"/>
+        <origin xyz="0.012 0.0 0.0" rpy="${pi/2.0} ${-pi} ${pi/2.0}"/>
     </joint>
 </robot>

File: sr_multi_description/urdf/right_srhand_bt_sp_biotacs_two_ur10.urdf.xacro (robot description, xacro)
@@ -25,5 +25,5 @@
         <parent link="ra_ee_link"/>
         <child link="rh_forearm"/>
-        <origin xyz="0.012 0.0 0.0" rpy="${pi/2.0} ${0.0} ${pi/2.0}"/>
+        <origin xyz="0.012 0.0 0.0" rpy="${pi/2.0} ${-pi} ${pi/2.0}"/>
     </joint>
 </robot>

File: sr_multi_description/urdf/right_srhand_extra_lite_ur5_joint_limited.urdf.xacro (robot description, xacro)
@@ -18,5 +18,5 @@
         <parent link="ra_ee_link"/>
         <child link="rh_forearm"/>
-        <origin xyz="0.012 0.0 0.0" rpy="${pi/2.0} ${0.0} ${pi/2.0}"/>
+        <origin xyz="0.012 0.0 0.0" rpy="${pi/2.0} ${-pi} ${pi/2.0}"/>
     </joint>
 </robot>

File: sr_multi_description/urdf/right_srhand_lite_ur10_joint_limited.urdf.xacro (robot description, xacro)
@@ -18,5 +18,5 @@
         <parent link="ra_ee_link"/>
         <child link="rh_forearm"/>
-        <origin xyz="0.012 0.0 0.0" rpy="${pi/2.0} ${0.0} ${pi/2.0}"/>
+        <origin xyz="0.012 0.0 0.0" rpy="${pi/2.0} ${-pi} ${pi/2.0}"/>
     </joint>
 </robot>

File: sr_multi_description/urdf/right_srhand_lite_ur5.urdf.xacro (robot description, xacro)
@@ -18,5 +18,5 @@
         <parent link="ra_ee_link"/>
         <child link="rh_forearm"/>
-        <origin xyz="0.012 0.0 0.0" rpy="${pi/2.0} ${0.0} ${pi/2.0}"/>
+        <origin xyz="0.012 0.0 0.0" rpy="${pi/2.0} ${-pi} ${pi/2.0}"/>
     </joint>
 </robot>

File: sr_multi_description/urdf/right_srhand_lite_ur5_joint_limited.urdf.xacro (robot description, xacro)
@@ -18,5 +18,5 @@
         <parent link="ra_ee_link"/>
         <child link="rh_forearm"/>
-        <origin xyz="0.012 0.0 0.0" rpy="${pi/2.0} ${0.0} ${pi/2.0}"/>
+        <origin xyz="0.012 0.0 0.0" rpy="${pi/2.0} ${-pi} ${pi/2.0}"/>
     </joint>
 </robot>

File: sr_multi_description/urdf/right_srhand_stand_ur10.urdf.xacro (robot description, xacro)
@@ -23,5 +23,5 @@
         <parent link="ra_ee_link"/>
         <child link="rh_forearm"/>
-        <origin xyz="0.012 0.0 0.0" rpy="${pi/2.0} ${0.0} ${pi/2.0}"/>
+        <origin xyz="0.012 0.0 0.0" rpy="${pi/2.0} ${-pi} ${pi/2.0}"/>
     </joint>
 </robot>

File: sr_multi_description/urdf/right_srhand_stand_ur10_bt_sp_biotacs.urdf.xacro (robot description, xacro)
@@ -23,5 +23,5 @@
         <parent link="ra_ee_link"/>
         <child link="rh_forearm"/>
-        <origin xyz="0.012 0.0 0.0" rpy="${pi/2.0} ${0.0} ${pi/2.0}"/>
+        <origin xyz="0.012 0.0 0.0" rpy="${pi/2.0} ${-pi} ${pi/2.0}"/>
     </joint>
 </robot>

File: sr_multi_description/urdf/right_srhand_two_ur10.urdf.xacro (robot description, xacro)
@@ -25,5 +25,5 @@
         <parent link="ra_ee_link"/>
         <child link="rh_forearm"/>
-        <origin xyz="0.012 0.0 0.0" rpy="${pi/2.0} ${0.0} ${pi/2.0}"/>
+        <origin xyz="0.012 0.0 0.0" rpy="${pi/2.0} ${-pi} ${pi/2.0}"/>
     </joint>
 </robot>

File: sr_multi_description/urdf/right_srhand_ur10.urdf.xacro (robot description, xacro)
@@ -18,5 +18,5 @@
         <parent link="ra_ee_link"/>
         <child link="rh_forearm"/>
-        <origin xyz="0.012 0.0 0.0" rpy="${pi/2.0} ${0.0} ${pi/2.0}"/>
+        <origin xyz="0.012 0.0 0.0" rpy="${pi/2.0} ${-pi} ${pi/2.0}"/>
     </joint>
 </robot>

File: sr_multi_description/urdf/right_srhand_ur10_biotacs.urdf.xacro (robot description, xacro)
@@ -18,5 +18,5 @@
         <parent link="ra_ee_link"/>
         <child link="rh_forearm"/>
-        <origin xyz="0.012 0.0 0.0" rpy="${pi/2.0} ${0.0} ${pi/2.0}"/>
+        <origin xyz="0.012 0.0 0.0" rpy="${pi/2.0} ${-pi} ${pi/2.0}"/>
     </joint>
 </robot>

File: sr_multi_description/urdf/right_srhand_ur10_joint_limited.urdf.xacro (robot description, xacro)
@@ -18,5 +18,5 @@
         <parent link="ra_ee_link"/>
         <child link="rh_forearm"/>
-        <origin xyz="0.012 0.0 0.0" rpy="${pi/2} ${0.0} ${pi/2}"/>
+        <origin xyz="0.012 0.0 0.0" rpy="${pi/2} ${-pi} ${pi/2}"/>
     </joint>
 </robot>

File: sr_multi_description/urdf/right_srhand_ur10_joint_limited_biotacs.urdf.xacro (robot description, xacro)
@@ -18,5 +18,5 @@
         <parent link="ra_ee_link"/>
         <child link="rh_forearm"/>
-        <origin xyz="0.012 0.0 0.0" rpy="${pi/2.0} ${0.0} ${pi/2.0}"/>
+        <origin xyz="0.012 0.0 0.0" rpy="${pi/2.0} ${-pi} ${pi/2.0}"/>
     </joint>
 </robot>

File: sr_multi_description/urdf/right_srhand_ur10_plus_biotacs.urdf.xacro (robot description, xacro)
@@ -18,5 +18,5 @@
         <parent link="ra_ee_link"/>
         <child link="rh_forearm"/>
-        <origin xyz="0.012 0.0 0.0" rpy="${pi/2.0} ${0.0} ${pi/2.0}"/>
+        <origin xyz="0.012 0.0 0.0" rpy="${pi/2.0} ${-pi} ${pi/2.0}"/>
     </joint>
 </robot>

File: sr_multi_description/urdf/right_srhand_ur5.urdf.xacro (robot description, xacro)
@@ -18,5 +18,5 @@
         <parent link="ra_ee_link"/>
         <child link="rh_forearm"/>
-        <origin xyz="0.012 0.0 0.0" rpy="${pi/2.0} ${0.0} ${pi/2.0}"/>
+        <origin xyz="0.012 0.0 0.0" rpy="${pi/2.0} ${-pi} ${pi/2.0}"/>
     </joint>
 </robot>

File: sr_multi_description/urdf/right_srhand_ur5_joint_limited.urdf.xacro (robot description, xacro)
@@ -18,5 +18,5 @@
         <parent link="ra_ee_link"/>
         <child link="rh_forearm"/>
-        <origin xyz="0.012 0.0 0.0" rpy="${pi/2.0} ${0.0} ${pi/2.0}"/>
+        <origin xyz="0.012 0.0 0.0" rpy="${pi/2.0} ${-pi} ${pi/2.0}"/>
     </joint>
 </robot>
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