Commit message: Changed name of joint arm and hand

File: sr_multi_description/urdf/left_srhand_ur10.urdf.xacro (robot description, xacro)
@@ -14,5 +14,5 @@
     <xacro:shadowhand muscletrans="false" muscle="false" bio="false" bt_sp="false" ubi="false" eli="false"
                       reflect="-1.0" prefix="lh_"/>
-    <joint name="arm_to_hand" type="fixed">
+    <joint name="la_arm_to_hand" type="fixed">
         <parent link="la_ee_link"/>
         <child link="lh_forearm"/>

File: sr_multi_description/urdf/left_srhand_ur10_joint_limited.urdf.xacro (robot description, xacro)
@@ -14,5 +14,5 @@
     <xacro:shadowhand muscletrans="false" muscle="false" bio="false" bt_sp="false" ubi="false" eli="false"
                       reflect="-1.0" prefix="lh_"/>
-    <joint name="arm_to_hand" type="fixed">
+    <joint name="la_arm_to_hand" type="fixed">
         <parent link="la_ee_link"/>
         <child link="lh_forearm"/>

File: sr_multi_description/urdf/right_srhand_ur10.urdf.xacro (robot description, xacro)
@@ -14,5 +14,5 @@
     <xacro:shadowhand muscletrans="false" muscle="false" bio="false" bt_sp="false" ubi="false" eli="false" reflect="1.0"
                       prefix="rh_"/>
-    <joint name="arm_to_hand" type="fixed">
+    <joint name="ra_arm_to_hand" type="fixed">
         <parent link="ra_ee_link"/>
         <child link="rh_forearm"/>

File: sr_multi_description/urdf/right_srhand_ur10_biotacs.urdf.xacro (robot description, xacro)
@@ -14,5 +14,5 @@
     <xacro:shadowhand muscletrans="false" muscle="false" bio="true" bt_sp="false" ubi="false" eli="false" reflect="1.0"
                       prefix="rh_"/>
-    <joint name="arm_to_hand" type="fixed">
+    <joint name="ra_arm_to_hand" type="fixed">
         <parent link="ra_ee_link"/>
         <child link="rh_forearm"/>

File: sr_multi_description/urdf/right_srhand_ur10_joint_limited.urdf.xacro (robot description, xacro)
@@ -14,5 +14,5 @@
     <xacro:shadowhand muscletrans="false" muscle="false" bio="false" bt_sp="false" ubi="false" eli="false" reflect="1.0"
                       prefix="rh_"/>
-    <joint name="arm_to_hand" type="fixed">
+    <joint name="ra_arm_to_hand" type="fixed">
         <parent link="ra_ee_link"/>
         <child link="rh_forearm"/>

File: sr_multi_description/urdf/right_srhand_ur10_joint_limited_biotacs.urdf.xacro (robot description, xacro)
@@ -14,5 +14,5 @@
     <xacro:shadowhand muscletrans="false" muscle="false" bio="true" bt_sp="false" ubi="false" eli="false" reflect="1.0"
                       prefix="rh_"/>
-    <joint name="arm_to_hand" type="fixed">
+    <joint name="ra_arm_to_hand" type="fixed">
         <parent link="ra_ee_link"/>
         <child link="rh_forearm"/>

Commit message: Changed the rest of urdfs

File: sr_multi_description/urdf/left_srhand_ur10.urdf.xacro (robot description, xacro)
@@ -3,8 +3,14 @@
     <xacro:include filename="$(find ur_description)/urdf/ur10.urdf.xacro"/>
     <link name="world"/>
+    <xacro:arg name="initial_z" default="0.0"/>
     <joint name="world_joint" type="fixed">
         <parent link="world"/>
-        <child link="la_base_link"/>
-        <origin xyz="0.0 0.0 0.0" rpy="0.0 0.0 0.0"/>
+        <child link="ra_base_link"/>
+        <xacro:if value="$(arg initial_z)">
+            <origin xyz="0.0 0.0 $(arg initial_z)" rpy="0.0 0.0 0.0"/>
+        </xacro:if>
+        <xacro:unless value="$(arg initial_z)">
+            <origin xyz="0.0 0.0 0.0" rpy="0.0 0.0 0.0"/>
+        </xacro:unless>
     </joint>
     <xacro:ur10_robot prefix="la_" joint_limited="false"/>

File: sr_multi_description/urdf/left_srhand_ur10_joint_limited.urdf.xacro (robot description, xacro)
@@ -3,8 +3,14 @@
     <xacro:include filename="$(find ur_description)/urdf/ur10.urdf.xacro"/>
     <link name="world"/>
+    <xacro:arg name="initial_z" default="0.0"/>
     <joint name="world_joint" type="fixed">
         <parent link="world"/>
-        <child link="la_base_link"/>
-        <origin xyz="0.0 0.0 0.0" rpy="0.0 0.0 0.0"/>
+        <child link="ra_base_link"/>
+        <xacro:if value="$(arg initial_z)">
+            <origin xyz="0.0 0.0 $(arg initial_z)" rpy="0.0 0.0 0.0"/>
+        </xacro:if>
+        <xacro:unless value="$(arg initial_z)">
+            <origin xyz="0.0 0.0 0.0" rpy="0.0 0.0 0.0"/>
+        </xacro:unless>
     </joint>
     <xacro:ur10_robot prefix="la_" joint_limited="true"/>

File: sr_multi_description/urdf/left_srhand_ur5.urdf.xacro (robot description, xacro)
@@ -3,8 +3,14 @@
     <xacro:include filename="$(find ur_description)/urdf/ur5.urdf.xacro"/>
     <link name="world"/>
+    <xacro:arg name="initial_z" default="0.0"/>
     <joint name="world_joint" type="fixed">
         <parent link="world"/>
-        <child link="la_base_link"/>
-        <origin xyz="0.0 0.0 0.0" rpy="0.0 0.0 0.0"/>
+        <child link="ra_base_link"/>
+        <xacro:if value="$(arg initial_z)">
+            <origin xyz="0.0 0.0 $(arg initial_z)" rpy="0.0 0.0 0.0"/>
+        </xacro:if>
+        <xacro:unless value="$(arg initial_z)">
+            <origin xyz="0.0 0.0 0.0" rpy="0.0 0.0 0.0"/>
+        </xacro:unless>
     </joint>
     <xacro:ur5_robot prefix="la_" joint_limited="false"/>

File: sr_multi_description/urdf/left_srhand_ur5_joint_limited.urdf.xacro (robot description, xacro)
@@ -3,8 +3,14 @@
     <xacro:include filename="$(find ur_description)/urdf/ur5.urdf.xacro"/>
     <link name="world"/>
+    <xacro:arg name="initial_z" default="0.0"/>
     <joint name="world_joint" type="fixed">
         <parent link="world"/>
-        <child link="la_base_link"/>
-        <origin xyz="0.0 0.0 0.0" rpy="0.0 0.0 0.0"/>
+        <child link="ra_base_link"/>
+        <xacro:if value="$(arg initial_z)">
+            <origin xyz="0.0 0.0 $(arg initial_z)" rpy="0.0 0.0 0.0"/>
+        </xacro:if>
+        <xacro:unless value="$(arg initial_z)">
+            <origin xyz="0.0 0.0 0.0" rpy="0.0 0.0 0.0"/>
+        </xacro:unless>
     </joint>
     <xacro:ur5_robot prefix="la_" joint_limited="true"/>

File: sr_multi_description/urdf/right_srhand_extra_lite_ur5_joint_limited.urdf.xacro (robot description, xacro)
@@ -3,8 +3,14 @@
     <xacro:include filename="$(find ur_description)/urdf/ur5.urdf.xacro"/>
     <link name="world"/>
+    <xacro:arg name="initial_z" default="0.0"/>
     <joint name="world_joint" type="fixed">
         <parent link="world"/>
         <child link="ra_base_link"/>
-        <origin xyz="0.0 0.0 0.0" rpy="0.0 0.0 0.0"/>
+        <xacro:if value="$(arg initial_z)">
+            <origin xyz="0.0 0.0 $(arg initial_z)" rpy="0.0 0.0 0.0"/>
+        </xacro:if>
+        <xacro:unless value="$(arg initial_z)">
+            <origin xyz="0.0 0.0 0.0" rpy="0.0 0.0 0.0"/>
+        </xacro:unless>
     </joint>
     <xacro:ur5_robot prefix="ra_" joint_limited="true"/>

File: sr_multi_description/urdf/right_srhand_lite_ur10_joint_limited.urdf.xacro (robot description, xacro)
@@ -3,8 +3,14 @@
     <xacro:include filename="$(find ur_description)/urdf/ur10.urdf.xacro"/>
     <link name="world"/>
+    <xacro:arg name="initial_z" default="0.0"/>
     <joint name="world_joint" type="fixed">
         <parent link="world"/>
         <child link="ra_base_link"/>
-        <origin xyz="0.0 0.0 0.0" rpy="0.0 0.0 0.0"/>
+        <xacro:if value="$(arg initial_z)">
+            <origin xyz="0.0 0.0 $(arg initial_z)" rpy="0.0 0.0 0.0"/>
+        </xacro:if>
+        <xacro:unless value="$(arg initial_z)">
+            <origin xyz="0.0 0.0 0.0" rpy="0.0 0.0 0.0"/>
+        </xacro:unless>
     </joint>
     <xacro:ur10_robot prefix="ra_" joint_limited="true"/>

File: sr_multi_description/urdf/right_srhand_lite_ur5.urdf.xacro (robot description, xacro)
@@ -3,8 +3,14 @@
     <xacro:include filename="$(find ur_description)/urdf/ur5.urdf.xacro"/>
     <link name="world"/>
+    <xacro:arg name="initial_z" default="0.0"/>
     <joint name="world_joint" type="fixed">
         <parent link="world"/>
         <child link="ra_base_link"/>
-        <origin xyz="0.0 0.0 0.0" rpy="0.0 0.0 0.0"/>
+        <xacro:if value="$(arg initial_z)">
+            <origin xyz="0.0 0.0 $(arg initial_z)" rpy="0.0 0.0 0.0"/>
+        </xacro:if>
+        <xacro:unless value="$(arg initial_z)">
+            <origin xyz="0.0 0.0 0.0" rpy="0.0 0.0 0.0"/>
+        </xacro:unless>
     </joint>
     <xacro:ur5_robot prefix="ra_" joint_limited="false"/>

File: sr_multi_description/urdf/right_srhand_lite_ur5_joint_limited.urdf.xacro (robot description, xacro)
@@ -3,8 +3,14 @@
     <xacro:include filename="$(find ur_description)/urdf/ur5.urdf.xacro"/>
     <link name="world"/>
+    <xacro:arg name="initial_z" default="0.0"/>
     <joint name="world_joint" type="fixed">
         <parent link="world"/>
         <child link="ra_base_link"/>
-        <origin xyz="0.0 0.0 0.0" rpy="0.0 0.0 0.0"/>
+        <xacro:if value="$(arg initial_z)">
+            <origin xyz="0.0 0.0 $(arg initial_z)" rpy="0.0 0.0 0.0"/>
+        </xacro:if>
+        <xacro:unless value="$(arg initial_z)">
+            <origin xyz="0.0 0.0 0.0" rpy="0.0 0.0 0.0"/>
+        </xacro:unless>
     </joint>
     <xacro:ur5_robot prefix="ra_" joint_limited="true"/>

File: sr_multi_description/urdf/right_srhand_ur10.urdf.xacro (robot description, xacro)
@@ -3,8 +3,14 @@
     <xacro:include filename="$(find ur_description)/urdf/ur10.urdf.xacro"/>
     <link name="world"/>
+    <xacro:arg name="initial_z" default="0.0"/>
     <joint name="world_joint" type="fixed">
         <parent link="world"/>
         <child link="ra_base_link"/>
-        <origin xyz="0.0 0.0 0.0" rpy="0.0 0.0 0.0"/>
+        <xacro:if value="$(arg initial_z)">
+            <origin xyz="0.0 0.0 $(arg initial_z)" rpy="0.0 0.0 0.0"/>
+        </xacro:if>
+        <xacro:unless value="$(arg initial_z)">
+            <origin xyz="0.0 0.0 0.0" rpy="0.0 0.0 0.0"/>
+        </xacro:unless>
     </joint>
     <xacro:ur10_robot prefix="ra_" joint_limited="false"/>

File: sr_multi_description/urdf/right_srhand_ur10_biotacs.urdf.xacro (robot description, xacro)
@@ -3,8 +3,14 @@
     <xacro:include filename="$(find ur_description)/urdf/ur10.urdf.xacro"/>
     <link name="world"/>
+    <xacro:arg name="initial_z" default="0.0"/>
     <joint name="world_joint" type="fixed">
         <parent link="world"/>
         <child link="ra_base_link"/>
-        <origin xyz="0.0 0.0 0.0" rpy="0.0 0.0 0.0"/>
+        <xacro:if value="$(arg initial_z)">
+            <origin xyz="0.0 0.0 $(arg initial_z)" rpy="0.0 0.0 0.0"/>
+        </xacro:if>
+        <xacro:unless value="$(arg initial_z)">
+            <origin xyz="0.0 0.0 0.0" rpy="0.0 0.0 0.0"/>
+        </xacro:unless>
     </joint>
     <xacro:ur10_robot prefix="ra_" joint_limited="false"/>

File: sr_multi_description/urdf/right_srhand_ur10_bt_sp_biotacs.urdf.xacro (robot description, xacro)
@@ -3,8 +3,14 @@
     <xacro:include filename="$(find ur_description)/urdf/ur10.urdf.xacro"/>
     <link name="world"/>
+    <xacro:arg name="initial_z" default="0.0"/>
     <joint name="world_joint" type="fixed">
         <parent link="world"/>
         <child link="ra_base_link"/>
-        <origin xyz="0.0 0.0 0.0" rpy="0.0 0.0 0.0"/>
+        <xacro:if value="$(arg initial_z)">
+            <origin xyz="0.0 0.0 $(arg initial_z)" rpy="0.0 0.0 0.0"/>
+        </xacro:if>
+        <xacro:unless value="$(arg initial_z)">
+            <origin xyz="0.0 0.0 0.0" rpy="0.0 0.0 0.0"/>
+        </xacro:unless>
     </joint>
     <xacro:ur10_robot prefix="ra_" joint_limited="true"/>

File: sr_multi_description/urdf/right_srhand_ur10_joint_limited_biotacs.urdf.xacro (robot description, xacro)
@@ -3,8 +3,14 @@
     <xacro:include filename="$(find ur_description)/urdf/ur10.urdf.xacro"/>
     <link name="world"/>
+    <xacro:arg name="initial_z" default="0.0"/>
     <joint name="world_joint" type="fixed">
         <parent link="world"/>
         <child link="ra_base_link"/>
-        <origin xyz="0.0 0.0 0.0" rpy="0.0 0.0 0.0"/>
+        <xacro:if value="$(arg initial_z)">
+            <origin xyz="0.0 0.0 $(arg initial_z)" rpy="0.0 0.0 0.0"/>
+        </xacro:if>
+        <xacro:unless value="$(arg initial_z)">
+            <origin xyz="0.0 0.0 0.0" rpy="0.0 0.0 0.0"/>
+        </xacro:unless>
     </joint>
     <xacro:ur10_robot prefix="ra_" joint_limited="true"/>

File: sr_multi_description/urdf/right_srhand_ur5.urdf.xacro (robot description, xacro)
@@ -3,8 +3,14 @@
     <xacro:include filename="$(find ur_description)/urdf/ur5.urdf.xacro"/>
     <link name="world"/>
+    <xacro:arg name="initial_z" default="0.0"/>
     <joint name="world_joint" type="fixed">
         <parent link="world"/>
         <child link="ra_base_link"/>
-        <origin xyz="0.0 0.0 0.0" rpy="0.0 0.0 0.0"/>
+        <xacro:if value="$(arg initial_z)">
+            <origin xyz="0.0 0.0 $(arg initial_z)" rpy="0.0 0.0 0.0"/>
+        </xacro:if>
+        <xacro:unless value="$(arg initial_z)">
+            <origin xyz="0.0 0.0 0.0" rpy="0.0 0.0 0.0"/>
+        </xacro:unless>
     </joint>
     <xacro:ur5_robot prefix="ra_" joint_limited="false"/>

File: sr_multi_description/urdf/right_srhand_ur5_joint_limited.urdf.xacro (robot description, xacro)
@@ -3,8 +3,14 @@
     <xacro:include filename="$(find ur_description)/urdf/ur5.urdf.xacro"/>
     <link name="world"/>
+    <xacro:arg name="initial_z" default="0.0"/>
     <joint name="world_joint" type="fixed">
         <parent link="world"/>
         <child link="ra_base_link"/>
-        <origin xyz="0.0 0.0 0.0" rpy="0.0 0.0 0.0"/>
+        <xacro:if value="$(arg initial_z)">
+            <origin xyz="0.0 0.0 $(arg initial_z)" rpy="0.0 0.0 0.0"/>
+        </xacro:if>
+        <xacro:unless value="$(arg initial_z)">
+            <origin xyz="0.0 0.0 0.0" rpy="0.0 0.0 0.0"/>
+        </xacro:unless>
     </joint>
     <xacro:ur5_robot prefix="ra_" joint_limited="true"/>

Commit message: Fix broken left models

File: sr_multi_description/urdf/left_srhand_ur10.urdf.xacro (robot description, xacro)
@@ -6,5 +6,5 @@
     <joint name="world_joint" type="fixed">
         <parent link="world"/>
-        <child link="ra_base_link"/>
+        <child link="la_base_link"/>
         <xacro:if value="$(arg initial_z)">
             <origin xyz="0.0 0.0 $(arg initial_z)" rpy="0.0 0.0 0.0"/>

File: sr_multi_description/urdf/left_srhand_ur10_joint_limited.urdf.xacro (robot description, xacro)
@@ -6,5 +6,5 @@
     <joint name="world_joint" type="fixed">
         <parent link="world"/>
-        <child link="ra_base_link"/>
+        <child link="la_base_link"/>
         <xacro:if value="$(arg initial_z)">
             <origin xyz="0.0 0.0 $(arg initial_z)" rpy="0.0 0.0 0.0"/>

File: sr_multi_description/urdf/left_srhand_ur5.urdf.xacro (robot description, xacro)
@@ -6,5 +6,5 @@
     <joint name="world_joint" type="fixed">
         <parent link="world"/>
-        <child link="ra_base_link"/>
+        <child link="la_base_link"/>
         <xacro:if value="$(arg initial_z)">
             <origin xyz="0.0 0.0 $(arg initial_z)" rpy="0.0 0.0 0.0"/>

File: sr_multi_description/urdf/left_srhand_ur5_joint_limited.urdf.xacro (robot description, xacro)
@@ -6,5 +6,5 @@
     <joint name="world_joint" type="fixed">
         <parent link="world"/>
-        <child link="ra_base_link"/>
+        <child link="la_base_link"/>
         <xacro:if value="$(arg initial_z)">
             <origin xyz="0.0 0.0 $(arg initial_z)" rpy="0.0 0.0 0.0"/>
