Commit message: Optimized code and removed potential error in xacro.

File: sr_multi_description/urdf/left_srhand_ur10.urdf.xacro (robot description, xacro)
@@ -7,10 +7,5 @@
         <parent link="world"/>
         <child link="la_base_link"/>
-        <xacro:if value="$(arg initial_z)">
-            <origin xyz="0.0 0.0 $(arg initial_z)" rpy="0.0 0.0 0.0"/>
-        </xacro:if>
-        <xacro:unless value="$(arg initial_z)">
-            <origin xyz="0.0 0.0 0.0" rpy="0.0 0.0 0.0"/>
-        </xacro:unless>
+        <origin xyz="0.0 0.0 $(arg initial_z)" rpy="0.0 0.0 0.0"/>
     </joint>
     <xacro:ur10_robot prefix="la_" joint_limited="false"/>

File: sr_multi_description/urdf/left_srhand_ur10_joint_limited.urdf.xacro (robot description, xacro)
@@ -7,10 +7,5 @@
         <parent link="world"/>
         <child link="la_base_link"/>
-        <xacro:if value="$(arg initial_z)">
-            <origin xyz="0.0 0.0 $(arg initial_z)" rpy="0.0 0.0 0.0"/>
-        </xacro:if>
-        <xacro:unless value="$(arg initial_z)">
-            <origin xyz="0.0 0.0 0.0" rpy="0.0 0.0 0.0"/>
-        </xacro:unless>
+        <origin xyz="0.0 0.0 $(arg initial_z)" rpy="0.0 0.0 0.0"/>
     </joint>
     <xacro:ur10_robot prefix="la_" joint_limited="true"/>

File: sr_multi_description/urdf/left_srhand_ur5.urdf.xacro (robot description, xacro)
@@ -7,10 +7,5 @@
         <parent link="world"/>
         <child link="la_base_link"/>
-        <xacro:if value="$(arg initial_z)">
-            <origin xyz="0.0 0.0 $(arg initial_z)" rpy="0.0 0.0 0.0"/>
-        </xacro:if>
-        <xacro:unless value="$(arg initial_z)">
-            <origin xyz="0.0 0.0 0.0" rpy="0.0 0.0 0.0"/>
-        </xacro:unless>
+        <origin xyz="0.0 0.0 $(arg initial_z)" rpy="0.0 0.0 0.0"/>
     </joint>
     <xacro:ur5_robot prefix="la_" joint_limited="false"/>

File: sr_multi_description/urdf/left_srhand_ur5_joint_limited.urdf.xacro (robot description, xacro)
@@ -7,10 +7,5 @@
         <parent link="world"/>
         <child link="la_base_link"/>
-        <xacro:if value="$(arg initial_z)">
-            <origin xyz="0.0 0.0 $(arg initial_z)" rpy="0.0 0.0 0.0"/>
-        </xacro:if>
-        <xacro:unless value="$(arg initial_z)">
-            <origin xyz="0.0 0.0 0.0" rpy="0.0 0.0 0.0"/>
-        </xacro:unless>
+        <origin xyz="0.0 0.0 $(arg initial_z)" rpy="0.0 0.0 0.0"/>
     </joint>
     <xacro:ur5_robot prefix="la_" joint_limited="true"/>

File: sr_multi_description/urdf/right_srhand_extra_lite_ur5_joint_limited.urdf.xacro (robot description, xacro)
@@ -7,10 +7,5 @@
         <parent link="world"/>
         <child link="ra_base_link"/>
-        <xacro:if value="$(arg initial_z)">
-            <origin xyz="0.0 0.0 $(arg initial_z)" rpy="0.0 0.0 0.0"/>
-        </xacro:if>
-        <xacro:unless value="$(arg initial_z)">
-            <origin xyz="0.0 0.0 0.0" rpy="0.0 0.0 0.0"/>
-        </xacro:unless>
+        <origin xyz="0.0 0.0 $(arg initial_z)" rpy="0.0 0.0 0.0"/>
     </joint>
     <xacro:ur5_robot prefix="ra_" joint_limited="true"/>

File: sr_multi_description/urdf/right_srhand_lite_ur10_joint_limited.urdf.xacro (robot description, xacro)
@@ -7,10 +7,5 @@
         <parent link="world"/>
         <child link="ra_base_link"/>
-        <xacro:if value="$(arg initial_z)">
-            <origin xyz="0.0 0.0 $(arg initial_z)" rpy="0.0 0.0 0.0"/>
-        </xacro:if>
-        <xacro:unless value="$(arg initial_z)">
-            <origin xyz="0.0 0.0 0.0" rpy="0.0 0.0 0.0"/>
-        </xacro:unless>
+        <origin xyz="0.0 0.0 $(arg initial_z)" rpy="0.0 0.0 0.0"/>
     </joint>
     <xacro:ur10_robot prefix="ra_" joint_limited="true"/>

File: sr_multi_description/urdf/right_srhand_lite_ur5.urdf.xacro (robot description, xacro)
@@ -7,10 +7,5 @@
         <parent link="world"/>
         <child link="ra_base_link"/>
-        <xacro:if value="$(arg initial_z)">
-            <origin xyz="0.0 0.0 $(arg initial_z)" rpy="0.0 0.0 0.0"/>
-        </xacro:if>
-        <xacro:unless value="$(arg initial_z)">
-            <origin xyz="0.0 0.0 0.0" rpy="0.0 0.0 0.0"/>
-        </xacro:unless>
+        <origin xyz="0.0 0.0 $(arg initial_z)" rpy="0.0 0.0 0.0"/>
     </joint>
     <xacro:ur5_robot prefix="ra_" joint_limited="false"/>

File: sr_multi_description/urdf/right_srhand_lite_ur5_joint_limited.urdf.xacro (robot description, xacro)
@@ -7,10 +7,5 @@
         <parent link="world"/>
         <child link="ra_base_link"/>
-        <xacro:if value="$(arg initial_z)">
-            <origin xyz="0.0 0.0 $(arg initial_z)" rpy="0.0 0.0 0.0"/>
-        </xacro:if>
-        <xacro:unless value="$(arg initial_z)">
-            <origin xyz="0.0 0.0 0.0" rpy="0.0 0.0 0.0"/>
-        </xacro:unless>
+        <origin xyz="0.0 0.0 $(arg initial_z)" rpy="0.0 0.0 0.0"/>
     </joint>
     <xacro:ur5_robot prefix="ra_" joint_limited="true"/>

File: sr_multi_description/urdf/right_srhand_stand_ur10.urdf.xacro (robot description, xacro)
@@ -6,10 +6,5 @@
         <parent link="world"/>
         <child link="stand_link"/>
-        <xacro:if value="$(arg initial_z)">
-            <origin xyz="0.0 0.0 $(arg initial_z)" rpy="0.0 0.0 0.0"/>
-        </xacro:if>
-        <xacro:unless value="$(arg initial_z)">
-            <origin xyz="0.0 0.0 0.0" rpy="0.0 0.0 0.0"/>
-        </xacro:unless>
+        <origin xyz="0.0 0.0 $(arg initial_z)" rpy="0.0 0.0 0.0"/>
     </joint>
     <xacro:include filename="$(find ur_description)/urdf/ur10.urdf.xacro"/>

File: sr_multi_description/urdf/right_srhand_stand_ur10_bt_sp_biotacs.urdf.xacro (robot description, xacro)
@@ -6,10 +6,5 @@
         <parent link="world"/>
         <child link="stand_link"/>
-        <xacro:if value="$(arg initial_z)">
-            <origin xyz="0.0 0.0 $(arg initial_z)" rpy="0.0 0.0 0.0"/>
-        </xacro:if>
-        <xacro:unless value="$(arg initial_z)">
-            <origin xyz="0.0 0.0 0.0" rpy="0.0 0.0 0.0"/>
-        </xacro:unless>
+        <origin xyz="0.0 0.0 $(arg initial_z)" rpy="0.0 0.0 0.0"/>
     </joint>
     <xacro:include filename="$(find ur_description)/urdf/ur10.urdf.xacro"/>

File: sr_multi_description/urdf/right_srhand_ur10_biotacs.urdf.xacro (robot description, xacro)
@@ -7,10 +7,5 @@
         <parent link="world"/>
         <child link="ra_base_link"/>
-        <xacro:if value="$(arg initial_z)">
-            <origin xyz="0.0 0.0 $(arg initial_z)" rpy="0.0 0.0 0.0"/>
-        </xacro:if>
-        <xacro:unless value="$(arg initial_z)">
-            <origin xyz="0.0 0.0 0.0" rpy="0.0 0.0 0.0"/>
-        </xacro:unless>
+        <origin xyz="0.0 0.0 $(arg initial_z)" rpy="0.0 0.0 0.0"/>
     </joint>
     <xacro:ur10_robot prefix="ra_" joint_limited="false"/>

File: sr_multi_description/urdf/right_srhand_ur10_bt_sp_biotacs.urdf.xacro (robot description, xacro)
@@ -7,10 +7,5 @@
         <parent link="world"/>
         <child link="ra_base_link"/>
-        <xacro:if value="$(arg initial_z)">
-            <origin xyz="0.0 0.0 $(arg initial_z)" rpy="0.0 0.0 0.0"/>
-        </xacro:if>
-        <xacro:unless value="$(arg initial_z)">
-            <origin xyz="0.0 0.0 0.0" rpy="0.0 0.0 0.0"/>
-        </xacro:unless>
+        <origin xyz="0.0 0.0 $(arg initial_z)" rpy="0.0 0.0 0.0"/>
     </joint>
     <xacro:ur10_robot prefix="ra_" joint_limited="false"/>

File: sr_multi_description/urdf/right_srhand_ur10_joint_limited_biotacs.urdf.xacro (robot description, xacro)
@@ -7,10 +7,5 @@
         <parent link="world"/>
         <child link="ra_base_link"/>
-        <xacro:if value="$(arg initial_z)">
-            <origin xyz="0.0 0.0 $(arg initial_z)" rpy="0.0 0.0 0.0"/>
-        </xacro:if>
-        <xacro:unless value="$(arg initial_z)">
-            <origin xyz="0.0 0.0 0.0" rpy="0.0 0.0 0.0"/>
-        </xacro:unless>
+        <origin xyz="0.0 0.0 $(arg initial_z)" rpy="0.0 0.0 0.0"/>
     </joint>
     <xacro:ur10_robot prefix="ra_" joint_limited="true"/>

File: sr_multi_description/urdf/right_srhand_ur10_plus_biotacs.urdf.xacro (robot description, xacro)
@@ -7,10 +7,5 @@
         <parent link="world"/>
         <child link="ra_base_link"/>
-        <xacro:if value="$(arg initial_z)">
-            <origin xyz="0.0 0.0 $(arg initial_z)" rpy="0.0 0.0 0.0"/>
-        </xacro:if>
-        <xacro:unless value="$(arg initial_z)">
-            <origin xyz="0.0 0.0 0.0" rpy="0.0 0.0 0.0"/>
-        </xacro:unless>
+        <origin xyz="0.0 0.0 $(arg initial_z)" rpy="0.0 0.0 0.0"/>
     </joint>
     <xacro:ur10_robot prefix="ra_" joint_limited="false"/>

File: sr_multi_description/urdf/right_srhand_ur5.urdf.xacro (robot description, xacro)
@@ -7,10 +7,5 @@
         <parent link="world"/>
         <child link="ra_base_link"/>
-        <xacro:if value="$(arg initial_z)">
-            <origin xyz="0.0 0.0 $(arg initial_z)" rpy="0.0 0.0 0.0"/>
-        </xacro:if>
-        <xacro:unless value="$(arg initial_z)">
-            <origin xyz="0.0 0.0 0.0" rpy="0.0 0.0 0.0"/>
-        </xacro:unless>
+        <origin xyz="0.0 0.0 $(arg initial_z)" rpy="0.0 0.0 0.0"/>
     </joint>
     <xacro:ur5_robot prefix="ra_" joint_limited="false"/>

File: sr_multi_description/urdf/right_srhand_ur5_joint_limited.urdf.xacro (robot description, xacro)
@@ -7,10 +7,5 @@
         <parent link="world"/>
         <child link="ra_base_link"/>
-        <xacro:if value="$(arg initial_z)">
-            <origin xyz="0.0 0.0 $(arg initial_z)" rpy="0.0 0.0 0.0"/>
-        </xacro:if>
-        <xacro:unless value="$(arg initial_z)">
-            <origin xyz="0.0 0.0 0.0" rpy="0.0 0.0 0.0"/>
-        </xacro:unless>
+        <origin xyz="0.0 0.0 $(arg initial_z)" rpy="0.0 0.0 0.0"/>
     </joint>
     <xacro:ur5_robot prefix="ra_" joint_limited="true"/>

Commit message: changing orientation of the arm

File: sr_multi_description/urdf/left_srhand_ur10.urdf.xacro (robot description, xacro)
@@ -7,5 +7,5 @@
         <parent link="world"/>
         <child link="la_base_link"/>
-        <origin xyz="0.0 0.0 $(arg initial_z)" rpy="0.0 0.0 0.0"/>
+        <origin xyz="0.0 0.0 $(arg initial_z)" rpy="0.0 0.0 ${pi}"/>
     </joint>
     <xacro:ur10_robot prefix="la_" joint_limited="false"/>
