Commit message: addding y separation option

File: sr_multi_description/urdf/bimanual_srhand_ur10.urdf.xacro (robot description, xacro)
@@ -4,5 +4,6 @@
     <xacro:arg name="arm_1_z" default="0.0"/>
     <xacro:arg name="arm_2_z" default="0.0"/>
-    <xacro:arg name="arm_separation" default="1.5"/>
+    <xacro:arg name="arm_x_separation" default="1.5"/>
+    <xacro:arg name="arm_y_separation" default="1.5"/>
     <joint name="world_to_arm_1_joint" type="fixed">
         <parent link="world"/>
@@ -14,5 +15,5 @@
         <parent link="world"/>
         <child link="la_base_link"/>
-        <origin xyz="$(arg arm_separation) 0.0 $(arg arm_2_z)" rpy="0.0 0.0 0.0"/>
+        <origin xyz="$(arg arm_x_separation) $(arg arm_y_separation) $(arg arm_2_z)" rpy="0.0 0.0 0.0"/>
     </joint>
     <xacro:ur10_robot prefix="la_" joint_limited="true"/>

Commit message: Changing orientation

File: sr_multi_description/urdf/bimanual_srhand_ur10.urdf.xacro (robot description, xacro)
@@ -5,5 +5,5 @@
     <xacro:arg name="arm_2_z" default="0.0"/>
     <xacro:arg name="arm_x_separation" default="1.5"/>
-    <xacro:arg name="arm_y_separation" default="1.5"/>
+    <xacro:arg name="arm_y_separation" default="0.0"/>
     <joint name="world_to_arm_1_joint" type="fixed">
         <parent link="world"/>
@@ -21,5 +21,5 @@
     <xacro:include filename="$(find sr_description)/hand/xacro/full_hand.urdf.xacro"/>
     <xacro:include filename="$(find sr_description)/other/xacro/gazebo/gazebo.urdf.xacro"/>
-    <xacro:shadowhand muscletrans="false" muscle="false" bio="false" bt_sp="false" ubi="false" eli="false" reflect="-1.0" prefix="rh_" lf="true" cable_mesh="true"/>
+    <xacro:shadowhand muscletrans="false" muscle="false" bio="false" bt_sp="false" ubi="false" eli="false" reflect="1.0" prefix="rh_" lf="true" cable_mesh="true"/>
     <joint name="ra_arm_to_hand" type="fixed">
         <parent link="ra_ee_link"/>
@@ -27,9 +27,9 @@
         <origin xyz="0.012 0.0 0.0" rpy="${pi/2.0} ${0.0} ${pi/2.0}"/>
     </joint>
-    <xacro:shadowhand muscletrans="false" muscle="false" bio="false" bt_sp="false" ubi="false" eli="false" reflect="1.0" prefix="lh_" lf="true" cable_mesh="true"/>
+    <xacro:shadowhand muscletrans="false" muscle="false" bio="false" bt_sp="false" ubi="false" eli="false" reflect="-1.0" prefix="lh_" lf="true" cable_mesh="true"/>
     <joint name="la_arm_to_hand" type="fixed">
         <parent link="la_ee_link"/>
         <child link="lh_forearm"/>
-        <origin xyz="0.012 0.0 0.0" rpy="${pi/2.0} ${0.0} ${pi/2.0}"/>
+        <origin xyz="0.012 0.0 0.0" rpy="${pi/2.0} ${0.0} -${pi/2.0}"/>
     </joint>
 </robot>

Commit message: updated for new bimanual world

File: sr_multi_description/urdf/bimanual_srhand_ur10.urdf.xacro (robot description, xacro)
@@ -9,7 +9,7 @@
         <parent link="world"/>
         <child link="ra_base_link"/>
-        <origin xyz="0.0 0.0 $(arg arm_1_z)" rpy="0.0 0.0 0.0"/>
+        <origin xyz="0.0 0.0 $(arg arm_1_z)" rpy="0.0 0.0 ${pi}"/>
     </joint>
-    <xacro:ur10_robot prefix="ra_" joint_limited="true"/>
+    <xacro:ur10_robot prefix="ra_" joint_limited="false"/>
     <joint name="world_to_arm_2_joint" type="fixed">
         <parent link="world"/>
@@ -17,5 +17,5 @@
         <origin xyz="$(arg arm_x_separation) $(arg arm_y_separation) $(arg arm_2_z)" rpy="0.0 0.0 0.0"/>
     </joint>
-    <xacro:ur10_robot prefix="la_" joint_limited="true"/>
+    <xacro:ur10_robot prefix="la_" joint_limited="false"/>
     <xacro:include filename="$(find sr_description)/materials.urdf.xacro"/>
     <xacro:include filename="$(find sr_description)/hand/xacro/full_hand.urdf.xacro"/>
@@ -31,5 +31,5 @@
         <parent link="la_ee_link"/>
         <child link="lh_forearm"/>
-        <origin xyz="0.012 0.0 0.0" rpy="${pi/2.0} ${0.0} -${pi/2.0}"/>
+        <origin xyz="0.012 0.0 0.0" rpy="${pi/2.0} ${0.0} ${pi/2.0}"/>
     </joint>
 </robot>

Commit message: update for correct arm positions

File: sr_multi_description/urdf/bimanual_srhand_ur10.urdf.xacro (robot description, xacro)
@@ -9,5 +9,5 @@
         <parent link="world"/>
         <child link="ra_base_link"/>
-        <origin xyz="0.0 0.0 $(arg arm_1_z)" rpy="0.0 0.0 ${pi}"/>
+        <origin xyz="0.0 0.0 $(arg arm_1_z)" rpy="0.0 0.0 0.0"/>
     </joint>
     <xacro:ur10_robot prefix="ra_" joint_limited="false"/>
@@ -15,5 +15,5 @@
         <parent link="world"/>
         <child link="la_base_link"/>
-        <origin xyz="$(arg arm_x_separation) $(arg arm_y_separation) $(arg arm_2_z)" rpy="0.0 0.0 0.0"/>
+        <origin xyz="$(arg arm_x_separation) $(arg arm_y_separation) $(arg arm_2_z)" rpy="0.0 0.0 ${pi}"/>
     </joint>
     <xacro:ur10_robot prefix="la_" joint_limited="false"/>
