Commit message: trying to include new driver via combined robot hw plugin

File: sr_multi_description/urdf/right_srhand_ur10_new_driver.urdf.xacro (robot description, xacro)
@@ -20,10 +20,4 @@
     kinematics_file="${load_yaml('$(arg kinematics_config)')}"
   />
-  <link name="world" />
-  <joint name="world_joint" type="fixed">
-    <parent link="world" />
-    <child link = "base_link" />
-    <origin xyz="0.0 0.0 0.0" rpy="0.0 0.0 0.0" />
-  </joint>
     <xacro:include filename="$(find sr_description)/materials.urdf.xacro"/>
     <xacro:include filename="$(find sr_description)/hand/xacro/full_hand.urdf.xacro"/>
