Commit message: Fixed ur5

File: sr_multi_description/urdf/left_srhand_ur5.urdf.xacro (robot description, xacro)
@@ -7,14 +7,14 @@
         <parent link="world"/>
         <child link="la_base_link"/>
-        <origin xyz="0.0 0.0 $(arg initial_z)" rpy="0.0 0.0 0.0"/>
+        <origin xyz="0.0 0.0 $(arg initial_z)" rpy="0.0 0.0 ${pi}"/>
     </joint>
     <xacro:arg name="kinematics_config" default="$(find ur_description)/config/ur10_default.yaml"/>
     <xacro:arg name="transmission_hw_interface" default="hardware_interface/PositionJointInterface"/>
-    <xacro:ur10_robot prefix="la_" joint_limited="false" transmission_hw_interface="$(arg transmission_hw_interface)" kinematics_file="${load_yaml('$(arg kinematics_config)')}"/>
+    <xacro:ur5_robot prefix="la_" joint_limited="false" transmission_hw_interface="$(arg transmission_hw_interface)" kinematics_file="${load_yaml('$(arg kinematics_config)')}"/>
     <xacro:include filename="$(find sr_description)/materials.urdf.xacro"/>
     <xacro:include filename="$(find sr_description)/hand/xacro/full_hand.urdf.xacro"/>
     <xacro:include filename="$(find sr_description)/other/xacro/gazebo/gazebo.urdf.xacro"/>
     <xacro:shadowhand muscletrans="false" muscle="false" bio="false" bt_sp="false" ubi="false" eli="false"
-                      reflect="-1.0" prefix="lh_" lf="true"/>
+                      reflect="-1.0" prefix="lh_" lf="true" cable_mesh="true"/>
     <joint name="la_arm_to_hand" type="fixed">
         <parent link="la_ee_link"/>

File: sr_multi_description/urdf/right_srhand_ur5.urdf.xacro (robot description, xacro)
@@ -16,5 +16,5 @@
     <xacro:include filename="$(find sr_description)/other/xacro/gazebo/gazebo.urdf.xacro"/>
     <xacro:shadowhand muscletrans="false" muscle="false" bio="false" bt_sp="false" ubi="false" eli="false"
-                      reflect="1.0" prefix="rh_" lf="true"/>
+                      reflect="1.0" prefix="rh_" lf="true" cable_mesh="true"/>
     <joint name="ra_arm_to_hand" type="fixed">
         <parent link="ra_ee_link"/>
