Commit message: add y separation to biotac left xacro

File: sr_multi_description/urdf/left_srhand_ur10e_bt_sp_biotacs.urdf.xacro (robot description, xacro)
@@ -4,8 +4,10 @@
     <link name="world"/>
     <xacro:arg name="initial_z" default="0.0"/>
+    <xacro:arg name="arm_x_separation" default="0.0"/>
+    <xacro:arg name="arm_y_separation" default="0.0"/>
     <joint name="world_joint" type="fixed">
         <parent link="world"/>
         <child link="la_base_link"/>
-        <origin xyz="0.0 0.0 $(arg initial_z)" rpy="0.0 0.0 ${pi}"/>
+        <origin xyz="$(arg arm_x_separation) $(arg arm_y_separation) $(arg initial_z)" rpy="0.0 0.0 ${pi}"/>
     </joint>
     <xacro:arg name="kinematics_config" default="$(find ur_e_description)/config/ur10e_default.yaml"/>
