Commit message: Fixing some files and scripts

File: sr_multi_description/urdf/left_srhand_lite_ur5e.urdf.xacro (robot description, xacro)
@@ -7,5 +7,5 @@
     <joint name="world_joint" type="fixed">
         <parent link="world"/>
-        <child link="ra_base_link"/>
+        <child link="la_base_link"/>
         <origin xyz="0.0 0.0 $(arg initial_z)" rpy="0.0 0.0 0.0"/>
     </joint>

Commit message: fixing orientation for left arms)

File: sr_multi_description/urdf/left_srhand_lite_ur5e.urdf.xacro (robot description, xacro)
@@ -8,5 +8,5 @@
         <parent link="world"/>
         <child link="la_base_link"/>
-        <origin xyz="0.0 0.0 $(arg initial_z)" rpy="0.0 0.0 0.0"/>
+        <origin xyz="0.0 0.0 $(arg initial_z)" rpy="0.0 0.0 {pi}"/>
     </joint>
     <xacro:ur5e_robot prefix="la_" joint_limited="false" transmission_hw_interface="$(arg transmission_hw_interface)" kinematics_file="${load_yaml('$(arg kinematics_config)')}"/>

File: sr_multi_description/urdf/left_srhand_ur10_joint_limited.urdf.xacro (robot description, xacro)
@@ -7,5 +7,5 @@
         <parent link="world"/>
         <child link="la_base_link"/>
-        <origin xyz="0.0 0.0 $(arg initial_z)" rpy="0.0 0.0 0.0"/>
+        <origin xyz="0.0 0.0 $(arg initial_z)" rpy="0.0 0.0 {pi}"/>
     </joint>
     <xacro:arg name="kinematics_config" default="$(find ur_description)/config/ur10_default.yaml"/>

File: sr_multi_description/urdf/left_srhand_ur5_joint_limited.urdf.xacro (robot description, xacro)
@@ -7,5 +7,5 @@
         <parent link="world"/>
         <child link="la_base_link"/>
-        <origin xyz="0.0 0.0 $(arg initial_z)" rpy="0.0 0.0 0.0"/>
+        <origin xyz="0.0 0.0 $(arg initial_z)" rpy="0.0 0.0 {pi}"/>
     </joint>
     <xacro:arg name="kinematics_config" default="$(find ur_description)/config/ur5_default.yaml"/>

File: sr_multi_description/urdf/left_srhand_ur5e.urdf.xacro (robot description, xacro)
@@ -8,5 +8,5 @@
         <parent link="world"/>
         <child link="la_base_link"/>
-        <origin xyz="0.0 0.0 $(arg initial_z)" rpy="0.0 0.0 0.0"/>
+        <origin xyz="0.0 0.0 $(arg initial_z)" rpy="0.0 0.0 {pi}"/>
     </joint>
     <xacro:ur5e_robot prefix="la_" joint_limited="false" transmission_hw_interface="$(arg transmission_hw_interface)" kinematics_file="${load_yaml('$(arg kinematics_config)')}"/>

Commit message: fixing orientation for left arms

File: sr_multi_description/urdf/left_srhand_lite_ur5e.urdf.xacro (robot description, xacro)
@@ -8,5 +8,5 @@
         <parent link="world"/>
         <child link="la_base_link"/>
-        <origin xyz="0.0 0.0 $(arg initial_z)" rpy="0.0 0.0 {pi}"/>
+        <origin xyz="0.0 0.0 $(arg initial_z)" rpy="0.0 0.0 ${pi}"/>
     </joint>
     <xacro:ur5e_robot prefix="la_" joint_limited="false" transmission_hw_interface="$(arg transmission_hw_interface)" kinematics_file="${load_yaml('$(arg kinematics_config)')}"/>

File: sr_multi_description/urdf/left_srhand_ur10_joint_limited.urdf.xacro (robot description, xacro)
@@ -7,5 +7,5 @@
         <parent link="world"/>
         <child link="la_base_link"/>
-        <origin xyz="0.0 0.0 $(arg initial_z)" rpy="0.0 0.0 {pi}"/>
+        <origin xyz="0.0 0.0 $(arg initial_z)" rpy="0.0 0.0 ${pi}"/>
     </joint>
     <xacro:arg name="kinematics_config" default="$(find ur_description)/config/ur10_default.yaml"/>

File: sr_multi_description/urdf/left_srhand_ur5_joint_limited.urdf.xacro (robot description, xacro)
@@ -7,5 +7,5 @@
         <parent link="world"/>
         <child link="la_base_link"/>
-        <origin xyz="0.0 0.0 $(arg initial_z)" rpy="0.0 0.0 {pi}"/>
+        <origin xyz="0.0 0.0 $(arg initial_z)" rpy="0.0 0.0 ${pi}"/>
     </joint>
     <xacro:arg name="kinematics_config" default="$(find ur_description)/config/ur5_default.yaml"/>

File: sr_multi_description/urdf/left_srhand_ur5e.urdf.xacro (robot description, xacro)
@@ -8,5 +8,5 @@
         <parent link="world"/>
         <child link="la_base_link"/>
-        <origin xyz="0.0 0.0 $(arg initial_z)" rpy="0.0 0.0 {pi}"/>
+        <origin xyz="0.0 0.0 $(arg initial_z)" rpy="0.0 0.0 ${pi}"/>
     </joint>
     <xacro:ur5e_robot prefix="la_" joint_limited="false" transmission_hw_interface="$(arg transmission_hw_interface)" kinematics_file="${load_yaml('$(arg kinematics_config)')}"/>

Commit message: working generic test

File: sr_multi_description/urdf/left_srhand_lite_ur5e.urdf.xacro (robot description, xacro)
@@ -8,5 +8,5 @@
         <parent link="world"/>
         <child link="la_base_link"/>
-        <origin xyz="0.0 0.0 $(arg initial_z)" rpy="0.0 0.0 0.0"/>
+        <origin xyz="0.0 0.0 $(arg initial_z)" rpy="0.0 0.0 ${pi}"/>
     </joint>
     <xacro:ur5e_robot prefix="la_" joint_limited="false" transmission_hw_interface="$(arg transmission_hw_interface)" kinematics_file="${load_yaml('$(arg kinematics_config)')}"/>
