Commit message: updating xacros

File: sr_multi_description/urdf/left_srhand_lite_ur5.urdf.xacro (robot description, xacro)
@@ -1,5 +1,7 @@
-<robot xmlns:xacro="http://ros.org/wiki/xacro" name="ur10srh">
+<robot xmlns:xacro="http://ros.org/wiki/xacro" name="ur5srh">
     <!--<xacro:include filename="$(find ur_description)/urdf/gazebo.urdf.xacro" />-->
-    <xacro:include filename="$(find ur_description)/urdf/ur10.urdf.xacro"/>
+    <xacro:include filename="$(find ur_description)/urdf/ur5.urdf.xacro"/>
+    <xacro:arg name="kinematics_config" default="$(find ur_description)/config/ur5_default.yaml"/>
+    <xacro:arg name="transmission_hw_interface" default="hardware_interface/PositionJointInterface"/>
     <link name="world"/>
     <xacro:arg name="initial_z" default="0.0"/>
@@ -11,12 +13,11 @@
         <origin xyz="$(arg arm_x_separation) $(arg arm_y_separation) $(arg initial_z)" rpy="0.0 0.0 ${pi}"/>
     </joint>
-    <xacro:arg name="kinematics_config" default="$(find ur_description)/config/ur10_default.yaml"/>
+    <xacro:arg name="kinematics_config" default="$(find ur_description)/config/ur5_default.yaml"/>
     <xacro:arg name="transmission_hw_interface" default="hardware_interface/PositionJointInterface"/>
-    <xacro:ur10_robot prefix="la_" joint_limited="false" transmission_hw_interface="$(arg transmission_hw_interface)" kinematics_file="${load_yaml('$(arg kinematics_config)')}"/>
+    <xacro:ur5_robot prefix="la_" joint_limited="false" transmission_hw_interface="$(arg transmission_hw_interface)" kinematics_file="${load_yaml('$(arg kinematics_config)')}"/>
     <xacro:include filename="$(find sr_description)/materials.urdf.xacro"/>
-    <xacro:include filename="$(find sr_description)/hand/xacro/full_hand.urdf.xacro"/>
+    <xacro:include filename="$(find sr_description)/hand/xacro/hand_lite.urdf.xacro"/>
     <xacro:include filename="$(find sr_description)/other/xacro/gazebo/gazebo.urdf.xacro"/>
-    <xacro:shadowhand muscletrans="false" muscle="false" bio="false" bt_sp="false" ubi="false" eli="false"
-                      reflect="-1.0" prefix="lh_" lf="true" cable_mesh="true"/>
+    <xacro:shadowhand muscletrans="false" muscle="false" bio="false" bt_sp="false" ubi="false" eli="false" reflect="-1.0" prefix="lh_" extra_lite="false"/>
     <joint name="la_arm_to_hand" type="fixed">
         <parent link="la_ee_link"/>

File: sr_multi_description/urdf/left_srhand_lite_ur5e.urdf.xacro (robot description, xacro)
@@ -5,8 +5,10 @@
     <link name="world"/>
     <xacro:arg name="initial_z" default="0.0"/>
+    <xacro:arg name="arm_x_separation" default="0.0"/>
+    <xacro:arg name="arm_y_separation" default="0.0"/>
     <joint name="world_joint" type="fixed">
         <parent link="world"/>
         <child link="la_base_link"/>
-        <origin xyz="0.0 0.0 $(arg initial_z)" rpy="0.0 0.0 ${pi}"/>
+        <origin xyz="$(arg arm_x_separation) $(arg arm_y_separation) $(arg initial_z)" rpy="0.0 0.0 ${pi}"/>
     </joint>
     <xacro:ur5e_robot prefix="la_" joint_limited="false" transmission_hw_interface="$(arg transmission_hw_interface)" kinematics_file="${load_yaml('$(arg kinematics_config)')}"/>

File: sr_multi_description/urdf/left_srhand_ur10_bt_sp_biotacs.urdf.xacro (robot description, xacro)
@@ -4,8 +4,10 @@
     <link name="world"/>
     <xacro:arg name="initial_z" default="0.0"/>
+    <xacro:arg name="arm_x_separation" default="0.0"/>
+    <xacro:arg name="arm_y_separation" default="0.0"/>
     <joint name="world_joint" type="fixed">
         <parent link="world"/>
         <child link="la_base_link"/>
-        <origin xyz="0.0 0.0 $(arg initial_z)" rpy="0.0 0.0 ${pi}"/>
+        <origin xyz="$(arg arm_x_separation) $(arg arm_y_separation) $(arg initial_z)" rpy="0.0 0.0 ${pi}"/>
     </joint>
     <xacro:arg name="kinematics_config" default="$(find ur_description)/config/ur10_default.yaml"/>

File: sr_multi_description/urdf/left_srhand_ur10_joint_limited.urdf.xacro (robot description, xacro)
@@ -4,8 +4,10 @@
     <link name="world"/>
     <xacro:arg name="initial_z" default="0.0"/>
+    <xacro:arg name="arm_x_separation" default="0.0"/>
+    <xacro:arg name="arm_y_separation" default="0.0"/>
     <joint name="world_joint" type="fixed">
         <parent link="world"/>
         <child link="la_base_link"/>
-        <origin xyz="0.0 0.0 $(arg initial_z)" rpy="0.0 0.0 ${pi}"/>
+        <origin xyz="$(arg arm_x_separation) $(arg arm_y_separation) $(arg initial_z)" rpy="0.0 0.0 ${pi}"/>
     </joint>
     <xacro:arg name="kinematics_config" default="$(find ur_description)/config/ur10_default.yaml"/>

File: sr_multi_description/urdf/left_srhand_ur5.urdf.xacro (robot description, xacro)
@@ -4,8 +4,10 @@
     <link name="world"/>
     <xacro:arg name="initial_z" default="0.0"/>
+    <xacro:arg name="arm_x_separation" default="0.0"/>
+    <xacro:arg name="arm_y_separation" default="0.0"/>
     <joint name="world_joint" type="fixed">
         <parent link="world"/>
         <child link="la_base_link"/>
-        <origin xyz="0.0 0.0 $(arg initial_z)" rpy="0.0 0.0 ${pi}"/>
+        <origin xyz="$(arg arm_x_separation) $(arg arm_y_separation) $(arg initial_z)" rpy="0.0 0.0 ${pi}"/>
     </joint>
     <xacro:arg name="kinematics_config" default="$(find ur_description)/config/ur5_default.yaml"/>

File: sr_multi_description/urdf/left_srhand_ur5_joint_limited.urdf.xacro (robot description, xacro)
@@ -4,8 +4,10 @@
     <link name="world"/>
     <xacro:arg name="initial_z" default="0.0"/>
+    <xacro:arg name="arm_x_separation" default="0.0"/>
+    <xacro:arg name="arm_y_separation" default="0.0"/>
     <joint name="world_joint" type="fixed">
         <parent link="world"/>
         <child link="la_base_link"/>
-        <origin xyz="0.0 0.0 $(arg initial_z)" rpy="0.0 0.0 ${pi}"/>
+        <origin xyz="$(arg arm_x_separation) $(arg arm_y_separation) $(arg initial_z)" rpy="0.0 0.0 ${pi}"/>
     </joint>
     <xacro:arg name="kinematics_config" default="$(find ur_description)/config/ur5_default.yaml"/>

File: sr_multi_description/urdf/left_srhand_ur5e.urdf.xacro (robot description, xacro)
@@ -5,8 +5,10 @@
     <link name="world"/>
     <xacro:arg name="initial_z" default="0.0"/>
+    <xacro:arg name="arm_x_separation" default="0.0"/>
+    <xacro:arg name="arm_y_separation" default="0.0"/>
     <joint name="world_joint" type="fixed">
         <parent link="world"/>
         <child link="la_base_link"/>
-        <origin xyz="0.0 0.0 $(arg initial_z)" rpy="0.0 0.0 ${pi}"/>
+        <origin xyz="$(arg arm_x_separation) $(arg arm_y_separation) $(arg initial_z)" rpy="0.0 0.0 ${pi}"/>
     </joint>
     <xacro:ur5e_robot prefix="la_" joint_limited="false" transmission_hw_interface="$(arg transmission_hw_interface)" kinematics_file="${load_yaml('$(arg kinematics_config)')}"/>
