Commit message: updates

File: sr_multi_description/urdf/bimanual_srhand_ur10e.urdf.xacro (robot description, xacro)
@@ -28,5 +28,5 @@
         <parent link="ra_flange"/>
         <child link="rh_forearm"/>
-        <origin xyz="0.012 0.0 0.0" rpy="${pi/2.0} ${0.0} ${pi/2.0}"/>
+        <origin xyz="0.012 0.0 0.0" rpy="${pi/2.0} ${pi} ${pi/2.0}"/>
     </joint>
     <xacro:shadowhand muscletrans="false" muscle="false" bio="false" bt_sp="false" ubi="false" eli="false" reflect="-1.0" prefix="lh_" lf="true" cable_mesh="true"/>
@@ -34,5 +34,5 @@
         <parent link="la_flange"/>
         <child link="lh_forearm"/>
-        <origin xyz="0.012 0.0 0.0" rpy="${pi/2.0} ${0.0} ${pi/2.0}"/>
+        <origin xyz="0.012 0.0 0.0" rpy="${pi/2.0} ${pi} ${pi/2.0}"/>
     </joint>
 </robot>

File: sr_multi_description/urdf/left_srhand_ur10e.urdf.xacro (robot description, xacro)
@@ -21,5 +21,5 @@
         <parent link="la_flange"/>
         <child link="lh_forearm"/>
-        <origin xyz="0.012 0.0 0.0" rpy="${pi/2.0} ${0.0} ${pi/2.0}"/>
+        <origin xyz="0.012 0.0 0.0" rpy="${pi/2.0} ${pi} ${pi/2.0}"/>
     </joint>
 </robot>

File: sr_multi_description/urdf/right_srhand_ur10e.urdf.xacro (robot description, xacro)
@@ -20,5 +20,5 @@
         <parent link="ra_flange"/>
         <child link="rh_forearm"/>
-        <origin xyz="0.012 0.0 0.0" rpy="${pi/2.0} ${0.0} ${pi/2.0}"/>
+        <origin xyz="0.012 0.0 0.0" rpy="${pi/2.0} ${pi} ${pi/2.0}"/>
     </joint>
 </robot>
