Commit message: updating hand position

File: sr_multi_description/urdf/bimanual_srhand_lite_ur5e.urdf.xacro (robot description, xacro)
@@ -27,5 +27,5 @@
         <parent link="ra_flange"/>
         <child link="rh_forearm"/>
-        <origin xyz="0.012 0.0 0.0" rpy="${pi/2.0} ${0.0} ${pi/2.0}"/>
+        <origin xyz="0.012 0.0 0.0" rpy="${pi/2.0} ${pi} ${pi/2.0}"/>
     </joint>
     <xacro:shadowhand muscletrans="false" muscle="false" bio="false" bt_sp="false" ubi="false" eli="false" reflect="-1.0" prefix="lh_" extra_lite="false"/>
@@ -33,5 +33,5 @@
         <parent link="la_flange"/>
         <child link="lh_forearm"/>
-        <origin xyz="0.012 0.0 0.0" rpy="${pi/2.0} ${0.0} ${pi/2.0}"/>
+        <origin xyz="0.012 0.0 0.0" rpy="${pi/2.0} ${pi} ${pi/2.0}"/>
     </joint>
 </robot>

File: sr_multi_description/urdf/bimanual_srhand_plus_bt_sp_biotacs_ur10.urdf.xacro (robot description, xacro)
@@ -28,5 +28,5 @@
         <parent link="ra_flange"/>
         <child link="rh_forearm"/>
-        <origin xyz="0.012 0.0 0.0" rpy="${pi/2.0} ${0.0} ${pi/2.0}"/>
+        <origin xyz="0.012 0.0 0.0" rpy="${pi/2.0} ${pi} ${pi/2.0}"/>
     </joint>
     <xacro:shadowhand muscletrans="false" muscle="false" hand_type="hand_e_plus" bio="false" bt_sp="true" ubi="false" eli="false" reflect="-1.0" prefix="lh_" lf="true" cable_mesh="true"/>
@@ -34,5 +34,5 @@
         <parent link="la_flange"/>
         <child link="lh_forearm"/>
-        <origin xyz="0.012 0.0 0.0" rpy="${pi/2.0} ${0.0} ${pi/2.0}"/>
+        <origin xyz="0.012 0.0 0.0" rpy="${pi/2.0} ${pi} ${pi/2.0}"/>
     </joint>
 </robot>

File: sr_multi_description/urdf/bimanual_srhand_plus_bt_sp_biotacs_ur10e.urdf.xacro (robot description, xacro)
@@ -28,5 +28,5 @@
         <parent link="ra_flange"/>
         <child link="rh_forearm"/>
-        <origin xyz="0.012 0.0 0.0" rpy="${pi/2.0} ${0.0} ${pi/2.0}"/>
+        <origin xyz="0.012 0.0 0.0" rpy="${pi/2.0} ${pi} ${pi/2.0}"/>
     </joint>
     <xacro:shadowhand muscletrans="false" muscle="false" hand_type="hand_e_plus" bio="false" bt_sp="true" ubi="false" eli="false" reflect="-1.0" prefix="lh_" lf="true" cable_mesh="true"/>
@@ -34,5 +34,5 @@
         <parent link="la_flange"/>
         <child link="lh_forearm"/>
-        <origin xyz="0.012 0.0 0.0" rpy="${pi/2.0} ${0.0} ${pi/2.0}"/>
+        <origin xyz="0.012 0.0 0.0" rpy="${pi/2.0} ${pi} ${pi/2.0}"/>
     </joint>
 </robot>

File: sr_multi_description/urdf/bimanual_srhand_ur10.urdf.xacro (robot description, xacro)
@@ -28,5 +28,5 @@
         <parent link="ra_flange"/>
         <child link="rh_forearm"/>
-        <origin xyz="0.012 0.0 0.0" rpy="${pi/2.0} ${0.0} ${pi/2.0}"/>
+        <origin xyz="0.012 0.0 0.0" rpy="${pi/2.0} ${pi} ${pi/2.0}"/>
     </joint>
     <xacro:shadowhand muscletrans="false" muscle="false" bio="false" bt_sp="false" ubi="false" eli="false" reflect="-1.0" prefix="lh_" lf="true" cable_mesh="true"/>
@@ -34,5 +34,5 @@
         <parent link="la_flange"/>
         <child link="lh_forearm"/>
-        <origin xyz="0.012 0.0 0.0" rpy="${pi/2.0} ${0.0} ${pi/2.0}"/>
+        <origin xyz="0.012 0.0 0.0" rpy="${pi/2.0} ${pi} ${pi/2.0}"/>
     </joint>
 </robot>

File: sr_multi_description/urdf/bimanual_srhand_ur5e.urdf.xacro (robot description, xacro)
@@ -27,5 +27,5 @@
         <parent link="ra_flange"/>
         <child link="rh_forearm"/>
-        <origin xyz="0.012 0.0 0.0" rpy="${pi/2.0} ${0.0} ${pi/2.0}"/>
+        <origin xyz="0.012 0.0 0.0" rpy="${pi/2.0} ${pi} ${pi/2.0}"/>
     </joint>
     <xacro:shadowhand muscletrans="false" muscle="false" bio="false" bt_sp="false" ubi="false" eli="false" reflect="-1.0" prefix="lh_" lf="true" cable_mesh="true"/>
@@ -33,5 +33,5 @@
         <parent link="la_flange"/>
         <child link="lh_forearm"/>
-        <origin xyz="0.012 0.0 0.0" rpy="${pi/2.0} ${0.0} ${pi/2.0}"/>
+        <origin xyz="0.012 0.0 0.0" rpy="${pi/2.0} ${pi} ${pi/2.0}"/>
     </joint>
 </robot>

File: sr_multi_description/urdf/for_moveit/srhand_ur10arm.urdf.xacro (robot description, xacro)
@@ -16,5 +16,5 @@
         <parent link="ra_flange"/>
         <child link="rh_forearm"/>
-        <origin xyz="0.012 0.0 0.0" rpy="${pi/2.0} ${0.0} ${pi/2.0}"/>
+        <origin xyz="0.012 0.0 0.0" rpy="${pi/2.0} ${pi} ${pi/2.0}"/>
     </joint>
 </robot>

File: sr_multi_description/urdf/left_srhand_lite_ur5.urdf.xacro (robot description, xacro)
@@ -22,5 +22,5 @@
         <parent link="la_flange"/>
         <child link="lh_forearm"/>
-        <origin xyz="0.012 0.0 0.0" rpy="${pi/2.0} ${0.0} ${pi/2.0}"/>
+        <origin xyz="0.012 0.0 0.0" rpy="${pi/2.0} ${pi} ${pi/2.0}"/>
     </joint>
 </robot>

File: sr_multi_description/urdf/left_srhand_lite_ur5e.urdf.xacro (robot description, xacro)
@@ -20,5 +20,5 @@
         <parent link="la_flange"/>
         <child link="lh_forearm"/>
-        <origin xyz="0.012 0.0 0.0" rpy="${pi/2.0} ${0.0} ${pi/2.0}"/>
+        <origin xyz="0.012 0.0 0.0" rpy="${pi/2.0} ${pi} ${pi/2.0}"/>
     </joint>
 </robot>

File: sr_multi_description/urdf/left_srhand_ur10.urdf.xacro (robot description, xacro)
@@ -22,5 +22,5 @@
         <parent link="la_flange"/>
         <child link="lh_forearm"/>
-        <origin xyz="0.012 0.0 0.0" rpy="${pi/2.0} ${0.0} ${pi/2.0}"/>
+        <origin xyz="0.012 0.0 0.0" rpy="${pi/2.0} ${pi} ${pi/2.0}"/>
     </joint>
 </robot>

File: sr_multi_description/urdf/left_srhand_ur10_bt_sp_biotacs.urdf.xacro (robot description, xacro)
@@ -22,5 +22,5 @@
         <parent link="la_flange"/>
         <child link="lh_forearm"/>
-        <origin xyz="0.012 0.0 0.0" rpy="${pi/2.0} ${0.0} ${pi/2.0}"/>
+        <origin xyz="0.012 0.0 0.0" rpy="${pi/2.0} ${pi} ${pi/2.0}"/>
     </joint>
 </robot>

File: sr_multi_description/urdf/left_srhand_ur10e_bt_sp_biotacs.urdf.xacro (robot description, xacro)
@@ -22,5 +22,5 @@
         <parent link="la_flange"/>
         <child link="lh_forearm"/>
-        <origin xyz="0.012 0.0 0.0" rpy="${pi/2.0} ${0.0} ${pi/2.0}"/>
+        <origin xyz="0.012 0.0 0.0" rpy="${pi/2.0} ${pi} ${pi/2.0}"/>
     </joint>
 </robot>

File: sr_multi_description/urdf/left_srhand_ur5.urdf.xacro (robot description, xacro)
@@ -22,5 +22,5 @@
         <parent link="la_flange"/>
         <child link="lh_forearm"/>
-        <origin xyz="0.012 0.0 0.0" rpy="${pi/2.0} ${0.0} ${pi/2.0}"/>
+        <origin xyz="0.012 0.0 0.0" rpy="${pi/2.0} ${pi} ${pi/2.0}"/>
     </joint>
 </robot>

File: sr_multi_description/urdf/left_srhand_ur5e.urdf.xacro (robot description, xacro)
@@ -20,5 +20,5 @@
         <parent link="la_flange"/>
         <child link="lh_forearm"/>
-        <origin xyz="0.012 0.0 0.0" rpy="${pi/2.0} ${0.0} ${pi/2.0}"/>
+        <origin xyz="0.012 0.0 0.0" rpy="${pi/2.0} ${pi} ${pi/2.0}"/>
     </joint>
 </robot>

File: sr_multi_description/urdf/right_srhand_bt_sp_biotacs_two_ur10.urdf.xacro (robot description, xacro)
@@ -27,5 +27,5 @@
         <parent link="ra_flange"/>
         <child link="rh_forearm"/>
-        <origin xyz="0.012 0.0 0.0" rpy="${pi/2.0} ${0.0} ${pi/2.0}"/>
+        <origin xyz="0.012 0.0 0.0" rpy="${pi/2.0} ${pi} ${pi/2.0}"/>
     </joint>
 </robot>

File: sr_multi_description/urdf/right_srhand_lite_ur10e.urdf.xacro (robot description, xacro)
@@ -19,5 +19,5 @@
         <parent link="ra_flange"/>
         <child link="rh_forearm"/>
-        <origin xyz="0.012 0.0 0.0" rpy="${pi/2.0} ${0.0} ${pi/2.0}"/>
+        <origin xyz="0.012 0.0 0.0" rpy="${pi/2.0} ${pi} ${pi/2.0}"/>
     </joint>
 </robot>

File: sr_multi_description/urdf/right_srhand_lite_ur5.urdf.xacro (robot description, xacro)
@@ -20,5 +20,5 @@
         <parent link="ra_flange"/>
         <child link="rh_forearm"/>
-        <origin xyz="0.012 0.0 0.0" rpy="${pi/2.0} ${0.0} ${pi/2.0}"/>
+        <origin xyz="0.012 0.0 0.0" rpy="${pi/2.0} ${pi} ${pi/2.0}"/>
     </joint>
 </robot>

File: sr_multi_description/urdf/right_srhand_lite_ur5e.urdf.xacro (robot description, xacro)
@@ -18,5 +18,5 @@
         <parent link="ra_flange"/>
         <child link="rh_forearm"/>
-        <origin xyz="0.012 0.0 0.0" rpy="${pi/2.0} ${0.0} ${pi/2.0}"/>
+        <origin xyz="0.012 0.0 0.0" rpy="${pi/2.0} ${pi} ${pi/2.0}"/>
     </joint>
 </robot>

File: sr_multi_description/urdf/right_srhand_two_ur10.urdf.xacro (robot description, xacro)
@@ -27,5 +27,5 @@
         <parent link="ra_flange"/>
         <child link="rh_forearm"/>
-        <origin xyz="0.012 0.0 0.0" rpy="${pi/2.0} ${0.0} ${pi/2.0}"/>
+        <origin xyz="0.012 0.0 0.0" rpy="${pi/2.0} ${pi} ${pi/2.0}"/>
     </joint>
 </robot>

File: sr_multi_description/urdf/right_srhand_ur10.urdf.xacro (robot description, xacro)
@@ -20,5 +20,5 @@
         <parent link="ra_flange"/>
         <child link="rh_forearm"/>
-        <origin xyz="0.012 0.0 0.0" rpy="${pi/2.0} ${0.0} ${pi/2.0}"/>
+        <origin xyz="0.012 0.0 0.0" rpy="${pi/2.0} ${pi} ${pi/2.0}"/>
     </joint>
 </robot>

File: sr_multi_description/urdf/right_srhand_ur10_biotacs.urdf.xacro (robot description, xacro)
@@ -20,5 +20,5 @@
         <parent link="ra_flange"/>
         <child link="rh_forearm"/>
-        <origin xyz="0.012 0.0 0.0" rpy="${pi/2.0} ${0.0} ${pi/2.0}"/>
+        <origin xyz="0.012 0.0 0.0" rpy="${pi/2.0} ${pi} ${pi/2.0}"/>
     </joint>
 </robot>
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