Commit message: Parametrized xacro arm side and ur model

File: sr_multi_description/urdf/sr_ur.urdf.xacro (robot description, xacro)
@@ -1,8 +1,15 @@
-<robot xmlns:xacro="http://ros.org/wiki/xacro" name="ursrbox">
-  <!-- Arm -->
-  <xacro:include filename="$(find ur_description)/urdf/inc/ur10e_macro.xacro"/>
-  <xacro:arg name="kinematics_config" default="$(find ur_description)/config/ur10e/default_kinematics.yaml"/>
+<robot xmlns:xacro="http://www.ros.org/wiki/xacro"
+       xmlns:sensor="http://playerstage.sourceforge.net/gazebo/xmlschema/#sensor"
+       xmlns:controller="http://playerstage.sourceforge.net/gazebo/xmlschema/#controller"
+       xmlns:interface="http://playerstage.sourceforge.net/gazebo/xmlschema/#interface" name="ursr">
+  <link name="world"/>
+  <xacro:arg name="initial_y" default="0.0"/>
+  <xacro:arg name="initial_z" default="0.0"/>
+  <xacro:arg name="initial_yaw" default="0.0"/>
   <xacro:arg name="transmission_hw_interface" default="hardware_interface/PositionJointInterface"/>
-  <xacro:ur10e_robot prefix="ra_" transmission_hw_interface="$(arg transmission_hw_interface)" kinematics_parameters_file="$(arg kinematics_config)"/>
+  <xacro:arg name="side" default="right"/>
+  <xacro:arg name="robot_model" default="ur10e"/>
+  <xacro:arg name="kinematics_config" default="$(find ur_description)/config/$(arg robot_model)/default_kinematics.yaml"/>
+  <xacro:include filename="$(find ur_description)/urdf/inc/$(arg robot_model)_macro.xacro"/>
   <gazebo>
     <plugin filename="libgazebo_ros_control.so" name="gazebo_ros_control">
@@ -10,11 +17,26 @@
     </plugin>
   </gazebo>
-  <!-- Join arm and world -->
-  <link name="world"/>
-  <xacro:arg name="initial_z" default="0.0"/>
+  <xacro:if value="${'$(arg side)' == 'right'}">
+      <xacro:arg name="arm_prefix" default="ra" />
+  </xacro:if>
+  <xacro:if value="${'$(arg side)' == 'left'}">
+      <xacro:arg name="arm_prefix" default="la" />
+  </xacro:if>
+  <xacro:if value="${'$(arg robot_model)' == 'ur10e'}">
+      <xacro:ur10e_robot prefix="$(arg arm_prefix)_" transmission_hw_interface="$(arg transmission_hw_interface)" kinematics_parameters_file="$(arg kinematics_config)"/>
+    </xacro:if>
+    <xacro:if value="${'$(arg robot_model)' == 'ur10'}">
+      <xacro:ur10_robot prefix="$(arg arm_prefix)_" transmission_hw_interface="$(arg transmission_hw_interface)" kinematics_parameters_file="$(arg kinematics_config)"/>
+    </xacro:if>
+    <xacro:if value="${'$(arg robot_model)' == 'ur5e'}">
+      <xacro:ur5e_robot prefix="$(arg arm_prefix)_" transmission_hw_interface="$(arg transmission_hw_interface)" kinematics_parameters_file="$(arg kinematics_config)"/>
+    </xacro:if>
+    <xacro:if value="${'$(arg robot_model)' == 'ur5'}">
+      <xacro:ur5_robot prefix="$(arg arm_prefix)_" transmission_hw_interface="$(arg transmission_hw_interface)" kinematics_parameters_file="$(arg kinematics_config)"/>
+  </xacro:if>
   <joint name="world_joint" type="fixed">
-      <parent link="world"/>
-      <child link="ra_base_link"/>
-      <origin xyz="0.0 0.0 $(arg initial_z)" rpy="0.0 0.0 0.0"/>
+    <parent link="world"/>
+    <child link="$(arg arm_prefix)_base_link"/>
+    <origin xyz="0.0 $(arg initial_y) $(arg initial_z)" rpy="0.0 0.0 $(arg initial_yaw)"/>
   </joint>
 </robot>
