Commit message: possibility of spawing single hand with two arms

File: sr_multi_description/urdf/bimanual_srhand_ur.urdf.xacro (robot description, xacro)
@@ -36,4 +36,5 @@
         <origin xyz="$(arg arm_x_separation) $(arg arm_y_separation) $(arg arm_2_z)" rpy="0.0 0.0 ${pi}"/>
     </joint>
+    <xacro:arg name="hands" default="both"/>
     <xacro:arg name="right_hand_type" default="hand_e"/>
     <xacro:arg name="right_hand_version" default="E3M5"/>
@@ -53,19 +54,27 @@
     <xacro:include filename="$(find sr_description)/hand/xacro/hand.urdf.xacro"/>
     <xacro:include filename="$(find sr_description)/other/xacro/gazebo.urdf.xacro"/>
-    <xacro:sr_hand side="right" hand_type="$(arg right_hand_type)" hand_version="$(arg right_hand_version)"
-                   fingers="$(arg right_fingers)" tip_sensors="$(arg right_tip_sensors)" mid_sensors="$(arg right_mid_sensors)"
-                   prox_sensors="$(arg right_prox_sensors)" palm_sensor="$(arg right_palm_sensor)"/>
-    <joint name="ra_arm_to_hand" type="fixed">
-        <parent link="ra_flange"/>
-        <child link="rh_forearm"/>
-        <origin xyz="0.012 0.0 0.0" rpy="${pi/2.0} ${pi} ${pi/2.0}"/>
-    </joint>
-    <xacro:sr_hand side="left" hand_type="$(arg left_hand_type)" hand_version="$(arg left_hand_version)"
-                fingers="$(arg left_fingers)" tip_sensors="$(arg left_tip_sensors)" mid_sensors="$(arg left_mid_sensors)"
-                prox_sensors="$(arg left_prox_sensors)" palm_sensor="$(arg left_palm_sensor)"/>
-    <joint name="la_arm_to_hand" type="fixed">
-        <parent link="la_flange"/>
-        <child link="lh_forearm"/>
-        <origin xyz="0.012 0.0 0.0" rpy="${pi/2.0} ${pi} ${pi/2.0}"/>
-    </joint>
+    <xacro:if value="${'$(arg hands)' == 'both' or '$(arg hands)' == 'right'}">
+        <xacro:sr_hand side="right" hand_type="$(arg right_hand_type)" hand_version="$(arg right_hand_version)"
+                    fingers="$(arg right_fingers)" tip_sensors="$(arg right_tip_sensors)" mid_sensors="$(arg right_mid_sensors)"
+                    prox_sensors="$(arg right_prox_sensors)" palm_sensor="$(arg right_palm_sensor)"/>
+    </xacro:if>
+    <xacro:if value="${'$(arg hands)' == 'both' or '$(arg hands)' == 'right'}">
+        <joint name="ra_arm_to_hand" type="fixed">
+            <parent link="ra_flange"/>
+            <child link="rh_forearm"/>
+            <origin xyz="0.012 0.0 0.0" rpy="${pi/2.0} ${pi} ${pi/2.0}"/>
+        </joint>
+    </xacro:if>
+    <xacro:if value="${'$(arg hands)' == 'both' or '$(arg hands)' == 'left'}">
+        <xacro:sr_hand side="left" hand_type="$(arg left_hand_type)" hand_version="$(arg left_hand_version)"
+                    fingers="$(arg left_fingers)" tip_sensors="$(arg left_tip_sensors)" mid_sensors="$(arg left_mid_sensors)"
+                    prox_sensors="$(arg left_prox_sensors)" palm_sensor="$(arg left_palm_sensor)"/>
+    </xacro:if>
+    <xacro:if value="${'$(arg hands)' == 'both' or '$(arg hands)' == 'left'}">
+        <joint name="la_arm_to_hand" type="fixed">
+            <parent link="la_flange"/>
+            <child link="lh_forearm"/>
+            <origin xyz="0.012 0.0 0.0" rpy="${pi/2.0} ${pi} ${pi/2.0}"/>
+        </joint>
+    </xacro:if>
 </robot>

Commit message: Removing box from arm without hand and bimanual system without hands (#723)
* F refactoring sr description multi (#704)

* Work in progress with refactoring

* Passing params. Still failing in str

* Hand e working with changes made by ubi

* Adding all the right args

* Refactored bimanual hand to accept the new xacro structure

* refarctoring

* parametrizing hand_ur10e

* ur10 and ur10e ready

* unimanuals ready

* bimanuals working

* lint

* unimanual launchfiules done

* bimanual done

* urdfs minimized

* unimanual cleaned up configs

* working on bimanual

* working, cleanup time

* some cleanup

* cleaning

* removing debug code

* Update sr_multi_description/urdf/bimanual_srhand_ur.urdf.xacro

Co-authored-by: Beatriz Leon <beatriz@shadowrobot.com>

* Update sr_robot_launch/launch/sr_bimanual_hardware_control_loop.launch

Co-authored-by: Beatriz Leon <beatriz@shadowrobot.com>

* Update sr_robot_launch/launch/sr_bimanual_simulation_control_loop.launch

Co-authored-by: Beatriz Leon <beatriz@shadowrobot.com>

* Update sr_robot_launch/launch/sr_bimanual_simulation_control_loop.launch

Co-authored-by: Beatriz Leon <beatriz@shadowrobot.com>

* Update sr_multi_description/urdf/bimanual_srhand_ur.urdf.xacro

Co-authored-by: Beatriz Leon <beatriz@shadowrobot.com>

* according to review

Co-authored-by: Beatriz Leon <beatriz@shadowrobot.com>

* fixing controllers spawning

* cleaning old names

* fixing contrcution of robot descrpiton

* small fix

* testing

* debugging

* debugging

* fixing for bimanual

* cleaning

* fixing flag

* fixing left arm placement

* removing redundant param

* passing args from the top

* Update args (#718)

* Update sr_ur_arm_hand.launch

* Update sr_simulation_control_loop.launch

* Fixing lint error

* dummy commit

* Created minimal launch of ur without box

* Parametrized xacro arm side and ur model

* Added ur10e autodetection

* Added all ur robot_config

* Added gazebo/gazebo.urdf.xacro

* Update right_ur10e.yaml

* added end effector on other groups to urs

* added path sr_description

* passed param hands

* pointed to new config files with only the arm

* robot model arg

* possibility of spawing single hand with two arms

* conditions left right hw launch

* add right left payload 0 when hands are none

* name changes

* reorganized payload conditions

* removed unused parameters

* layout

* layout and comment

Co-authored-by: mikramarc <michal@shadowrobot.com>
Co-authored-by: Beatriz Leon <beatriz@shadowrobot.com>
Co-authored-by: giusebar <giuseppe@shadowrobot.com>

File: sr_multi_description/urdf/bimanual_srhand_ur.urdf.xacro (robot description, xacro)
@@ -36,4 +36,5 @@
         <origin xyz="$(arg arm_x_separation) $(arg arm_y_separation) $(arg arm_2_z)" rpy="0.0 0.0 ${pi}"/>
     </joint>
+    <xacro:arg name="hands" default="both"/>
     <xacro:arg name="right_hand_type" default="hand_e"/>
     <xacro:arg name="right_hand_version" default="E3M5"/>
@@ -53,19 +54,23 @@
     <xacro:include filename="$(find sr_description)/hand/xacro/hand.urdf.xacro"/>
     <xacro:include filename="$(find sr_description)/other/xacro/gazebo.urdf.xacro"/>
-    <xacro:sr_hand side="right" hand_type="$(arg right_hand_type)" hand_version="$(arg right_hand_version)"
-                   fingers="$(arg right_fingers)" tip_sensors="$(arg right_tip_sensors)" mid_sensors="$(arg right_mid_sensors)"
-                   prox_sensors="$(arg right_prox_sensors)" palm_sensor="$(arg right_palm_sensor)"/>
-    <joint name="ra_arm_to_hand" type="fixed">
-        <parent link="ra_flange"/>
-        <child link="rh_forearm"/>
-        <origin xyz="0.012 0.0 0.0" rpy="${pi/2.0} ${pi} ${pi/2.0}"/>
-    </joint>
-    <xacro:sr_hand side="left" hand_type="$(arg left_hand_type)" hand_version="$(arg left_hand_version)"
-                fingers="$(arg left_fingers)" tip_sensors="$(arg left_tip_sensors)" mid_sensors="$(arg left_mid_sensors)"
-                prox_sensors="$(arg left_prox_sensors)" palm_sensor="$(arg left_palm_sensor)"/>
-    <joint name="la_arm_to_hand" type="fixed">
-        <parent link="la_flange"/>
-        <child link="lh_forearm"/>
-        <origin xyz="0.012 0.0 0.0" rpy="${pi/2.0} ${pi} ${pi/2.0}"/>
-    </joint>
+    <xacro:if value="${'$(arg hands)' == 'both' or '$(arg hands)' == 'right'}">
+        <xacro:sr_hand side="right" hand_type="$(arg right_hand_type)" hand_version="$(arg right_hand_version)"
+                    fingers="$(arg right_fingers)" tip_sensors="$(arg right_tip_sensors)" mid_sensors="$(arg right_mid_sensors)"
+                    prox_sensors="$(arg right_prox_sensors)" palm_sensor="$(arg right_palm_sensor)"/>
+        <joint name="ra_arm_to_hand" type="fixed">
+            <parent link="ra_flange"/>
+            <child link="rh_forearm"/>
+            <origin xyz="0.012 0.0 0.0" rpy="${pi/2.0} ${pi} ${pi/2.0}"/>
+        </joint>
+    </xacro:if>
+    <xacro:if value="${'$(arg hands)' == 'both' or '$(arg hands)' == 'left'}">
+        <xacro:sr_hand side="left" hand_type="$(arg left_hand_type)" hand_version="$(arg left_hand_version)"
+                    fingers="$(arg left_fingers)" tip_sensors="$(arg left_tip_sensors)" mid_sensors="$(arg left_mid_sensors)"
+                    prox_sensors="$(arg left_prox_sensors)" palm_sensor="$(arg left_palm_sensor)"/>
+        <joint name="la_arm_to_hand" type="fixed">
+            <parent link="la_flange"/>
+            <child link="lh_forearm"/>
+            <origin xyz="0.012 0.0 0.0" rpy="${pi/2.0} ${pi} ${pi/2.0}"/>
+        </joint>
+    </xacro:if>
 </robot>

Commit message: modified distance arm hand

File: sr_multi_description/urdf/bimanual_srhand_ur.urdf.xacro (robot description, xacro)
@@ -61,5 +61,5 @@
             <parent link="ra_flange"/>
             <child link="rh_forearm"/>
-            <origin xyz="0.012 0.0 0.0" rpy="${pi/2.0} ${pi} ${pi/2.0}"/>
+            <origin xyz="-0.012 0.0 0.0" rpy="${pi/2.0} ${pi} ${pi/2.0}"/>
         </joint>
     </xacro:if>
@@ -71,5 +71,5 @@
             <parent link="la_flange"/>
             <child link="lh_forearm"/>
-            <origin xyz="0.012 0.0 0.0" rpy="${pi/2.0} ${pi} ${pi/2.0}"/>
+            <origin xyz="-0.012 0.0 0.0" rpy="${pi/2.0} ${pi} ${pi/2.0}"/>
         </joint>
     </xacro:if>

File: sr_multi_description/urdf/srhand_two_ur.urdf.xacro (robot description, xacro)
@@ -57,5 +57,5 @@
         <parent link="ra_flange"/>
         <child link="$(arg hand_prefix)_forearm"/>
-        <origin xyz="0.012 0.0 0.0" rpy="${pi/2.0} ${pi} ${pi/2.0}"/>
+        <origin xyz="-0.012 0.0 0.0" rpy="${pi/2.0} ${pi} ${pi/2.0}"/>
     </joint>
 </robot>

File: sr_multi_description/urdf/srhand_ur.urdf.xacro (robot description, xacro)
@@ -53,5 +53,5 @@
         <parent link="$(arg arm_prefix)_flange"/>
         <child link="$(arg hand_prefix)_forearm"/>
-        <origin xyz="0.012 0.0 0.0" rpy="${pi/2.0} ${pi} ${pi/2.0}"/>
+        <origin xyz="-0.012 0.0 0.0" rpy="${pi/2.0} ${pi} ${pi/2.0}"/>
     </joint>
 </robot>

Commit message: removed 0.012 distance

File: sr_multi_description/urdf/bimanual_srhand_ur.urdf.xacro (robot description, xacro)
@@ -61,5 +61,5 @@
             <parent link="ra_flange"/>
             <child link="rh_forearm"/>
-            <origin xyz="-0.012 0.0 0.0" rpy="${pi/2.0} ${pi} ${pi/2.0}"/>
+            <origin xyz="0.0 0.0 0.0" rpy="${pi/2.0} ${pi} ${pi/2.0}"/>
         </joint>
     </xacro:if>
@@ -71,5 +71,5 @@
             <parent link="la_flange"/>
             <child link="lh_forearm"/>
-            <origin xyz="-0.012 0.0 0.0" rpy="${pi/2.0} ${pi} ${pi/2.0}"/>
+            <origin xyz="0.0 0.0 0.0" rpy="${pi/2.0} ${pi} ${pi/2.0}"/>
         </joint>
     </xacro:if>

File: sr_multi_description/urdf/srhand_two_ur.urdf.xacro (robot description, xacro)
@@ -57,5 +57,5 @@
         <parent link="ra_flange"/>
         <child link="$(arg hand_prefix)_forearm"/>
-        <origin xyz="-0.012 0.0 0.0" rpy="${pi/2.0} ${pi} ${pi/2.0}"/>
+        <origin xyz="0.0 0.0 0.0" rpy="${pi/2.0} ${pi} ${pi/2.0}"/>
     </joint>
 </robot>

Commit message: Added arguments for mounting plates and removed 0.012 distance (#732)
* added mounting plate

* avoid fail when no arms

* modified distance arm hand

* Changing arms by mounting plate

* Changing coordinates

* Changing coordinates

* Removing hand lite condition not needed

* Update sr_simulation_control_loop.launch

* removed 0.012 distance

Co-authored-by: Beatriz Leon <beatriz@shadowrobot.com>
Co-authored-by: Fotios Papadopoulos <fotios@shadowrobot.com>

File: sr_multi_description/urdf/bimanual_srhand_ur.urdf.xacro (robot description, xacro)
@@ -56,20 +56,20 @@
     <xacro:if value="${'$(arg hands)' == 'both' or '$(arg hands)' == 'right'}">
         <xacro:sr_hand side="right" hand_type="$(arg right_hand_type)" hand_version="$(arg right_hand_version)"
-                    fingers="$(arg right_fingers)" tip_sensors="$(arg right_tip_sensors)" mid_sensors="$(arg right_mid_sensors)"
-                    prox_sensors="$(arg right_prox_sensors)" palm_sensor="$(arg right_palm_sensor)"/>
+            fingers="$(arg right_fingers)" tip_sensors="$(arg right_tip_sensors)" mid_sensors="$(arg right_mid_sensors)"
+            prox_sensors="$(arg right_prox_sensors)" palm_sensor="$(arg right_palm_sensor)" mounting_plate="true"/>
         <joint name="ra_arm_to_hand" type="fixed">
             <parent link="ra_flange"/>
             <child link="rh_forearm"/>
-            <origin xyz="0.012 0.0 0.0" rpy="${pi/2.0} ${pi} ${pi/2.0}"/>
+            <origin xyz="0.0 0.0 0.0" rpy="${pi/2.0} ${pi} ${pi/2.0}"/>
         </joint>
     </xacro:if>
     <xacro:if value="${'$(arg hands)' == 'both' or '$(arg hands)' == 'left'}">
         <xacro:sr_hand side="left" hand_type="$(arg left_hand_type)" hand_version="$(arg left_hand_version)"
-                    fingers="$(arg left_fingers)" tip_sensors="$(arg left_tip_sensors)" mid_sensors="$(arg left_mid_sensors)"
-                    prox_sensors="$(arg left_prox_sensors)" palm_sensor="$(arg left_palm_sensor)"/>
+            fingers="$(arg left_fingers)" tip_sensors="$(arg left_tip_sensors)" mid_sensors="$(arg left_mid_sensors)"
+            prox_sensors="$(arg left_prox_sensors)" palm_sensor="$(arg left_palm_sensor)" mounting_plate="true"/>
         <joint name="la_arm_to_hand" type="fixed">
             <parent link="la_flange"/>
             <child link="lh_forearm"/>
-            <origin xyz="0.012 0.0 0.0" rpy="${pi/2.0} ${pi} ${pi/2.0}"/>
+            <origin xyz="0.0 0.0 0.0" rpy="${pi/2.0} ${pi} ${pi/2.0}"/>
         </joint>
     </xacro:if>

File: sr_multi_description/urdf/srhand_two_ur.urdf.xacro (robot description, xacro)
@@ -57,5 +57,5 @@
         <parent link="ra_flange"/>
         <child link="$(arg hand_prefix)_forearm"/>
-        <origin xyz="0.012 0.0 0.0" rpy="${pi/2.0} ${pi} ${pi/2.0}"/>
+        <origin xyz="0.0 0.0 0.0" rpy="${pi/2.0} ${pi} ${pi/2.0}"/>
     </joint>
 </robot>

File: sr_multi_description/urdf/srhand_ur.urdf.xacro (robot description, xacro)
@@ -44,5 +44,5 @@
     <xacro:sr_hand side="$(arg side)" hand_type="$(arg hand_type)" hand_version="$(arg hand_version)"
                    fingers="$(arg fingers)" tip_sensors="$(arg tip_sensors)" mid_sensors="$(arg mid_sensors)"
-                   prox_sensors="$(arg prox_sensors)" palm_sensor="$(arg palm_sensor)"/>
+                   prox_sensors="$(arg prox_sensors)" palm_sensor="$(arg palm_sensor)" mounting_plate="true"/>
     <joint name="world_joint" type="fixed">
         <parent link="world"/>
@@ -53,5 +53,5 @@
         <parent link="$(arg arm_prefix)_flange"/>
         <child link="$(arg hand_prefix)_forearm"/>
-        <origin xyz="0.012 0.0 0.0" rpy="${pi/2.0} ${pi} ${pi/2.0}"/>
+        <origin xyz="0.0 0.0 0.0" rpy="${pi/2.0} ${pi} ${pi/2.0}"/>
     </joint>
 </robot>
