Commit message: fixing left arm placement

File: sr_multi_description/urdf/srhand_ur.urdf.xacro (robot description, xacro)
@@ -4,5 +4,7 @@
        xmlns:interface="http://playerstage.sourceforge.net/gazebo/xmlschema/#interface" name="ursrh">
     <link name="world"/>
+    <xacro:arg name="initial_y" default="0.0"/>
     <xacro:arg name="initial_z" default="0.0"/>
+    <xacro:arg name="initial_yaw" default="0.0"/>
     <xacro:arg name="transmission_hw_interface" default="hardware_interface/PositionJointInterface"/>
     <xacro:arg name="robot_model" default="ur10e"/>
@@ -46,5 +48,5 @@
         <parent link="world"/>
         <child link="$(arg arm_prefix)_base_link"/>
-        <origin xyz="0.0 0.0 $(arg initial_z)" rpy="0.0 0.0 0.0"/>
+        <origin xyz="0.0 $(arg initial_y) $(arg initial_z)" rpy="0.0 0.0 $(arg initial_yaw)"/>
     </joint>
     <joint name="$(arg arm_prefix)_arm_to_hand" type="fixed">

Commit message: Changing coordinates

File: sr_multi_description/urdf/srhand_ur.urdf.xacro (robot description, xacro)
@@ -53,5 +53,5 @@
         <parent link="$(arg arm_prefix)_flange"/>
         <child link="$(arg hand_prefix)_forearm"/>
-        <origin xyz="-0.012 0.0 0.0" rpy="${pi/2.0} ${pi} ${pi/2.0}"/>
+        <origin xyz="0.012 0.0 0.0" rpy="${pi/2.0} ${pi} ${pi/2.0}"/>
     </joint>
 </robot>

Commit message: Changing coordinates

File: sr_multi_description/urdf/srhand_ur.urdf.xacro (robot description, xacro)
@@ -53,5 +53,5 @@
         <parent link="$(arg arm_prefix)_flange"/>
         <child link="$(arg hand_prefix)_forearm"/>
-        <origin xyz="0.012 0.0 0.0" rpy="${pi/2.0} ${pi} ${pi/2.0}"/>
+        <origin xyz="0.0 0.0 0.0" rpy="${pi/2.0} ${pi} ${pi/2.0}"/>
     </joint>
 </robot>

Commit message: Add a LAXONE FT sensor to the unimanual hand+ur robot xacro

File: sr_multi_description/urdf/srhand_ur.urdf.xacro (robot description, xacro)
@@ -74,8 +74,16 @@
         <origin xyz="0.0 $(arg initial_y) $(arg initial_z)" rpy="0.0 0.0 $(arg initial_yaw)"/>
     </joint>
-    <joint name="$(arg arm_prefix)_arm_to_hand" type="fixed">
-        <parent link="$(arg arm_prefix)_flange"/>
-        <child link="$(arg hand_prefix)_forearm"/>
+    <xacro:arg name="ft_sensor_prefix" default="ft_sensor0"/>
+    <xacro:include filename="$(find rokubimini_description)/urdf/BFT_LAXS_ECAT_M8.urdf.xacro" />
+    <xacro:BFT_LAXS_ECAT_M8 prefix="$(arg ft_sensor_prefix)" />
+    <joint name="$(arg arm_prefix)_arm_to_ft_sensor" type="fixed">
+        <parent link="$(arg arm_prefix)_flange" />
+        <child link = "$(arg ft_sensor_prefix)_mounting" />
         <origin xyz="0.0 0.0 0.0" rpy="${pi/2.0} ${pi} ${pi/2.0}"/>
     </joint>
+    <joint name="$(arg side)_ft_sensor_to_hand" type="fixed">
+        <parent link="$(arg ft_sensor_prefix)_wrench"/>
+        <child link="$(arg hand_prefix)_forearm"/>
+        <origin xyz="0.0 0.0 0.0" rpy="0.0 0.0 0.0"/>
+    </joint>
 </robot>

Commit message: fix rotations

File: sr_multi_description/urdf/srhand_ur.urdf.xacro (robot description, xacro)
@@ -80,10 +80,10 @@
         <parent link="$(arg arm_prefix)_flange" />
         <child link = "$(arg ft_sensor_prefix)_mounting" />
-        <origin xyz="0.0 0.0 0.0" rpy="${pi/2.0} ${pi} ${pi/2.0}"/>
+        <origin xyz="0.0 0.0 0.0" rpy="${pi/2.0} ${pi/2.0} ${pi/2.0}"/>
     </joint>
     <joint name="$(arg side)_ft_sensor_to_hand" type="fixed">
         <parent link="$(arg ft_sensor_prefix)_wrench"/>
         <child link="$(arg hand_prefix)_forearm"/>
-        <origin xyz="0.0 0.0 0.0" rpy="0.0 0.0 0.0"/>
+        <origin xyz="0.0 0.0 0.0" rpy="0.0 0.0 -${pi/2.0}"/>
     </joint>
 </robot>
