Commit message: First complete version. need testing

File: sr_multi_moveit/sr_box_ur10_moveit_config/config/ur10_with_box.urdf.xacro (robot description, xacro)
@@ -3,7 +3,12 @@
   <xacro:include filename="$(find ur_description)/urdf/ur10.urdf.xacro"/>
   <xacro:ur10_robot prefix="ra_" joint_limited="false"/>
-  <gazebo>
+  <!--gazebo>
     <plugin name="ros_control" filename="libgazebo_ros_control.so">
       <robotSimType>gazebo_ros_control/DefaultRobotHWSim</robotSimType>
+    </plugin>
+  </gazebo-->
+  <gazebo>
+    <plugin filename="libgazebo_ros_control.so" name="gazebo_ros_control">
+      <robotSimType>sr_gazebo_sim/SrGazeboHWSim</robotSimType>
     </plugin>
   </gazebo>
@@ -20,5 +25,5 @@
   <xacro:hand_box name="hand_box" width="0.22" depth="0.17" height="0.24"/>
   <!-- Join arm and hand -->
-  <joint name="ra_arm_to_hand1" type="fixed">
+  <joint name="ra_arm_to_hand" type="fixed">
     <parent link="ra_ee_link"/>
     <child link="hand_base_attach"/>
