Commit message: updating arm_box and srdfs

File: sr_multi_moveit/sr_box_ur10_moveit_config/config/la_ur10_with_box.urdf.xacro (robot description, xacro)
@@ -1,8 +1,8 @@
 <robot xmlns:xacro="http://ros.org/wiki/xacro" name="ursrbox">
   <!-- Arm -->
-  <xacro:include filename="$(find ur_description)/urdf/ur10.urdf.xacro"/>
-  <xacro:arg name="kinematics_config" default="$(find ur_description)/config/ur10_default.yaml"/>
+  <xacro:include filename="$(find ur_description)/urdf/inc/ur10_macro.xacro"/>
+  <xacro:arg name="kinematics_config" default="$(find ur_description)/config/ur10/default_kinematics.yaml"/>
   <xacro:arg name="transmission_hw_interface" default="hardware_interface/PositionJointInterface"/>
-  <xacro:ur10_robot prefix="la_" joint_limited="false" transmission_hw_interface="$(arg transmission_hw_interface)" kinematics_file="${load_yaml('$(arg kinematics_config)')}"/>
+  <xacro:ur10_robot prefix="la_" transmission_hw_interface="$(arg transmission_hw_interface)" kinematics_parameters_file="$(arg kinematics_config)"/>
   <gazebo>
     <plugin filename="libgazebo_ros_control.so" name="gazebo_ros_control">
@@ -23,5 +23,5 @@
   <!-- Join arm and hand -->
   <joint name="la_arm_to_hand" type="fixed">
-    <parent link="la_ee_link"/>
+    <parent link="la_flange"/>
     <child link="hand_base_attach"/>
     <origin rpy="1.570796325 3.14159265 1.570796325" xyz="0.012 0.0 0.0"/>

File: sr_multi_moveit/sr_box_ur10_moveit_config/config/la_ur10e_with_box.urdf.xacro (robot description, xacro)
@@ -1,8 +1,8 @@
 <robot xmlns:xacro="http://ros.org/wiki/xacro" name="ursrbox">
   <!-- Arm -->
-  <xacro:include filename="$(find ur_e_description)/urdf/ur10e.urdf.xacro"/>
-  <xacro:arg name="kinematics_config" default="$(find ur_e_description)/config/ur10e_default.yaml"/>
+  <xacro:include filename="$(find ur_description)/urdf/inc/ur10e_macro.xacro"/>
+  <xacro:arg name="kinematics_config" default="$(find ur_description)/config/ur10e/default_kinematics.yaml"/>
   <xacro:arg name="transmission_hw_interface" default="hardware_interface/PositionJointInterface"/>
-  <xacro:ur10e_robot prefix="la_" joint_limited="false" transmission_hw_interface="$(arg transmission_hw_interface)" kinematics_file="${load_yaml('$(arg kinematics_config)')}"/>
+  <xacro:ur10e_robot prefix="la_" transmission_hw_interface="$(arg transmission_hw_interface)" kinematics_parameters_file="$(arg kinematics_config)"/>
   <gazebo>
     <plugin filename="libgazebo_ros_control.so" name="gazebo_ros_control">
@@ -23,5 +23,5 @@
   <!-- Join arm and hand -->
   <joint name="la_arm_to_hand" type="fixed">
-    <parent link="la_ee_link"/>
+    <parent link="la_flange"/>
     <child link="hand_base_attach"/>
     <origin rpy="1.570796325 3.14159265 1.570796325" xyz="0.012 0.0 0.0"/>

File: sr_multi_moveit/sr_box_ur10_moveit_config/config/la_ur3_with_box.urdf.xacro (robot description, xacro)
@@ -1,6 +1,6 @@
 <robot xmlns:xacro="http://ros.org/wiki/xacro" name="ursrbox">
   <!-- Arm -->
-  <xacro:include filename="$(find ur_description)/urdf/ur3.urdf.xacro"/>
-  <xacro:ur3_robot prefix="la_" joint_limited="false"/>
+  <xacro:include filename="$(find ur_description)/urdf/inc/ur3_macro.xacro"/>
+  <xacro:ur3_robot prefix="la_"/>
   <gazebo>
     <plugin filename="libgazebo_ros_control.so" name="gazebo_ros_control">
@@ -21,5 +21,5 @@
   <!-- Join arm and hand -->
   <joint name="la_arm_to_hand" type="fixed">
-    <parent link="la_ee_link"/>
+    <parent link="la_flange"/>
     <child link="hand_base_attach"/>
     <origin rpy="1.570796325 3.14159265 1.570796325" xyz="0.012 0.0 0.0"/>

File: sr_multi_moveit/sr_box_ur10_moveit_config/config/la_ur5_with_box.urdf.xacro (robot description, xacro)
@@ -1,6 +1,6 @@
 <robot xmlns:xacro="http://ros.org/wiki/xacro" name="ursrbox">
   <!-- Arm -->
-  <xacro:include filename="$(find ur_description)/urdf/ur5.urdf.xacro"/>
-  <xacro:ur5_robot prefix="la_" joint_limited="false"/>
+  <xacro:include filename="$(find ur_description)/urdf/inc/ur5_macro.xacro"/>
+  <xacro:ur5_robot prefix="la_"/>
   <gazebo>
     <plugin filename="libgazebo_ros_control.so" name="gazebo_ros_control">
@@ -21,5 +21,5 @@
   <!-- Join arm and hand -->
   <joint name="la_arm_to_hand" type="fixed">
-    <parent link="la_ee_link"/>
+    <parent link="la_flange"/>
     <child link="hand_base_attach"/>
     <origin rpy="1.570796325 3.14159265 1.570796325" xyz="0.012 0.0 0.0"/>

File: sr_multi_moveit/sr_box_ur10_moveit_config/config/ra_ur10_with_box.urdf.xacro (robot description, xacro)
@@ -1,8 +1,8 @@
 <robot xmlns:xacro="http://ros.org/wiki/xacro" name="ursrbox">
   <!-- Arm -->
-  <xacro:include filename="$(find ur_description)/urdf/ur10.urdf.xacro"/>
-  <xacro:arg name="kinematics_config" default="$(find ur_description)/config/ur10_default.yaml"/>
+  <xacro:include filename="$(find ur_description)/urdf/inc/ur10_macro.xacro"/>
+  <xacro:arg name="kinematics_config" default="$(find ur_description)/config/ur10/default_kinematics.yaml"/>
   <xacro:arg name="transmission_hw_interface" default="hardware_interface/PositionJointInterface"/>
-  <xacro:ur10_robot prefix="ra_" joint_limited="false" transmission_hw_interface="$(arg transmission_hw_interface)" kinematics_file="${load_yaml('$(arg kinematics_config)')}"/>
+  <xacro:ur10_robot prefix="ra_" transmission_hw_interface="$(arg transmission_hw_interface)" kinematics_parameters_file="$(arg kinematics_config)"/>
   <gazebo>
     <plugin filename="libgazebo_ros_control.so" name="gazebo_ros_control">
@@ -23,5 +23,5 @@
   <!-- Join arm and hand -->
   <joint name="ra_arm_to_hand" type="fixed">
-    <parent link="ra_ee_link"/>
+    <parent link="ra_flange"/>
     <child link="hand_base_attach"/>
     <origin rpy="1.570796325 3.14159265 1.570796325" xyz="0.012 0.0 0.0"/>

File: sr_multi_moveit/sr_box_ur10_moveit_config/config/ra_ur10e_with_box.urdf.xacro (robot description, xacro)
@@ -1,8 +1,8 @@
 <robot xmlns:xacro="http://ros.org/wiki/xacro" name="ursrbox">
   <!-- Arm -->
-  <xacro:include filename="$(find ur_e_description)/urdf/ur10e.urdf.xacro"/>
-  <xacro:arg name="kinematics_config" default="$(find ur_e_description)/config/ur10e_default.yaml"/>
+  <xacro:include filename="$(find ur_description)/urdf/inc/ur10e_macro.xacro"/>
+  <xacro:arg name="kinematics_config" default="$(find ur_description)/config/ur10e/default_kinematics.yaml"/>
   <xacro:arg name="transmission_hw_interface" default="hardware_interface/PositionJointInterface"/>
-  <xacro:ur10e_robot prefix="ra_" joint_limited="false" transmission_hw_interface="$(arg transmission_hw_interface)" kinematics_file="${load_yaml('$(arg kinematics_config)')}"/>
+  <xacro:ur10e_robot prefix="ra_" transmission_hw_interface="$(arg transmission_hw_interface)" kinematics_parameters_file="$(arg kinematics_config)"/>
   <gazebo>
     <plugin filename="libgazebo_ros_control.so" name="gazebo_ros_control">
@@ -23,5 +23,5 @@
   <!-- Join arm and hand -->
   <joint name="ra_arm_to_hand" type="fixed">
-    <parent link="ra_ee_link"/>
+    <parent link="ra_flange"/>
     <child link="hand_base_attach"/>
     <origin rpy="1.570796325 3.14159265 1.570796325" xyz="0.012 0.0 0.0"/>

File: sr_multi_moveit/sr_box_ur10_moveit_config/config/ra_ur3_with_box.urdf.xacro (robot description, xacro)
@@ -1,8 +1,8 @@
 <robot xmlns:xacro="http://ros.org/wiki/xacro" name="ursrbox">
   <!-- Arm -->
-  <xacro:include filename="$(find ur_description)/urdf/ur3.urdf.xacro"/>
-  <xacro:arg name="kinematics_config" default="$(find ur_description)/config/ur3_default.yaml"/>
+  <xacro:include filename="$(find ur_description)/urdf/inc/ur3_macro.xacro"/>
+  <xacro:arg name="kinematics_config" default="$(find ur_description)/config/ur3/default_kinematics.yaml"/>
   <xacro:arg name="transmission_hw_interface" default="hardware_interface/PositionJointInterface"/>
-  <xacro:ur3_robot prefix="ra_" joint_limited="false" transmission_hw_interface="$(arg transmission_hw_interface)" kinematics_file="${load_yaml('$(arg kinematics_config)')}"/>
+  <xacro:ur3_robot prefix="la_" transmission_hw_interface="$(arg transmission_hw_interface)" kinematics_parameters_file="$(arg kinematics_config)"/>
   <gazebo>
     <plugin filename="libgazebo_ros_control.so" name="gazebo_ros_control">
@@ -23,5 +23,5 @@
   <!-- Join arm and hand -->
   <joint name="ra_arm_to_hand" type="fixed">
-    <parent link="ra_ee_link"/>
+    <parent link="ra_flange"/>
     <child link="hand_base_attach"/>
     <origin rpy="1.570796325 3.14159265 1.570796325" xyz="0.012 0.0 0.0"/>

File: sr_multi_moveit/sr_box_ur10_moveit_config/config/ra_ur5_with_box.urdf.xacro (robot description, xacro)
@@ -1,8 +1,8 @@
 <robot xmlns:xacro="http://ros.org/wiki/xacro" name="ursrbox">
   <!-- Arm -->
-  <xacro:include filename="$(find ur_description)/urdf/ur5.urdf.xacro"/>
-  <xacro:arg name="kinematics_config" default="$(find ur_description)/config/ur5_default.yaml"/>
+  <xacro:include filename="$(find ur_description)/urdf/inc/ur5_macro.xacro"/>
+  <xacro:arg name="kinematics_config" default="$(find ur_description)/config/ur5/default_kinematics.yaml"/>
   <xacro:arg name="transmission_hw_interface" default="hardware_interface/PositionJointInterface"/>
-  <xacro:ur5_robot prefix="ra_" joint_limited="false" transmission_hw_interface="$(arg transmission_hw_interface)" kinematics_file="${load_yaml('$(arg kinematics_config)')}"/>
+  <xacro:urr_robot prefix="ra_" transmission_hw_interface="$(arg transmission_hw_interface)" kinematics_parameters_file="$(arg kinematics_config)"/>
   <gazebo>
     <plugin filename="libgazebo_ros_control.so" name="gazebo_ros_control">
@@ -23,5 +23,5 @@
   <!-- Join arm and hand -->
   <joint name="ra_arm_to_hand" type="fixed">
-    <parent link="ra_ee_link"/>
+    <parent link="ra_flange"/>
     <child link="hand_base_attach"/>
     <origin rpy="1.570796325 3.14159265 1.570796325" xyz="0.012 0.0 0.0"/>

File: sr_multi_moveit/sr_box_ur10_moveit_config/config/ra_ur5e_with_box.urdf.xacro (robot description, xacro)
@@ -1,8 +1,8 @@
 <robot xmlns:xacro="http://ros.org/wiki/xacro" name="ursrbox">
   <!-- Arm -->
-  <xacro:include filename="$(find ur_e_description)/urdf/ur5e.urdf.xacro"/>
-  <xacro:arg name="kinematics_config" default="$(find ur_e_description)/config/ur5e_default.yaml"/>
+  <xacro:include filename="$(find ur_description)/urdf/inc/ur5e_macro.xacro"/>
+  <xacro:arg name="kinematics_config" default="$(find ur_description)/config/ur5e/default_kinematics.yaml"/>
   <xacro:arg name="transmission_hw_interface" default="hardware_interface/PositionJointInterface"/>
-  <xacro:ur5e_robot prefix="ra_" joint_limited="false" transmission_hw_interface="$(arg transmission_hw_interface)" kinematics_file="${load_yaml('$(arg kinematics_config)')}"/>
+  <xacro:ur5e_robot prefix="la_" transmission_hw_interface="$(arg transmission_hw_interface)" kinematics_parameters_file="$(arg kinematics_config)"/>
   <gazebo>
     <plugin filename="libgazebo_ros_control.so" name="gazebo_ros_control">
@@ -23,5 +23,5 @@
   <!-- Join arm and hand -->
   <joint name="ra_arm_to_hand" type="fixed">
-    <parent link="ra_ee_link"/>
+    <parent link="ra_flange"/>
     <child link="hand_base_attach"/>
     <origin rpy="1.570796325 3.14159265 1.570796325" xyz="0.012 0.0 0.0"/>
