Commit message: Removed distal and middle params used for old biotacs

File: sr_moveit_hand_config/config/shadowhand.srdf.xacro (robot description, xacro)
@@ -32,6 +32,6 @@
     <link name="${prefix}${link_prefix}knuckle" />
     <link name="${prefix}${link_prefix}proximal" />
-    <link name="${prefix}${link_prefix}${middle}" />
-    <link name="${prefix}${link_prefix}${distal}" />
+    <link name="${prefix}${link_prefix}middle" />
+    <link name="${prefix}${link_prefix}distal" />
   </xacro:macro>
   <xacro:macro name="thumbjoints" params="prefix" >
@@ -49,5 +49,5 @@
     <link name="${prefix}thhub" />
     <link name="${prefix}thmiddle" />
-    <link name="${prefix}th${distal}" />
+    <link name="${prefix}thdistal" />
   </xacro:macro>
   <!--GROUP STATES: Purpose: Define a named state for a particular group, in terms of joint values. This is useful to define states like 'folded arms'-->
@@ -103,22 +103,22 @@
   </xacro:macro>
   <xacro:macro name="finger_collisions" params="prefix link_prefix lf" >
-    <disable_collisions link1="${prefix}${link_prefix}${distal}" link2="${prefix}${link_prefix}${middle}" reason="Adjacent" />
-    <disable_collisions link1="${prefix}${link_prefix}${distal}" link2="${prefix}${link_prefix}knuckle" reason="Never" />
-    <disable_collisions link1="${prefix}${link_prefix}${distal}" link2="${prefix}${link_prefix}proximal" reason="Never" />
-    <disable_collisions link1="${prefix}${link_prefix}${distal}" link2="${prefix}forearm" reason="Never" />
-    <disable_collisions link1="${prefix}${link_prefix}${distal}" link2="${prefix}palm" reason="Never" />
+    <disable_collisions link1="${prefix}${link_prefix}distal" link2="${prefix}${link_prefix}middle" reason="Adjacent" />
+    <disable_collisions link1="${prefix}${link_prefix}distal" link2="${prefix}${link_prefix}knuckle" reason="Never" />
+    <disable_collisions link1="${prefix}${link_prefix}distal" link2="${prefix}${link_prefix}proximal" reason="Never" />
+    <disable_collisions link1="${prefix}${link_prefix}distal" link2="${prefix}forearm" reason="Never" />
+    <disable_collisions link1="${prefix}${link_prefix}distal" link2="${prefix}palm" reason="Never" />
     <xacro:unless value="$(arg is_lite)">
-      <disable_collisions link1="${prefix}${link_prefix}${distal}" link2="${prefix}wrist" reason="Never" />
+      <disable_collisions link1="${prefix}${link_prefix}distal" link2="${prefix}wrist" reason="Never" />
       <disable_collisions link1="${prefix}${link_prefix}knuckle" link2="${prefix}wrist" reason="Never" />
       <disable_collisions link1="${prefix}${link_prefix}proximal" link2="${prefix}wrist" reason="Never" />
-      <disable_collisions link1="${prefix}${link_prefix}${middle}" link2="${prefix}wrist" reason="Never" />
+      <disable_collisions link1="${prefix}${link_prefix}middle" link2="${prefix}wrist" reason="Never" />
     </xacro:unless>
     <disable_collisions link1="${prefix}${link_prefix}knuckle" link2="${prefix}${link_prefix}proximal" reason="Adjacent" />
-    <disable_collisions link1="${prefix}${link_prefix}knuckle" link2="${prefix}${link_prefix}${middle}" reason="Never" />
+    <disable_collisions link1="${prefix}${link_prefix}knuckle" link2="${prefix}${link_prefix}middle" reason="Never" />
     <disable_collisions link1="${prefix}${link_prefix}knuckle" link2="${prefix}forearm" reason="Never" />
     <disable_collisions link1="${prefix}${link_prefix}knuckle" link2="${prefix}palm" reason="Adjacent" />
-    <disable_collisions link1="${prefix}${link_prefix}${middle}" link2="${prefix}${link_prefix}proximal" reason="Adjacent" />
-    <disable_collisions link1="${prefix}${link_prefix}${middle}" link2="${prefix}forearm" reason="Never" />
-    <disable_collisions link1="${prefix}${link_prefix}${middle}" link2="${prefix}palm" reason="Never" />
+    <disable_collisions link1="${prefix}${link_prefix}middle" link2="${prefix}${link_prefix}proximal" reason="Adjacent" />
+    <disable_collisions link1="${prefix}${link_prefix}middle" link2="${prefix}forearm" reason="Never" />
+    <disable_collisions link1="${prefix}${link_prefix}middle" link2="${prefix}palm" reason="Never" />
     <disable_collisions link1="${prefix}${link_prefix}proximal" link2="${prefix}forearm" reason="Never" />
     <disable_collisions link1="${prefix}${link_prefix}proximal" link2="${prefix}palm" reason="Never" />
@@ -130,7 +130,7 @@
       </xacro:unless>
       <disable_collisions link1="${prefix}lfmetacarpal" link2="${prefix}palm" reason="Adjacent" />
-      <disable_collisions link1="${prefix}lfmetacarpal" link2="${prefix}lf${middle}" reason="Never" />
+      <disable_collisions link1="${prefix}lfmetacarpal" link2="${prefix}lfmiddle" reason="Never" />
       <disable_collisions link1="${prefix}lfmetacarpal" link2="${prefix}lfproximal" reason="Never" />
-      <disable_collisions link1="${prefix}lf${distal}" link2="${prefix}lfmetacarpal" reason="Never" />
+      <disable_collisions link1="${prefix}lfdistal" link2="${prefix}lfmetacarpal" reason="Never" />
       <disable_collisions link1="${prefix}lfknuckle" link2="${prefix}lfmetacarpal" reason="Adjacent" />
     </xacro:if>
@@ -138,5 +138,5 @@
   <xacro:macro name="thumb_collisions" params="prefix" >
     <disable_collisions link1="${prefix}forearm" link2="${prefix}thbase" reason="Never" />
-    <disable_collisions link1="${prefix}forearm" link2="${prefix}th${distal}" reason="Never" />
+    <disable_collisions link1="${prefix}forearm" link2="${prefix}thdistal" reason="Never" />
     <disable_collisions link1="${prefix}forearm" link2="${prefix}thhub" reason="Never" />
     <disable_collisions link1="${prefix}forearm" link2="${prefix}thmiddle" reason="Never" />
@@ -150,13 +150,13 @@
       <disable_collisions link1="${prefix}thhub" link2="${prefix}wrist" reason="Never" />
       <disable_collisions link1="${prefix}thbase" link2="${prefix}wrist" reason="Never" />
-      <disable_collisions link1="${prefix}th${distal}" link2="${prefix}wrist" reason="Never" />
-    </xacro:unless>
-    <disable_collisions link1="${prefix}thbase" link2="${prefix}th${distal}" reason="Never" />
+      <disable_collisions link1="${prefix}thdistal" link2="${prefix}wrist" reason="Never" />
+    </xacro:unless>
+    <disable_collisions link1="${prefix}thbase" link2="${prefix}thdistal" reason="Never" />
     <disable_collisions link1="${prefix}thbase" link2="${prefix}thhub" reason="Never" />
     <disable_collisions link1="${prefix}thbase" link2="${prefix}thmiddle" reason="Never" />
     <disable_collisions link1="${prefix}thbase" link2="${prefix}thproximal" reason="Adjacent" />
-    <disable_collisions link1="${prefix}th${distal}" link2="${prefix}thhub" reason="Never" />
-    <disable_collisions link1="${prefix}th${distal}" link2="${prefix}thmiddle" reason="Adjacent" />
-    <disable_collisions link1="${prefix}th${distal}" link2="${prefix}thproximal" reason="Never" />
+    <disable_collisions link1="${prefix}thdistal" link2="${prefix}thhub" reason="Never" />
+    <disable_collisions link1="${prefix}thdistal" link2="${prefix}thmiddle" reason="Adjacent" />
+    <disable_collisions link1="${prefix}thdistal" link2="${prefix}thproximal" reason="Never" />
     <disable_collisions link1="${prefix}thhub" link2="${prefix}thmiddle" reason="Adjacent" />
     <disable_collisions link1="${prefix}thhub" link2="${prefix}thproximal" reason="Adjacent" />
@@ -172,24 +172,24 @@
   <!-- finger to other finger with a finger in between -->
   <xacro:macro name="finger_farfinger_collisions" params="prefix link_prefix link_prefix2 lf" >
-    <disable_collisions link1="${prefix}${link_prefix}${distal}" link2="${prefix}${link_prefix2}knuckle" reason="Never" />
-    <disable_collisions link1="${prefix}${link_prefix}knuckle" link2="${prefix}${link_prefix2}${distal2}" reason="Never" />
+    <disable_collisions link1="${prefix}${link_prefix}distal" link2="${prefix}${link_prefix2}knuckle" reason="Never" />
+    <disable_collisions link1="${prefix}${link_prefix}knuckle" link2="${prefix}${link_prefix2}distal" reason="Never" />
     <disable_collisions link1="${prefix}${link_prefix}knuckle" link2="${prefix}${link_prefix2}knuckle" reason="Never" />
-    <disable_collisions link1="${prefix}${link_prefix}knuckle" link2="${prefix}${link_prefix2}${middle2}" reason="Never" />
+    <disable_collisions link1="${prefix}${link_prefix}knuckle" link2="${prefix}${link_prefix2}middle" reason="Never" />
     <disable_collisions link1="${prefix}${link_prefix}knuckle" link2="${prefix}${link_prefix2}proximal" reason="Never" />
-    <disable_collisions link1="${prefix}${link_prefix}${middle}" link2="${prefix}${link_prefix2}knuckle" reason="Never" />
+    <disable_collisions link1="${prefix}${link_prefix}middle" link2="${prefix}${link_prefix2}knuckle" reason="Never" />
     <disable_collisions link1="${prefix}${link_prefix}proximal" link2="${prefix}${link_prefix2}knuckle" reason="Never" />
     <xacro:if value="${lf}">
       <!-- Little finger special case -->
-      <disable_collisions link1="${prefix}${link_prefix}${distal}" link2="${prefix}lfmetacarpal" reason="Never" />
+      <disable_collisions link1="${prefix}${link_prefix}distal" link2="${prefix}lfmetacarpal" reason="Never" />
       <disable_collisions link1="${prefix}${link_prefix}knuckle" link2="${prefix}lfmetacarpal" reason="Never" />
-      <disable_collisions link1="${prefix}${link_prefix}${middle}" link2="${prefix}lfmetacarpal" reason="Never" />
+      <disable_collisions link1="${prefix}${link_prefix}middle" link2="${prefix}lfmetacarpal" reason="Never" />
       <disable_collisions link1="${prefix}${link_prefix}proximal" link2="${prefix}lfmetacarpal" reason="Never" />
     </xacro:if>
     <xacro:unless value="${lf}">
       <!-- Standard finger -->
-      <disable_collisions link1="${prefix}${link_prefix}${distal}" link2="${prefix}${link_prefix2}proximal" reason="Never" />
-      <disable_collisions link1="${prefix}${link_prefix}${middle}" link2="${prefix}${link_prefix2}proximal" reason="Never" />
-      <disable_collisions link1="${prefix}${link_prefix}proximal" link2="${prefix}${link_prefix2}${distal2}" reason="Never" />
-      <disable_collisions link1="${prefix}${link_prefix}proximal" link2="${prefix}${link_prefix2}${middle2}" reason="Never" />
+      <disable_collisions link1="${prefix}${link_prefix}distal" link2="${prefix}${link_prefix2}proximal" reason="Never" />
+      <disable_collisions link1="${prefix}${link_prefix}middle" link2="${prefix}${link_prefix2}proximal" reason="Never" />
+      <disable_collisions link1="${prefix}${link_prefix}proximal" link2="${prefix}${link_prefix2}distal" reason="Never" />
+      <disable_collisions link1="${prefix}${link_prefix}proximal" link2="${prefix}${link_prefix2}middle" reason="Never" />
       <disable_collisions link1="${prefix}${link_prefix}proximal" link2="${prefix}${link_prefix2}proximal" reason="Never" />
     </xacro:unless>
@@ -197,36 +197,36 @@
   <!-- finger with two fingers in between (only ff-lf) -->
   <xacro:macro name="first_little_collisions" params="prefix" >
-    <disable_collisions link1="${prefix}ff${distal}" link2="${prefix}lfknuckle" reason="Never" />
-    <disable_collisions link1="${prefix}ff${distal}" link2="${prefix}lfproximal" reason="Never" />
-    <disable_collisions link1="${prefix}ffknuckle" link2="${prefix}lf${distal2}" reason="Never" />
+    <disable_collisions link1="${prefix}ffdistal" link2="${prefix}lfknuckle" reason="Never" />
+    <disable_collisions link1="${prefix}ffdistal" link2="${prefix}lfproximal" reason="Never" />
+    <disable_collisions link1="${prefix}ffknuckle" link2="${prefix}lfdistal" reason="Never" />
     <disable_collisions link1="${prefix}ffknuckle" link2="${prefix}lfknuckle" reason="Never" />
-    <disable_collisions link1="${prefix}ffknuckle" link2="${prefix}lf${middle2}" reason="Never" />
+    <disable_collisions link1="${prefix}ffknuckle" link2="${prefix}lfmiddle" reason="Never" />
     <disable_collisions link1="${prefix}ffknuckle" link2="${prefix}lfproximal" reason="Never" />
-    <disable_collisions link1="${prefix}ff${middle}" link2="${prefix}lfknuckle" reason="Never" />
-    <disable_collisions link1="${prefix}ff${middle}" link2="${prefix}lf${middle2}" reason="Never" />
-    <disable_collisions link1="${prefix}ff${middle}" link2="${prefix}lfproximal" reason="Never" />
+    <disable_collisions link1="${prefix}ffmiddle" link2="${prefix}lfknuckle" reason="Never" />
+    <disable_collisions link1="${prefix}ffmiddle" link2="${prefix}lfmiddle" reason="Never" />
+    <disable_collisions link1="${prefix}ffmiddle" link2="${prefix}lfproximal" reason="Never" />
     <disable_collisions link1="${prefix}ffproximal" link2="${prefix}lfknuckle" reason="Never" />
-    <disable_collisions link1="${prefix}ffproximal" link2="${prefix}lf${distal2}" reason="Never" />
-    <disable_collisions link1="${prefix}ffproximal" link2="${prefix}lf${middle2}" reason="Never" />
+    <disable_collisions link1="${prefix}ffproximal" link2="${prefix}lfdistal" reason="Never" />
+    <disable_collisions link1="${prefix}ffproximal" link2="${prefix}lfmiddle" reason="Never" />
     <disable_collisions link1="${prefix}ffproximal" link2="${prefix}lfproximal" reason="Never" />
-    <disable_collisions link1="${prefix}ff${distal}" link2="${prefix}lfmetacarpal" reason="Never" />
+    <disable_collisions link1="${prefix}ffdistal" link2="${prefix}lfmetacarpal" reason="Never" />
     <disable_collisions link1="${prefix}ffknuckle" link2="${prefix}lfmetacarpal" reason="Never" />
-    <disable_collisions link1="${prefix}ff${middle}" link2="${prefix}lfmetacarpal" reason="Never" />
+    <disable_collisions link1="${prefix}ffmiddle" link2="${prefix}lfmetacarpal" reason="Never" />
     <disable_collisions link1="${prefix}ffproximal" link2="${prefix}lfmetacarpal" reason="Never" />
   </xacro:macro>
    <!-- finger next to other finger -->
    <xacro:macro name="finger_closefinger_collisions" params="prefix link_prefix link_prefix2 lf" >
-    <disable_collisions link1="${prefix}${link_prefix}${distal}" link2="${prefix}${link_prefix2}knuckle" reason="Never" />
-    <disable_collisions link1="${prefix}${link_prefix}knuckle" link2="${prefix}${link_prefix2}${distal2}" reason="Never" />
+    <disable_collisions link1="${prefix}${link_prefix}distal" link2="${prefix}${link_prefix2}knuckle" reason="Never" />
+    <disable_collisions link1="${prefix}${link_prefix}knuckle" link2="${prefix}${link_prefix2}distal" reason="Never" />
     <disable_collisions link1="${prefix}${link_prefix}knuckle" link2="${prefix}${link_prefix2}knuckle" reason="Never" />
-    <disable_collisions link1="${prefix}${link_prefix}knuckle" link2="${prefix}${link_prefix2}${middle2}" reason="Never" />
+    <disable_collisions link1="${prefix}${link_prefix}knuckle" link2="${prefix}${link_prefix2}middle" reason="Never" />
     <disable_collisions link1="${prefix}${link_prefix}knuckle" link2="${prefix}${link_prefix2}proximal" reason="Never" />
-    <disable_collisions link1="${prefix}${link_prefix}${middle}" link2="${prefix}${link_prefix2}knuckle" reason="Never" />
+    <disable_collisions link1="${prefix}${link_prefix}middle" link2="${prefix}${link_prefix2}knuckle" reason="Never" />
     <disable_collisions link1="${prefix}${link_prefix}proximal" link2="${prefix}${link_prefix2}knuckle" reason="Never" />
     <xacro:if value="${lf}">
       <!-- Little finger special case -->
-      <disable_collisions link1="${prefix}${link_prefix}${distal}" link2="${prefix}lfmetacarpal" reason="Never" />
+      <disable_collisions link1="${prefix}${link_prefix}distal" link2="${prefix}lfmetacarpal" reason="Never" />
       <disable_collisions link1="${prefix}${link_prefix}knuckle" link2="${prefix}lfmetacarpal" reason="Never" />
-      <disable_collisions link1="${prefix}${link_prefix}${middle}" link2="${prefix}lfmetacarpal" reason="Never" />
+      <disable_collisions link1="${prefix}${link_prefix}middle" link2="${prefix}lfmetacarpal" reason="Never" />
       <disable_collisions link1="${prefix}${link_prefix}proximal" link2="${prefix}lfmetacarpal" reason="Never" />
     </xacro:if>
@@ -234,16 +234,16 @@
    <!-- finger to thumb, far is 1 if at least one finger is in between -->
    <xacro:macro name="finger_thumb_collisions" params="prefix link_prefix far lf" >
-    <disable_collisions link1="${prefix}${link_prefix}${distal}" link2="${prefix}thbase" reason="Never" />
-    <disable_collisions link1="${prefix}${link_prefix}${distal}" link2="${prefix}thhub" reason="Never" />
+    <disable_collisions link1="${prefix}${link_prefix}distal" link2="${prefix}thbase" reason="Never" />
+    <disable_collisions link1="${prefix}${link_prefix}distal" link2="${prefix}thhub" reason="Never" />
     <disable_collisions link1="${prefix}${link_prefix}knuckle" link2="${prefix}thbase" reason="Never" />
-    <disable_collisions link1="${prefix}${link_prefix}knuckle" link2="${prefix}${thdistal}" reason="Never" />
+    <disable_collisions link1="${prefix}${link_prefix}knuckle" link2="${prefix}thdistal" reason="Never" />
     <disable_collisions link1="${prefix}${link_prefix}knuckle" link2="${prefix}thhub" reason="Never" />
     <disable_collisions link1="${prefix}${link_prefix}knuckle" link2="${prefix}thmiddle" reason="Never" />
     <disable_collisions link1="${prefix}${link_prefix}knuckle" link2="${prefix}thproximal" reason="Never" />
-    <disable_collisions link1="${prefix}${link_prefix}${middle}" link2="${prefix}thbase" reason="Never" />
-    <disable_collisions link1="${prefix}${link_prefix}${middle}" link2="${prefix}thhub" reason="Never" />
-    <disable_collisions link1="${prefix}${link_prefix}${middle}" link2="${prefix}thproximal" reason="Never" />
+    <disable_collisions link1="${prefix}${link_prefix}middle" link2="${prefix}thbase" reason="Never" />
+    <disable_collisions link1="${prefix}${link_prefix}middle" link2="${prefix}thhub" reason="Never" />
+    <disable_collisions link1="${prefix}${link_prefix}middle" link2="${prefix}thproximal" reason="Never" />
     <xacro:if value="${far}">
-      <disable_collisions link1="${prefix}${link_prefix}${distal}" link2="${prefix}thproximal" reason="Never" />
+      <disable_collisions link1="${prefix}${link_prefix}distal" link2="${prefix}thproximal" reason="Never" />
     </xacro:if>
     <disable_collisions link1="${prefix}${link_prefix}proximal" link2="${prefix}thbase" reason="Never" />
@@ -253,7 +253,7 @@
     <xacro:if value="${lf}">
       <!-- Little finger special case -->
-      <disable_collisions link1="${prefix}${link_prefix}${distal}" link2="${prefix}thmiddle" reason="Never" />
+      <disable_collisions link1="${prefix}${link_prefix}distal" link2="${prefix}thmiddle" reason="Never" />
       <disable_collisions link1="${prefix}lfmetacarpal" link2="${prefix}thbase" reason="Never" />
-      <disable_collisions link1="${prefix}lfmetacarpal" link2="${prefix}${thdistal}" reason="Never" />
+      <disable_collisions link1="${prefix}lfmetacarpal" link2="${prefix}thdistal" reason="Never" />
       <disable_collisions link1="${prefix}lfmetacarpal" link2="${prefix}thhub" reason="Never" />
       <disable_collisions link1="${prefix}lfmetacarpal" link2="${prefix}thmiddle" reason="Never" />

File: sr_moveit_hand_config/config/shadowhands_prefix.srdf.xacro (robot description, xacro)
@@ -13,26 +13,17 @@
   <group name="$(arg hand_name)">
     <xacro:if value="$(arg th)">
-      <xacro:property name="distal" value="distal"/>
       <xacro:thumbjoints prefix="$(arg prefix)"/>
     </xacro:if>
     <xacro:if value="$(arg ff)">
-      <xacro:property name="distal" value="distal"/>
-      <xacro:property name="middle" value="middle"/>
       <xacro:fingerjoints prefix="$(arg prefix)" joint_prefix="FF" lf="0"/>
     </xacro:if>
     <xacro:if value="$(arg mf)">
-      <xacro:property name="distal" value="distal"/>
-      <xacro:property name="middle" value="middle"/>
       <xacro:fingerjoints prefix="$(arg prefix)" joint_prefix="MF" lf="0"/>
     </xacro:if>
     <xacro:if value="$(arg rf)">
-      <xacro:property name="distal" value="distal"/>
-      <xacro:property name="middle" value="middle"/>
       <xacro:fingerjoints prefix="$(arg prefix)" joint_prefix="RF" lf="0"/>
     </xacro:if>
     <xacro:unless value="$(arg is_lite)">
       <xacro:if value="$(arg lf)">
-        <xacro:property name="distal" value="distal"/>
-        <xacro:property name="middle" value="middle"/>
         <xacro:fingerjoints prefix="$(arg prefix)" joint_prefix="LF" lf="1"/>
       </xacro:if>
@@ -263,27 +254,18 @@
   <!-- single fingers collision -->
   <xacro:if value="$(arg ff)">
-    <xacro:property name="distal" value="distal"/>
-    <xacro:property name="middle" value="middle"/>
     <xacro:finger_collisions prefix="$(arg prefix)" link_prefix="ff" lf="0" />
   </xacro:if>
   <xacro:if value="$(arg mf)">
-    <xacro:property name="distal" value="distal"/>
-    <xacro:property name="middle" value="middle"/>
     <xacro:finger_collisions prefix="$(arg prefix)" link_prefix="mf" lf="0" />
   </xacro:if>
   <xacro:if value="$(arg rf)">
-    <xacro:property name="distal" value="distal"/>
-    <xacro:property name="middle" value="middle"/>
     <xacro:finger_collisions prefix="$(arg prefix)" link_prefix="rf" lf="0" />
   </xacro:if>
   <xacro:unless value="$(arg is_lite)">
     <xacro:if value="$(arg lf)">
-      <xacro:property name="distal" value="distal"/>
-      <xacro:property name="middle" value="middle"/>
       <xacro:finger_collisions prefix="$(arg prefix)" link_prefix="lf" lf="1" />
     </xacro:if>
   </xacro:unless>
   <xacro:if value="$(arg th)">
-    <xacro:property name="distal" value="distal"/>
     <xacro:thumb_collisions prefix="$(arg prefix)" />
   </xacro:if>
@@ -292,22 +274,14 @@
     <xacro:property name="thdistal" value="thdistal"/>
     <xacro:if value="$(arg ff)">
-      <xacro:property name="distal" value="distal"/>
-      <xacro:property name="middle" value="middle"/>
       <xacro:finger_thumb_collisions  prefix="$(arg prefix)" link_prefix="ff" far="0" lf="0" />
     </xacro:if>
     <xacro:if value="$(arg mf)">
-      <xacro:property name="distal" value="distal"/>
-      <xacro:property name="middle" value="middle"/>
       <xacro:finger_thumb_collisions  prefix="$(arg prefix)" link_prefix="mf" far="1" lf="0" />
     </xacro:if>
     <xacro:if value="$(arg rf)">
-      <xacro:property name="distal" value="distal"/>
-      <xacro:property name="middle" value="middle"/>
       <xacro:finger_thumb_collisions  prefix="$(arg prefix)" link_prefix="rf" far="1" lf="0" />
     </xacro:if>
     <xacro:unless value="$(arg is_lite)">
       <xacro:if value="$(arg lf)">
-       <xacro:property name="distal" value="distal"/>
-       <xacro:property name="middle" value="middle"/>
        <xacro:finger_thumb_collisions  prefix="$(arg prefix)" link_prefix="lf" far="1" lf="1" />
       </xacro:if>

Commit message: added the thtip

File: sr_moveit_hand_config/config/shadowhand.srdf.xacro (robot description, xacro)
@@ -43,4 +43,5 @@
     <joint name="${prefix}THJ2" />
     <joint name="${prefix}THJ1" />
+ 	<joint name="${prefix}thtip" />
   </xacro:macro>
   <xacro:macro name="thumblinks" params="prefix" >
