Commit message: Fixed several issues

File: sr_moveit_hand_config/config/shadowhand.srdf.xacro (robot description, xacro)
@@ -71,4 +71,22 @@
       <joint name="${prefix}THJ4" value="0" />
       <joint name="${prefix}THJ5" value="0" />
+  </xacro:macro>
+  <xacro:macro name="finger_state_pack" params="prefix joint_prefix lf">
+      <joint name="${prefix}${joint_prefix}J1" value="0.35" />
+      <joint name="${prefix}${joint_prefix}J2" value="1.5707" />
+      <joint name="${prefix}${joint_prefix}J3" value="1.5707" />
+      <joint name="${prefix}${joint_prefix}J4" value="0" />
+      <xacro:if value="${lf}">
+       <joint name="${prefix}${joint_prefix}J5" value="0" />
+      </xacro:if>
+  </xacro:macro>
+  <xacro:macro name="thumb_state_pack" params="prefix">
+      <joint name="${prefix}THJ1" value="0.35" />
+      <joint name="${prefix}THJ2" value="0.58" />
+      <xacro:unless value="$(arg is_lite)">
+        <joint name="${prefix}THJ3" value="0" />
+      </xacro:unless>
+      <joint name="${prefix}THJ4" value="0.39" />
+      <joint name="${prefix}THJ5" value="0.19" />
   </xacro:macro>
   <xacro:macro name="finger_thumb_state_open" params="prefix finger_name joint_prefix lf is_lite">

File: sr_moveit_hand_config/config/shadowhands_prefix.srdf.xacro (robot description, xacro)
@@ -115,4 +115,25 @@
     </xacro:unless>
   </group_state>
+  <group_state name="hand_pack" group="$(arg hand_name)">
+    <xacro:if value="$(arg th)">
+        <xacro:thumb_state_pack  prefix="$(arg prefix)" />
+    </xacro:if>
+    <xacro:if value="$(arg ff)">
+        <xacro:finger_state_pack  prefix="$(arg prefix)" joint_prefix="FF" lf="0" />
+    </xacro:if>
+    <xacro:if value="$(arg mf)">
+        <xacro:finger_state_pack  prefix="$(arg prefix)" joint_prefix="MF" lf="0" />
+    </xacro:if>
+    <xacro:if value="$(arg rf)">
+        <xacro:finger_state_pack  prefix="$(arg prefix)" joint_prefix="RF" lf="0" />
+    </xacro:if>
+    <xacro:unless value="$(arg is_lite)">
+      <xacro:if value="$(arg lf)">
+          <xacro:finger_state_pack  prefix="$(arg prefix)" joint_prefix="LF" lf="1" />
+      </xacro:if>
+      <joint name="$(arg prefix)WRJ1" value="0" />
+      <joint name="$(arg prefix)WRJ2" value="0" />
+    </xacro:unless>
+  </group_state>
   <!-- single fingers state -->
   <xacro:if value="$(arg ff)">
@@ -143,4 +164,31 @@
     </group_state>
   </xacro:if>
+  <xacro:if value="$(arg ff)">
+    <group_state name="first_finger_pack" group="$(arg prefix)first_finger">
+        <xacro:finger_state_pack  prefix="$(arg prefix)" joint_prefix="FF" lf="0" />
+      </group_state>
+  </xacro:if>
+  <xacro:if value="$(arg mf)">
+    <group_state name="middle_finger_pack" group="$(arg prefix)middle_finger">
+      <xacro:finger_state_pack  prefix="$(arg prefix)" joint_prefix="MF" lf="0" />
+    </group_state>
+  </xacro:if>
+  <xacro:if value="$(arg rf)">
+    <group_state name="ring_finger_pack" group="$(arg prefix)ring_finger">
+      <xacro:finger_state_pack  prefix="$(arg prefix)" joint_prefix="RF" lf="0" />
+    </group_state>
+  </xacro:if>
+  <xacro:unless value="$(arg is_lite)">
+    <xacro:if value="$(arg lf)">
+      <group_state name="little_finger_pack" group="$(arg prefix)little_finger">
+        <xacro:finger_state_pack  prefix="$(arg prefix)" joint_prefix="LF" lf="1" />
+      </group_state>
+    </xacro:if>
+  </xacro:unless>
+  <xacro:if value="$(arg th)">
+    <group_state name="thumb_pack" group="$(arg prefix)thumb">
+        <xacro:thumb_state_pack  prefix="$(arg prefix)" />
+    </group_state>
+  </xacro:if>
   <!-- all fingers state -->
   <group_state name="fingers_open" group="$(arg prefix)fingers">
@@ -160,4 +208,23 @@
       <xacro:if value="$(arg lf)">
           <xacro:finger_state_open  prefix="$(arg prefix)" joint_prefix="LF" lf="1" />
+      </xacro:if>
+    </xacro:unless>
+  </group_state>
+  <group_state name="fingers_pack" group="$(arg prefix)fingers">
+    <xacro:if value="$(arg th)">
+        <xacro:thumb_state_pack  prefix="$(arg prefix)" />
+    </xacro:if>
+    <xacro:if value="$(arg ff)">
+        <xacro:finger_state_pack  prefix="$(arg prefix)" joint_prefix="FF" lf="0" />
+    </xacro:if>
+    <xacro:if value="$(arg mf)">
+        <xacro:finger_state_pack  prefix="$(arg prefix)" joint_prefix="MF" lf="0" />
+    </xacro:if>
+    <xacro:if value="$(arg rf)">
+        <xacro:finger_state_pack  prefix="$(arg prefix)" joint_prefix="RF" lf="0" />
+    </xacro:if>
+    <xacro:unless value="$(arg is_lite)">
+      <xacro:if value="$(arg lf)">
+          <xacro:finger_state_pack  prefix="$(arg prefix)" joint_prefix="LF" lf="1" />
       </xacro:if>
     </xacro:unless>

Commit message: Detected biotac hand and changed stored position accordingly

File: sr_moveit_hand_config/config/shadowhand.srdf.xacro (robot description, xacro)
@@ -72,6 +72,11 @@
       <joint name="${prefix}THJ5" value="0" />
   </xacro:macro>
-  <xacro:macro name="finger_state_pack" params="prefix joint_prefix lf">
+  <xacro:macro name="finger_state_pack" params="prefix joint_prefix lf is_biotac">
+  	<xacro:unless value="${is_biotac}">
+      <joint name="${prefix}${joint_prefix}J1" value="1.5707" />
+    </xacro:unless>
+    <xacro:if value="${is_biotac}">
       <joint name="${prefix}${joint_prefix}J1" value="0.35" />
+    </xacro:if>
       <joint name="${prefix}${joint_prefix}J2" value="1.5707" />
       <joint name="${prefix}${joint_prefix}J3" value="1.5707" />
@@ -81,12 +86,23 @@
       </xacro:if>
   </xacro:macro>
-  <xacro:macro name="thumb_state_pack" params="prefix">
+  <xacro:macro name="thumb_state_pack" params="prefix is_biotac">
+    <xacro:unless value="${is_biotac}">
+      <joint name="${prefix}THJ1" value="0.52" />
+      <joint name="${prefix}THJ2" value="0.61" />
+      <xacro:unless value="$(arg is_lite)">
+        <joint name="${prefix}THJ3" value="0.00" />
+      </xacro:unless>
+      <joint name="${prefix}THJ4" value="1.20" />
+      <joint name="${prefix}THJ5" value="0.22" />
+    </xacro:unless>
+    <xacro:if value="${is_biotac}">
       <joint name="${prefix}THJ1" value="0.35" />
       <joint name="${prefix}THJ2" value="0.58" />
       <xacro:unless value="$(arg is_lite)">
-        <joint name="${prefix}THJ3" value="0" />
+      <joint name="${prefix}THJ3" value="0.00" />
       </xacro:unless>
       <joint name="${prefix}THJ4" value="0.39" />
       <joint name="${prefix}THJ5" value="0.19" />
+    </xacro:if>
   </xacro:macro>
   <xacro:macro name="finger_thumb_state_open" params="prefix finger_name joint_prefix lf is_lite">

File: sr_moveit_hand_config/config/shadowhands_prefix.srdf.xacro (robot description, xacro)
@@ -9,4 +9,5 @@
   <xacro:arg name="th" default="1"/>
   <xacro:arg name="is_lite" default="0"/>
+  <xacro:arg name="is_biotac" default="0"/>
   <xacro:arg name="robot_name" default="shadowhand_motor"/>
   <xacro:arg name="hand_name" default="right_hand"/>
@@ -123,18 +124,39 @@
   <group_state name="pack" group="$(arg hand_name)">
     <xacro:if value="$(arg th)">
-        <xacro:thumb_state_pack  prefix="$(arg prefix)" />
-    </xacro:if>
-    <xacro:if value="$(arg ff)">
-        <xacro:finger_state_pack  prefix="$(arg prefix)" joint_prefix="FF" lf="0" />
-    </xacro:if>
-    <xacro:if value="$(arg mf)">
-        <xacro:finger_state_pack  prefix="$(arg prefix)" joint_prefix="MF" lf="0" />
-    </xacro:if>
-    <xacro:if value="$(arg rf)">
-        <xacro:finger_state_pack  prefix="$(arg prefix)" joint_prefix="RF" lf="0" />
-    </xacro:if>
-    <xacro:unless value="$(arg is_lite)">
-      <xacro:if value="$(arg lf)">
-          <xacro:finger_state_pack  prefix="$(arg prefix)" joint_prefix="LF" lf="1" />
+        <xacro:thumb_state_pack  prefix="$(arg prefix)" is_biotac="$(arg is_biotac)" />
+    </xacro:if>
+    <xacro:if value="$(arg ff)">
+        <xacro:finger_state_pack  prefix="$(arg prefix)" joint_prefix="FF" lf="0" is_biotac="$(arg is_biotac)"/>
+    </xacro:if>
+    <xacro:if value="$(arg mf)">
+        <xacro:finger_state_pack  prefix="$(arg prefix)" joint_prefix="MF" lf="0" is_biotac="$(arg is_biotac)"/>
+    </xacro:if>
+    <xacro:if value="$(arg rf)">
+        <xacro:finger_state_pack  prefix="$(arg prefix)" joint_prefix="RF" lf="0" is_biotac="$(arg is_biotac)"/>
+    </xacro:if>
+    <xacro:unless value="$(arg is_lite)">
+      <xacro:if value="$(arg lf)">
+          <xacro:finger_state_pack  prefix="$(arg prefix)" joint_prefix="LF" lf="1" is_biotac="$(arg is_biotac)"/>
+      </xacro:if>
+      <joint name="$(arg prefix)WRJ1" value="0" />
+      <joint name="$(arg prefix)WRJ2" value="0" />
+    </xacro:unless>
+  </group_state>
+  <group_state name="fingers_pack_thumb_open" group="$(arg hand_name)">
+    <xacro:if value="$(arg th)">
+        <xacro:thumb_state_open  prefix="$(arg prefix)" />
+    </xacro:if>
+    <xacro:if value="$(arg ff)">
+        <xacro:finger_state_pack  prefix="$(arg prefix)" joint_prefix="FF" lf="0" is_biotac="$(arg is_biotac)"/>
+    </xacro:if>
+    <xacro:if value="$(arg mf)">
+        <xacro:finger_state_pack  prefix="$(arg prefix)" joint_prefix="MF" lf="0" is_biotac="$(arg is_biotac)"/>
+    </xacro:if>
+    <xacro:if value="$(arg rf)">
+        <xacro:finger_state_pack  prefix="$(arg prefix)" joint_prefix="RF" lf="0" is_biotac="$(arg is_biotac)"/>
+    </xacro:if>
+    <xacro:unless value="$(arg is_lite)">
+      <xacro:if value="$(arg lf)">
+          <xacro:finger_state_pack  prefix="$(arg prefix)" joint_prefix="LF" lf="1" is_biotac="$(arg is_biotac)"/>
       </xacro:if>
       <joint name="$(arg prefix)WRJ1" value="0" />
@@ -172,15 +194,15 @@
   <xacro:if value="$(arg ff)">
     <group_state name="first_finger_pack" group="$(arg prefix)first_finger">
-        <xacro:finger_state_pack  prefix="$(arg prefix)" joint_prefix="FF" lf="0" />
+        <xacro:finger_state_pack  prefix="$(arg prefix)" joint_prefix="FF" lf="0" is_biotac="$(arg is_biotac)"/>
       </group_state>
   </xacro:if>
   <xacro:if value="$(arg mf)">
     <group_state name="middle_finger_pack" group="$(arg prefix)middle_finger">
-      <xacro:finger_state_pack  prefix="$(arg prefix)" joint_prefix="MF" lf="0" />
+      <xacro:finger_state_pack  prefix="$(arg prefix)" joint_prefix="MF" lf="0" is_biotac="$(arg is_biotac)"/>
     </group_state>
   </xacro:if>
   <xacro:if value="$(arg rf)">
     <group_state name="ring_finger_pack" group="$(arg prefix)ring_finger">
-      <xacro:finger_state_pack  prefix="$(arg prefix)" joint_prefix="RF" lf="0" />
+      <xacro:finger_state_pack  prefix="$(arg prefix)" joint_prefix="RF" lf="0" is_biotac="$(arg is_biotac)"/>
     </group_state>
   </xacro:if>
@@ -188,5 +210,5 @@
     <xacro:if value="$(arg lf)">
       <group_state name="little_finger_pack" group="$(arg prefix)little_finger">
-        <xacro:finger_state_pack  prefix="$(arg prefix)" joint_prefix="LF" lf="1" />
+        <xacro:finger_state_pack  prefix="$(arg prefix)" joint_prefix="LF" lf="1" is_biotac="$(arg is_biotac)"/>
       </group_state>
     </xacro:if>
@@ -194,5 +216,5 @@
   <xacro:if value="$(arg th)">
     <group_state name="thumb_pack" group="$(arg prefix)thumb">
-        <xacro:thumb_state_pack  prefix="$(arg prefix)" />
+        <xacro:thumb_state_pack  prefix="$(arg prefix)" is_biotac="$(arg is_biotac)" />
     </group_state>
   </xacro:if>
@@ -219,18 +241,37 @@
   <group_state name="fingers_pack" group="$(arg prefix)fingers">
     <xacro:if value="$(arg th)">
-        <xacro:thumb_state_pack  prefix="$(arg prefix)" />
-    </xacro:if>
-    <xacro:if value="$(arg ff)">
-        <xacro:finger_state_pack  prefix="$(arg prefix)" joint_prefix="FF" lf="0" />
-    </xacro:if>
-    <xacro:if value="$(arg mf)">
-        <xacro:finger_state_pack  prefix="$(arg prefix)" joint_prefix="MF" lf="0" />
-    </xacro:if>
-    <xacro:if value="$(arg rf)">
-        <xacro:finger_state_pack  prefix="$(arg prefix)" joint_prefix="RF" lf="0" />
-    </xacro:if>
-    <xacro:unless value="$(arg is_lite)">
-      <xacro:if value="$(arg lf)">
-          <xacro:finger_state_pack  prefix="$(arg prefix)" joint_prefix="LF" lf="1" />
+        <xacro:thumb_state_pack  prefix="$(arg prefix)" is_biotac="$(arg is_biotac)" />
+    </xacro:if>
+    <xacro:if value="$(arg ff)">
+        <xacro:finger_state_pack  prefix="$(arg prefix)" joint_prefix="FF" lf="0" is_biotac="$(arg is_biotac)"/>
+    </xacro:if>
+    <xacro:if value="$(arg mf)">
+        <xacro:finger_state_pack  prefix="$(arg prefix)" joint_prefix="MF" lf="0" is_biotac="$(arg is_biotac)"/>
+    </xacro:if>
+    <xacro:if value="$(arg rf)">
+        <xacro:finger_state_pack  prefix="$(arg prefix)" joint_prefix="RF" lf="0" is_biotac="$(arg is_biotac)"/>
+    </xacro:if>
+    <xacro:unless value="$(arg is_lite)">
+      <xacro:if value="$(arg lf)">
+          <xacro:finger_state_pack  prefix="$(arg prefix)" joint_prefix="LF" lf="1" is_biotac="$(arg is_biotac)"/>
+      </xacro:if>
+    </xacro:unless>
+  </group_state>
+  <group_state name="fingers_pack_thumb_open" group="$(arg prefix)fingers">
+    <xacro:if value="$(arg th)">
+        <xacro:thumb_state_open  prefix="$(arg prefix)" />
+    </xacro:if>
+    <xacro:if value="$(arg ff)">
+        <xacro:finger_state_pack  prefix="$(arg prefix)" joint_prefix="FF" lf="0" is_biotac="$(arg is_biotac)"/>
+    </xacro:if>
+    <xacro:if value="$(arg mf)">
+        <xacro:finger_state_pack  prefix="$(arg prefix)" joint_prefix="MF" lf="0" is_biotac="$(arg is_biotac)"/>
+    </xacro:if>
+    <xacro:if value="$(arg rf)">
+        <xacro:finger_state_pack  prefix="$(arg prefix)" joint_prefix="RF" lf="0" is_biotac="$(arg is_biotac)"/>
+    </xacro:if>
+    <xacro:unless value="$(arg is_lite)">
+      <xacro:if value="$(arg lf)">
+          <xacro:finger_state_pack  prefix="$(arg prefix)" joint_prefix="LF" lf="1" is_biotac="$(arg is_biotac)"/>
       </xacro:if>
     </xacro:unless>

Commit message: Modified thumb joints a bit. Tested with real extra lite hand

File: sr_moveit_hand_config/config/shadowhand.srdf.xacro (robot description, xacro)
@@ -94,5 +94,5 @@
       </xacro:unless>
       <joint name="${prefix}THJ4" value="1.20" />
-      <joint name="${prefix}THJ5" value="0.22" />
+      <joint name="${prefix}THJ5" value="0.30" />
     </xacro:unless>
     <xacro:if value="${is_biotac}">

Commit message: Update shadowhand.srdf.xacro

File: sr_moveit_hand_config/config/shadowhand.srdf.xacro (robot description, xacro)
@@ -94,5 +94,5 @@
       </xacro:unless>
       <joint name="${prefix}THJ4" value="1.20" />
-      <joint name="${prefix}THJ5" value="0.30" />
+      <joint name="${prefix}THJ5" value="0.22" />
     </xacro:unless>
     <xacro:if value="${is_biotac}">

Commit message: Opening the thumb a bit more to avoid collisions

File: sr_moveit_hand_config/config/shadowhand.srdf.xacro (robot description, xacro)
@@ -94,5 +94,5 @@
       </xacro:unless>
       <joint name="${prefix}THJ4" value="1.20" />
-      <joint name="${prefix}THJ5" value="0.22" />
+      <joint name="${prefix}THJ5" value="0.17" />
     </xacro:unless>
     <xacro:if value="${is_biotac}">

Commit message: updating

File: sr_moveit_hand_config/config/shadowhand.srdf.xacro (robot description, xacro)
@@ -129,5 +129,5 @@
    <!--END EFFECTOR: Purpose: Represent information about an end effector.-->
    <xacro:macro name="finger_ee" params="prefix link_prefix finger_name hand_name" >
-    <end_effector name="${prefix}${link_prefix}tip_ee" parent_link="${prefix}${link_prefix}tip" group="${prefix}${finger_name}" parent_group="${hand_name}" />
+    <end_effector name="${prefix}${link_prefix}tip_ee" parent_link="${prefix}palm" group="${prefix}${finger_name}" parent_group="${prefix}wrist" />
    </xacro:macro>
   <!--VIRTUAL JOINT: Purpose: this element defines a virtual joint between a robot link and an external frame of reference (considered fixed with respect to the robot)-->
@@ -210,4 +210,5 @@
     </xacro:unless>
     <disable_collisions link1="${prefix}forearm" link2="${prefix}palm" reason="Never" />
+    <disable_collisions link1="${prefix}palm" link2="${prefix}manipulator" reason="Never" />
   </xacro:macro>
   <!-- finger to other finger with a finger in between -->

File: sr_moveit_hand_config/config/shadowhands_prefix.srdf.xacro (robot description, xacro)
@@ -41,9 +41,14 @@
     </group>
   </xacro:unless>
+  <group name="$(arg prefix)forearm">
+    <link name="$(arg prefix)forearm" />
+  </group>
+  <group name="$(arg prefix)manipulator">
+    <chain base_link="$(arg prefix)forearm" tip_link="$(arg prefix)manipulator" />
+  </group>
   <!-- single finger groups -->
   <xacro:if value="$(arg ff)">
     <group name="$(arg prefix)first_finger">
       <xacro:fingerjoints prefix="$(arg prefix)" joint_prefix="FF" lf="0"/>
-      <chain base_link="$(arg prefix)palm" tip_link="$(arg prefix)fftip" />
     </group>
   </xacro:if>
@@ -51,5 +56,4 @@
     <group name="$(arg prefix)middle_finger">
       <xacro:fingerjoints prefix="$(arg prefix)" joint_prefix="MF" lf="0"/>
-      <chain base_link="$(arg prefix)palm" tip_link="$(arg prefix)mftip" />
     </group>
   </xacro:if>
@@ -57,5 +61,4 @@
     <group name="$(arg prefix)ring_finger">
       <xacro:fingerjoints prefix="$(arg prefix)" joint_prefix="RF" lf="0"/>
-      <chain base_link="$(arg prefix)palm" tip_link="$(arg prefix)rftip" />
     </group>
   </xacro:if>
@@ -64,5 +67,4 @@
       <group name="$(arg prefix)little_finger">
         <xacro:fingerjoints prefix="$(arg prefix)" joint_prefix="LF" lf="1"/>
-        <chain base_link="$(arg prefix)palm" tip_link="$(arg prefix)lftip" />
       </group>
     </xacro:if>
@@ -71,5 +73,4 @@
     <group name="$(arg prefix)thumb">
       <xacro:thumbjoints prefix="$(arg prefix)"/>
-      <chain base_link="$(arg prefix)palm" tip_link="$(arg prefix)thtip" />
     </group>
   </xacro:if>
@@ -297,6 +298,8 @@
   </xacro:if>
   <xacro:unless value="$(arg is_lite)">
-    <end_effector group="$(arg prefix)wrist" name="$(arg prefix)wrist_ee" parent_link="$(arg prefix)palm" parent_group="$(arg hand_name)"/>
-  </xacro:unless>
+    <end_effector group="$(arg prefix)wrist" name="$(arg prefix)wrist_ee" parent_link="$(arg prefix)forearm" parent_group="$(arg prefix)forearm"/>
+  </xacro:unless>
+  <end_effector group="$(arg prefix)fingers" name="$(arg prefix)palm_ee" parent_group="$(arg prefix)wrist" parent_link="$(arg prefix)palm"/>
+  <end_effector group="$(arg prefix)fingers" name="$(arg prefix)manipulator_ee" parent_group="$(arg prefix)manipulator" parent_link="$(arg prefix)manipulator"/>
   <!--DISABLE COLLISIONS: By default it is assumed that any link of the robot could potentially come into collision with any other link in the robot. This tag disables collision checking between a specified pair of links. -->
   <xacro:hand_collisions prefix="$(arg prefix)" />

Commit message: Fixed wrist group for hand lite

File: sr_moveit_hand_config/config/shadowhand.srdf.xacro (robot description, xacro)
@@ -127,8 +127,13 @@
     </group_state>
   </xacro:macro>
-   <!--END EFFECTOR: Purpose: Represent information about an end effector.-->
-   <xacro:macro name="finger_ee" params="prefix link_prefix finger_name hand_name" >
-    <end_effector name="${prefix}${link_prefix}tip_ee" parent_link="${prefix}palm" group="${prefix}${finger_name}" parent_group="${prefix}wrist" />
-   </xacro:macro>
+  <!--END EFFECTOR: Purpose: Represent information about an end effector.-->
+  <xacro:macro name="finger_ee" params="prefix link_prefix finger_name hand_name" >
+    <xacro:if value="$(arg is_lite)">
+      <end_effector name="${prefix}${link_prefix}tip_ee" parent_link="${prefix}palm" group="${prefix}${finger_name}" parent_group="${prefix}wrist_lite" />
+    </xacro:if>
+    <xacro:unless value="$(arg is_lite)">
+      <end_effector name="${prefix}${link_prefix}tip_ee" parent_link="${prefix}palm" group="${prefix}${finger_name}" parent_group="${prefix}wrist" />
+    </xacro:unless>
+  </xacro:macro>
   <!--VIRTUAL JOINT: Purpose: this element defines a virtual joint between a robot link and an external frame of reference (considered fixed with respect to the robot)-->
   <!--PASSIVE JOINT: Purpose: this element is used to mark joints that are not actuated-->

File: sr_moveit_hand_config/config/shadowhands_prefix.srdf.xacro (robot description, xacro)
@@ -37,8 +37,12 @@
   <xacro:unless value="$(arg is_lite)">
     <group name="$(arg prefix)wrist">
- 	  <joint name="$(arg prefix)WRJ2" />
-      <joint name="$(arg prefix)WRJ1" />
-    </group>
-  </xacro:unless>
+ 	  <chain base_link="$(arg prefix)forearm" tip_link="$(arg prefix)palm" />
+    </group>
+  </xacro:unless>
+  <xacro:if value="$(arg is_lite)">
+    <group name="$(arg prefix)wrist_lite">
+      <chain base_link="$(arg prefix)forearm" tip_link="$(arg prefix)palm" />
+    </group>
+  </xacro:if>
   <group name="$(arg prefix)forearm">
     <link name="$(arg prefix)forearm" />
@@ -299,6 +303,9 @@
   <xacro:unless value="$(arg is_lite)">
     <end_effector group="$(arg prefix)wrist" name="$(arg prefix)wrist_ee" parent_link="$(arg prefix)forearm" parent_group="$(arg prefix)forearm"/>
-  </xacro:unless>
-  <end_effector group="$(arg prefix)fingers" name="$(arg prefix)palm_ee" parent_group="$(arg prefix)wrist" parent_link="$(arg prefix)palm"/>
+    <end_effector group="$(arg prefix)fingers" name="$(arg prefix)palm_ee" parent_group="$(arg prefix)wrist" parent_link="$(arg prefix)palm"/>
+  </xacro:unless>
+  <xacro:if value="$(arg is_lite)">
+    <end_effector group="$(arg prefix)fingers" name="$(arg prefix)palm_ee" parent_group="$(arg prefix)wrist_lite" parent_link="$(arg prefix)palm"/>
+  </xacro:if>
   <end_effector group="$(arg prefix)fingers" name="$(arg prefix)manipulator_ee" parent_group="$(arg prefix)manipulator" parent_link="$(arg prefix)manipulator"/>
   <!--DISABLE COLLISIONS: By default it is assumed that any link of the robot could potentially come into collision with any other link in the robot. This tag disables collision checking between a specified pair of links. -->
