Commit message: End effectors fixed

File: sr_moveit_hand_config/config/shadowhand.srdf.xacro (robot description, xacro)
@@ -25,4 +25,7 @@
     <joint name="${prefix}${joint_prefix}tip" />
   </xacro:macro>
+  <xacro:macro name="fingerchains" params="prefix link_prefix lf">
+    <chain base_link="${prefix}palm" tip_link="${prefix}${link_prefix}tip"/>
+  </xacro:macro>
   <xacro:macro name="fingerlinks" params="prefix link_prefix lf">
     <xacro:if value="${lf}">
@@ -129,10 +132,5 @@
   <!--END EFFECTOR: Purpose: Represent information about an end effector.-->
   <xacro:macro name="finger_ee" params="prefix link_prefix finger_name hand_name" >
-    <xacro:if value="$(arg is_lite)">
-      <end_effector name="${prefix}${link_prefix}tip_ee" parent_link="${prefix}palm" group="${prefix}${finger_name}" parent_group="${prefix}wrist_lite" />
-    </xacro:if>
-    <xacro:unless value="$(arg is_lite)">
-      <end_effector name="${prefix}${link_prefix}tip_ee" parent_link="${prefix}palm" group="${prefix}${finger_name}" parent_group="${prefix}wrist" />
-    </xacro:unless>
+    <end_effector name="${prefix}${link_prefix}tip_ee" parent_link="${prefix}${link_prefix}tip" group="${prefix}${finger_name}_ee" parent_group="${prefix}${finger_name}" />
   </xacro:macro>
   <!--VIRTUAL JOINT: Purpose: this element defines a virtual joint between a robot link and an external frame of reference (considered fixed with respect to the robot)-->

File: sr_moveit_hand_config/config/shadowhands_prefix.srdf.xacro (robot description, xacro)
@@ -33,5 +33,4 @@
       <chain base_link="$(arg prefix)forearm" tip_link="$(arg prefix)palm" />
     </xacro:unless>
-    <group name="$(arg prefix)fingers" />
   </group>
   <xacro:unless value="$(arg is_lite)">
@@ -45,7 +44,4 @@
     </group>
   </xacro:if>
-  <group name="$(arg prefix)forearm">
-    <link name="$(arg prefix)forearm" />
-  </group>
   <group name="$(arg prefix)manipulator">
     <chain base_link="$(arg prefix)forearm" tip_link="$(arg prefix)manipulator" />
@@ -54,15 +50,24 @@
   <xacro:if value="$(arg ff)">
     <group name="$(arg prefix)first_finger">
-      <xacro:fingerjoints prefix="$(arg prefix)" joint_prefix="FF" lf="0"/>
+      <xacro:fingerchains prefix="$(arg prefix)" link_prefix="ff" lf="0"/>
+    </group>
+    <group name="$(arg prefix)first_finger_ee">
+      <link name="$(arg prefix)fftip"/>
     </group>
   </xacro:if>
   <xacro:if value="$(arg mf)">
     <group name="$(arg prefix)middle_finger">
-      <xacro:fingerjoints prefix="$(arg prefix)" joint_prefix="MF" lf="0"/>
+      <xacro:fingerchains prefix="$(arg prefix)" link_prefix="mf" lf="0"/>
+    </group>
+    <group name="$(arg prefix)middle_finger_ee">
+      <link name="$(arg prefix)mftip"/>
     </group>
   </xacro:if>
   <xacro:if value="$(arg rf)">
     <group name="$(arg prefix)ring_finger">
-      <xacro:fingerjoints prefix="$(arg prefix)" joint_prefix="RF" lf="0"/>
+      <xacro:fingerchains prefix="$(arg prefix)" link_prefix="rf" lf="0"/>
+    </group>
+    <group name="$(arg prefix)ring_finger_ee">
+      <link name="$(arg prefix)rftip"/>
     </group>
   </xacro:if>
@@ -70,11 +75,17 @@
     <xacro:if value="$(arg lf)">
       <group name="$(arg prefix)little_finger">
-        <xacro:fingerjoints prefix="$(arg prefix)" joint_prefix="LF" lf="1"/>
+        <xacro:fingerchains prefix="$(arg prefix)" link_prefix="lf" lf="1"/>
       </group>
+      <group name="$(arg prefix)little_finger_ee">
+        <link name="$(arg prefix)lftip"/>
+      </group>
     </xacro:if>
   </xacro:unless>
   <xacro:if value="$(arg th)">
     <group name="$(arg prefix)thumb">
-      <xacro:thumbjoints prefix="$(arg prefix)"/>
+      <xacro:fingerchains prefix="$(arg prefix)" link_prefix="th" lf="0"/>
+    </group>
+    <group name="$(arg prefix)thumb_ee">
+      <link name="$(arg prefix)thtip"/>
     </group>
   </xacro:if>
@@ -82,22 +93,17 @@
   <group name="$(arg prefix)fingers">
    <xacro:if value="$(arg th)">
-      <xacro:thumbjoints prefix="$(arg prefix)" />
       <group name="$(arg prefix)thumb" />
     </xacro:if>
     <xacro:if value="$(arg ff)">
-      <xacro:fingerjoints prefix="$(arg prefix)" joint_prefix="FF" lf="0"/>
       <group name="$(arg prefix)first_finger" />
     </xacro:if>
     <xacro:if value="$(arg mf)">
-      <xacro:fingerjoints prefix="$(arg prefix)" joint_prefix="MF" lf="0"/>
       <group name="$(arg prefix)middle_finger" />
     </xacro:if>
     <xacro:if value="$(arg rf)">
-      <xacro:fingerjoints prefix="$(arg prefix)" joint_prefix="RF" lf="0"/>
       <group name="$(arg prefix)ring_finger" />
     </xacro:if>
     <xacro:unless value="$(arg is_lite)">
       <xacro:if value="$(arg lf)">
-        <xacro:fingerjoints prefix="$(arg prefix)" joint_prefix="LF" lf="1"/>
         <group name="$(arg prefix)little_finger" />
       </xacro:if>
@@ -302,11 +308,9 @@
   </xacro:if>
   <xacro:unless value="$(arg is_lite)">
-    <end_effector group="$(arg prefix)wrist" name="$(arg prefix)wrist_ee" parent_link="$(arg prefix)forearm" parent_group="$(arg prefix)forearm"/>
-    <end_effector group="$(arg prefix)fingers" name="$(arg prefix)palm_ee" parent_group="$(arg prefix)wrist" parent_link="$(arg prefix)palm"/>
+    <end_effector name="$(arg prefix)wrist_ee" group="$(arg prefix)fingers" parent_link="$(arg prefix)palm" parent_group="$(arg prefix)wrist"/>
   </xacro:unless>
   <xacro:if value="$(arg is_lite)">
-    <end_effector group="$(arg prefix)fingers" name="$(arg prefix)palm_ee" parent_group="$(arg prefix)wrist_lite" parent_link="$(arg prefix)palm"/>
-  </xacro:if>
-  <end_effector group="$(arg prefix)fingers" name="$(arg prefix)manipulator_ee" parent_group="$(arg prefix)manipulator" parent_link="$(arg prefix)manipulator"/>
+    <end_effector name="$(arg prefix)wrist_ee" group="$(arg prefix)fingers" parent_link="$(arg prefix)palm" parent_group="$(arg prefix)wrist_lite"/>
+  </xacro:if>
   <!--DISABLE COLLISIONS: By default it is assumed that any link of the robot could potentially come into collision with any other link in the robot. This tag disables collision checking between a specified pair of links. -->
   <xacro:hand_collisions prefix="$(arg prefix)" />

Commit message: SRDF generator now loads multi-robot move group states from a yaml file. These groups can reference each other or SRDF-defined groups. Adding "relaxed hand" states and including them in arm start states (only if hand move groups exist).

File: sr_moveit_hand_config/config/shadowhand.srdf.xacro (robot description, xacro)
@@ -108,4 +108,40 @@
       <joint name="${prefix}THJ5" value="0.19" />
     </xacro:if>
+  </xacro:macro>
+  <xacro:macro name="finger_state_relaxed" params="prefix joint_prefix">
+    <xacro:if value="${joint_prefix == 'FF'}">
+      <joint name="${prefix}${joint_prefix}J1" value="0.0128" />
+      <joint name="${prefix}${joint_prefix}J2" value="0.8508" />
+      <joint name="${prefix}${joint_prefix}J3" value="0.0156" />
+      <joint name="${prefix}${joint_prefix}J4" value="-0.05" />
+    </xacro:if>
+    <xacro:if value="${joint_prefix == 'MF'}">
+      <joint name="${prefix}${joint_prefix}J1" value="0.0246" />
+      <joint name="${prefix}${joint_prefix}J2" value="0.7201" />
+      <joint name="${prefix}${joint_prefix}J3" value="0.1918" />
+      <joint name="${prefix}${joint_prefix}J4" value="-0.0160" />
+    </xacro:if>
+    <xacro:if value="${joint_prefix == 'RF'}">
+      <joint name="${prefix}${joint_prefix}J1" value="0.0189" />
+      <joint name="${prefix}${joint_prefix}J2" value="0.5994" />
+      <joint name="${prefix}${joint_prefix}J3" value="0.4371" />
+      <joint name="${prefix}${joint_prefix}J4" value="-0.0297" />
+    </xacro:if>
+    <xacro:if value="${joint_prefix == 'LF'}">
+      <joint name="${prefix}${joint_prefix}J1" value="0.0093" />
+      <joint name="${prefix}${joint_prefix}J2" value="0.7751" />
+      <joint name="${prefix}${joint_prefix}J3" value="0.0861" />
+      <joint name="${prefix}${joint_prefix}J4" value="-0.2209" />
+      <joint name="${prefix}${joint_prefix}J5" value="0.3325" />
+    </xacro:if>
+  </xacro:macro>
+  <xacro:macro name="thumb_state_relaxed" params="prefix">
+    <joint name="${prefix}THJ1" value="0.0837" />
+    <joint name="${prefix}THJ2" value="0.2629" />
+    <xacro:unless value="$(arg is_lite)">
+      <joint name="${prefix}THJ3" value="-0.0944" />
+    </xacro:unless>
+    <joint name="${prefix}THJ4" value="0.5838" />
+    <joint name="${prefix}THJ5" value="0.1794" />
   </xacro:macro>
   <xacro:macro name="finger_thumb_state_open" params="prefix finger_name joint_prefix lf is_lite">

File: sr_moveit_hand_config/config/shadowhands_prefix.srdf.xacro (robot description, xacro)
@@ -296,4 +296,44 @@
     </xacro:unless>
   </group_state>
+  <group_state name="relaxed" group="$(arg prefix)fingers">
+    <xacro:if value="$(arg th)">
+        <xacro:thumb_state_relaxed  prefix="$(arg prefix)"/>
+    </xacro:if>
+    <xacro:if value="$(arg ff)">
+        <xacro:finger_state_relaxed  prefix="$(arg prefix)" joint_prefix="FF"/>
+    </xacro:if>
+    <xacro:if value="$(arg mf)">
+        <xacro:finger_state_relaxed  prefix="$(arg prefix)" joint_prefix="MF"/>
+    </xacro:if>
+    <xacro:if value="$(arg rf)">
+        <xacro:finger_state_relaxed  prefix="$(arg prefix)" joint_prefix="RF"/>
+    </xacro:if>
+    <xacro:unless value="$(arg is_lite)">
+      <xacro:if value="$(arg lf)">
+          <xacro:finger_state_relaxed  prefix="$(arg prefix)" joint_prefix="LF"/>
+      </xacro:if>
+    </xacro:unless>
+  </group_state>
+  <group_state name="relaxed" group="$(arg hand_name)">
+    <xacro:if value="$(arg th)">
+        <xacro:thumb_state_relaxed  prefix="$(arg prefix)"/>
+    </xacro:if>
+    <xacro:if value="$(arg ff)">
+        <xacro:finger_state_relaxed  prefix="$(arg prefix)" joint_prefix="FF"/>
+    </xacro:if>
+    <xacro:if value="$(arg mf)">
+        <xacro:finger_state_relaxed  prefix="$(arg prefix)" joint_prefix="MF"/>
+    </xacro:if>
+    <xacro:if value="$(arg rf)">
+        <xacro:finger_state_relaxed  prefix="$(arg prefix)" joint_prefix="RF"/>
+    </xacro:if>
+    <xacro:unless value="$(arg is_lite)">
+      <xacro:if value="$(arg lf)">
+          <xacro:finger_state_relaxed  prefix="$(arg prefix)" joint_prefix="LF"/>
+      </xacro:if>
+      <joint name="$(arg prefix)WRJ1" value="0" />
+      <joint name="$(arg prefix)WRJ2" value="0" />
+    </xacro:unless>
+  </group_state>
   <!--END EFFECTOR: Purpose: Represent information about an end effector.-->
   <!-- single finger end-effectors -->

Commit message: Swapped the open.py and close.py demos to use named states not fixed values. Updated fixed values for finger J1-J2 to 70 degrees.

File: sr_moveit_hand_config/config/shadowhand.srdf.xacro (robot description, xacro)
@@ -101,10 +101,10 @@
   <xacro:macro name="finger_state_pack" params="prefix joint_prefix lf is_biotac">
   	<xacro:unless value="${is_biotac}">
-      <joint name="${prefix}${joint_prefix}J1" value="1.5707" />
+      <joint name="${prefix}${joint_prefix}J1" value="1.2217" />
     </xacro:unless>
     <xacro:if value="${is_biotac}">
       <joint name="${prefix}${joint_prefix}J1" value="0.35" />
     </xacro:if>
-      <joint name="${prefix}${joint_prefix}J2" value="1.5707" />
+      <joint name="${prefix}${joint_prefix}J2" value="1.2217" />
       <joint name="${prefix}${joint_prefix}J3" value="1.5707" />
       <joint name="${prefix}${joint_prefix}J4" value="0" />

Commit message: Changed the joint values for close.

File: sr_moveit_hand_config/config/shadowhand.srdf.xacro (robot description, xacro)
@@ -101,10 +101,10 @@
   <xacro:macro name="finger_state_pack" params="prefix joint_prefix lf is_biotac">
   	<xacro:unless value="${is_biotac}">
-      <joint name="${prefix}${joint_prefix}J1" value="1.2217" />
+      <joint name="${prefix}${joint_prefix}J1" value="1.0472" />
     </xacro:unless>
     <xacro:if value="${is_biotac}">
       <joint name="${prefix}${joint_prefix}J1" value="0.35" />
     </xacro:if>
-      <joint name="${prefix}${joint_prefix}J2" value="1.2217" />
+      <joint name="${prefix}${joint_prefix}J2" value="1.1344" />
       <joint name="${prefix}${joint_prefix}J3" value="1.5707" />
       <joint name="${prefix}${joint_prefix}J4" value="0" />
@@ -115,10 +115,10 @@
   <xacro:macro name="thumb_state_pack" params="prefix is_biotac">
     <xacro:unless value="${is_biotac}">
-      <joint name="${prefix}THJ1" value="0.52" />
-      <joint name="${prefix}THJ2" value="0.61" />
+      <joint name="${prefix}THJ1" value="0.92" />
+      <joint name="${prefix}THJ2" value="0.62" />
       <xacro:unless value="$(arg is_lite)">
         <joint name="${prefix}THJ3" value="0.00" />
       </xacro:unless>
-      <joint name="${prefix}THJ4" value="1.20" />
+      <joint name="${prefix}THJ4" value="1.12" />
       <joint name="${prefix}THJ5" value="0.17" />
     </xacro:unless>

Commit message: Reset the finger pack position. Adjusted the thumb so its closer to the hand.

File: sr_moveit_hand_config/config/shadowhand.srdf.xacro (robot description, xacro)
@@ -101,10 +101,10 @@
   <xacro:macro name="finger_state_pack" params="prefix joint_prefix lf is_biotac">
   	<xacro:unless value="${is_biotac}">
-      <joint name="${prefix}${joint_prefix}J1" value="1.0472" />
+      <joint name="${prefix}${joint_prefix}J1" value="1.5707" />
     </xacro:unless>
     <xacro:if value="${is_biotac}">
       <joint name="${prefix}${joint_prefix}J1" value="0.35" />
     </xacro:if>
-      <joint name="${prefix}${joint_prefix}J2" value="1.1344" />
+      <joint name="${prefix}${joint_prefix}J2" value="1.5707" />
       <joint name="${prefix}${joint_prefix}J3" value="1.5707" />
       <joint name="${prefix}${joint_prefix}J4" value="0" />
@@ -115,10 +115,10 @@
   <xacro:macro name="thumb_state_pack" params="prefix is_biotac">
     <xacro:unless value="${is_biotac}">
-      <joint name="${prefix}THJ1" value="0.92" />
-      <joint name="${prefix}THJ2" value="0.62" />
+      <joint name="${prefix}THJ1" value="0.72" />
+      <joint name="${prefix}THJ2" value="0.71" />
       <xacro:unless value="$(arg is_lite)">
         <joint name="${prefix}THJ3" value="0.00" />
       </xacro:unless>
-      <joint name="${prefix}THJ4" value="1.12" />
+      <joint name="${prefix}THJ4" value="1.20" />
       <joint name="${prefix}THJ5" value="0.17" />
     </xacro:unless>

Commit message: Updated the close and open demo (#806)
* Swapped the open.py and close.py demos to use named states not fixed values. Updated fixed values for finger J1-J2 to 70 degrees.

* Changed the joint values for close.

* Reset the finger pack position. Adjusted the thumb so its closer to the hand.

* Added named state for bimanual.

* Fixed open and close demo.

* Update sr_demos/scripts/sr_demos/open.py

Co-authored-by: Maximilian Zieba <77073326+maxzieba@users.noreply.github.com>

* Update close.py

* Update close.py

---------

Co-authored-by: Maximilian Zieba <77073326+maxzieba@users.noreply.github.com>

File: sr_moveit_hand_config/config/shadowhand.srdf.xacro (robot description, xacro)
@@ -115,6 +115,6 @@
   <xacro:macro name="thumb_state_pack" params="prefix is_biotac">
     <xacro:unless value="${is_biotac}">
-      <joint name="${prefix}THJ1" value="0.52" />
-      <joint name="${prefix}THJ2" value="0.61" />
+      <joint name="${prefix}THJ1" value="0.72" />
+      <joint name="${prefix}THJ2" value="0.71" />
       <xacro:unless value="$(arg is_lite)">
         <joint name="${prefix}THJ3" value="0.00" />
