Commit message: Adding params

File: sr_moveit_hand_config/config/shadowhand.srdf.xacro (robot description, xacro)
@@ -99,9 +99,9 @@
       <joint name="${prefix}THJ5" value="0" />
   </xacro:macro>
-  <xacro:macro name="finger_state_pack" params="prefix joint_prefix lf is_biotac">
-  	<xacro:unless value="${is_biotac}">
+  <xacro:macro name="finger_state_pack" params="prefix joint_prefix lf is_bt_2p">
+  	<xacro:unless value="${is_bt_2p}">
       <joint name="${prefix}${joint_prefix}J1" value="1.5707" />
     </xacro:unless>
-    <xacro:if value="${is_biotac}">
+    <xacro:if value="${is_bt_2p}">
       <joint name="${prefix}${joint_prefix}J1" value="0.35" />
     </xacro:if>
@@ -113,6 +113,6 @@
       </xacro:if>
   </xacro:macro>
-  <xacro:macro name="thumb_state_pack" params="prefix is_biotac">
-    <xacro:unless value="${is_biotac}">
+  <xacro:macro name="thumb_state_pack" params="prefix is_bt_2p">
+    <xacro:unless value="${is_bt_2p}">
       <joint name="${prefix}THJ1" value="0.72" />
       <joint name="${prefix}THJ2" value="0.71" />
@@ -123,5 +123,5 @@
       <joint name="${prefix}THJ5" value="0.17" />
     </xacro:unless>
-    <xacro:if value="${is_biotac}">
+    <xacro:if value="${is_bt_2p}">
       <joint name="${prefix}THJ1" value="0.35" />
       <joint name="${prefix}THJ2" value="0.58" />

File: sr_moveit_hand_config/config/shadowhands_prefix.srdf.xacro (robot description, xacro)
@@ -33,5 +33,6 @@
   <xacro:arg name="th" default="1"/>
   <xacro:arg name="is_lite" default="0"/>
-  <xacro:arg name="is_biotac" default="0"/>
+  <xacro:arg name="is_bt_2p" default="0"/>
+  <xacro:arg name="is_bt_sp" default="0"/>
   <xacro:arg name="robot_name" default="shadowhand_motor"/>
   <xacro:arg name="hand_name" default="right_hand"/>
@@ -148,18 +149,18 @@
   <group_state name="pack" group="$(arg hand_name)">
     <xacro:if value="$(arg th)">
-        <xacro:thumb_state_pack  prefix="$(arg prefix)" is_biotac="$(arg is_biotac)" />
-    </xacro:if>
-    <xacro:if value="$(arg ff)">
-        <xacro:finger_state_pack  prefix="$(arg prefix)" joint_prefix="FF" lf="0" is_biotac="$(arg is_biotac)"/>
-    </xacro:if>
-    <xacro:if value="$(arg mf)">
-        <xacro:finger_state_pack  prefix="$(arg prefix)" joint_prefix="MF" lf="0" is_biotac="$(arg is_biotac)"/>
-    </xacro:if>
-    <xacro:if value="$(arg rf)">
-        <xacro:finger_state_pack  prefix="$(arg prefix)" joint_prefix="RF" lf="0" is_biotac="$(arg is_biotac)"/>
-    </xacro:if>
-    <xacro:unless value="$(arg is_lite)">
-      <xacro:if value="$(arg lf)">
-          <xacro:finger_state_pack  prefix="$(arg prefix)" joint_prefix="LF" lf="1" is_biotac="$(arg is_biotac)"/>
+        <xacro:thumb_state_pack  prefix="$(arg prefix)" is_bt_2p="$(arg is_bt_2p)" />
+    </xacro:if>
+    <xacro:if value="$(arg ff)">
+        <xacro:finger_state_pack  prefix="$(arg prefix)" joint_prefix="FF" lf="0" is_bt_2p="$(arg is_bt_2p)"/>
+    </xacro:if>
+    <xacro:if value="$(arg mf)">
+        <xacro:finger_state_pack  prefix="$(arg prefix)" joint_prefix="MF" lf="0" is_bt_2p="$(arg is_bt_2p)"/>
+    </xacro:if>
+    <xacro:if value="$(arg rf)">
+        <xacro:finger_state_pack  prefix="$(arg prefix)" joint_prefix="RF" lf="0" is_bt_2p="$(arg is_bt_2p)"/>
+    </xacro:if>
+    <xacro:unless value="$(arg is_lite)">
+      <xacro:if value="$(arg lf)">
+          <xacro:finger_state_pack  prefix="$(arg prefix)" joint_prefix="LF" lf="1" is_bt_2p="$(arg is_bt_2p)"/>
       </xacro:if>
       <joint name="$(arg prefix)WRJ1" value="0" />
@@ -172,15 +173,15 @@
     </xacro:if>
     <xacro:if value="$(arg ff)">
-        <xacro:finger_state_pack  prefix="$(arg prefix)" joint_prefix="FF" lf="0" is_biotac="$(arg is_biotac)"/>
-    </xacro:if>
-    <xacro:if value="$(arg mf)">
-        <xacro:finger_state_pack  prefix="$(arg prefix)" joint_prefix="MF" lf="0" is_biotac="$(arg is_biotac)"/>
-    </xacro:if>
-    <xacro:if value="$(arg rf)">
-        <xacro:finger_state_pack  prefix="$(arg prefix)" joint_prefix="RF" lf="0" is_biotac="$(arg is_biotac)"/>
-    </xacro:if>
-    <xacro:unless value="$(arg is_lite)">
-      <xacro:if value="$(arg lf)">
-          <xacro:finger_state_pack  prefix="$(arg prefix)" joint_prefix="LF" lf="1" is_biotac="$(arg is_biotac)"/>
+        <xacro:finger_state_pack  prefix="$(arg prefix)" joint_prefix="FF" lf="0" is_bt_2p="$(arg is_bt_2p)"/>
+    </xacro:if>
+    <xacro:if value="$(arg mf)">
+        <xacro:finger_state_pack  prefix="$(arg prefix)" joint_prefix="MF" lf="0" is_bt_2p="$(arg is_bt_2p)"/>
+    </xacro:if>
+    <xacro:if value="$(arg rf)">
+        <xacro:finger_state_pack  prefix="$(arg prefix)" joint_prefix="RF" lf="0" is_bt_2p="$(arg is_bt_2p)"/>
+    </xacro:if>
+    <xacro:unless value="$(arg is_lite)">
+      <xacro:if value="$(arg lf)">
+          <xacro:finger_state_pack  prefix="$(arg prefix)" joint_prefix="LF" lf="1" is_bt_2p="$(arg is_bt_2p)"/>
       </xacro:if>
       <joint name="$(arg prefix)WRJ1" value="0" />
@@ -218,15 +219,15 @@
   <xacro:if value="$(arg ff)">
     <group_state name="first_finger_pack" group="$(arg prefix)first_finger">
-        <xacro:finger_state_pack  prefix="$(arg prefix)" joint_prefix="FF" lf="0" is_biotac="$(arg is_biotac)"/>
+        <xacro:finger_state_pack  prefix="$(arg prefix)" joint_prefix="FF" lf="0" is_bt_2p="$(arg is_bt_2p)"/>
       </group_state>
   </xacro:if>
   <xacro:if value="$(arg mf)">
     <group_state name="middle_finger_pack" group="$(arg prefix)middle_finger">
-      <xacro:finger_state_pack  prefix="$(arg prefix)" joint_prefix="MF" lf="0" is_biotac="$(arg is_biotac)"/>
+      <xacro:finger_state_pack  prefix="$(arg prefix)" joint_prefix="MF" lf="0" is_bt_2p="$(arg is_bt_2p)"/>
     </group_state>
   </xacro:if>
   <xacro:if value="$(arg rf)">
     <group_state name="ring_finger_pack" group="$(arg prefix)ring_finger">
-      <xacro:finger_state_pack  prefix="$(arg prefix)" joint_prefix="RF" lf="0" is_biotac="$(arg is_biotac)"/>
+      <xacro:finger_state_pack  prefix="$(arg prefix)" joint_prefix="RF" lf="0" is_bt_2p="$(arg is_bt_2p)"/>
     </group_state>
   </xacro:if>
@@ -234,5 +235,5 @@
     <xacro:if value="$(arg lf)">
       <group_state name="little_finger_pack" group="$(arg prefix)little_finger">
-        <xacro:finger_state_pack  prefix="$(arg prefix)" joint_prefix="LF" lf="1" is_biotac="$(arg is_biotac)"/>
+        <xacro:finger_state_pack  prefix="$(arg prefix)" joint_prefix="LF" lf="1" is_bt_2p="$(arg is_bt_2p)"/>
       </group_state>
     </xacro:if>
@@ -240,5 +241,5 @@
   <xacro:if value="$(arg th)">
     <group_state name="thumb_pack" group="$(arg prefix)thumb">
-        <xacro:thumb_state_pack  prefix="$(arg prefix)" is_biotac="$(arg is_biotac)" />
+        <xacro:thumb_state_pack  prefix="$(arg prefix)" is_bt_2p="$(arg is_bt_2p)" />
     </group_state>
   </xacro:if>
@@ -265,18 +266,18 @@
   <group_state name="fingers_pack" group="$(arg prefix)fingers">
     <xacro:if value="$(arg th)">
-        <xacro:thumb_state_pack  prefix="$(arg prefix)" is_biotac="$(arg is_biotac)" />
-    </xacro:if>
-    <xacro:if value="$(arg ff)">
-        <xacro:finger_state_pack  prefix="$(arg prefix)" joint_prefix="FF" lf="0" is_biotac="$(arg is_biotac)"/>
-    </xacro:if>
-    <xacro:if value="$(arg mf)">
-        <xacro:finger_state_pack  prefix="$(arg prefix)" joint_prefix="MF" lf="0" is_biotac="$(arg is_biotac)"/>
-    </xacro:if>
-    <xacro:if value="$(arg rf)">
-        <xacro:finger_state_pack  prefix="$(arg prefix)" joint_prefix="RF" lf="0" is_biotac="$(arg is_biotac)"/>
-    </xacro:if>
-    <xacro:unless value="$(arg is_lite)">
-      <xacro:if value="$(arg lf)">
-          <xacro:finger_state_pack  prefix="$(arg prefix)" joint_prefix="LF" lf="1" is_biotac="$(arg is_biotac)"/>
+        <xacro:thumb_state_pack  prefix="$(arg prefix)" is_bt_2p="$(arg is_bt_2p)" />
+    </xacro:if>
+    <xacro:if value="$(arg ff)">
+        <xacro:finger_state_pack  prefix="$(arg prefix)" joint_prefix="FF" lf="0" is_bt_2p="$(arg is_bt_2p)"/>
+    </xacro:if>
+    <xacro:if value="$(arg mf)">
+        <xacro:finger_state_pack  prefix="$(arg prefix)" joint_prefix="MF" lf="0" is_bt_2p="$(arg is_bt_2p)"/>
+    </xacro:if>
+    <xacro:if value="$(arg rf)">
+        <xacro:finger_state_pack  prefix="$(arg prefix)" joint_prefix="RF" lf="0" is_bt_2p="$(arg is_bt_2p)"/>
+    </xacro:if>
+    <xacro:unless value="$(arg is_lite)">
+      <xacro:if value="$(arg lf)">
+          <xacro:finger_state_pack  prefix="$(arg prefix)" joint_prefix="LF" lf="1" is_bt_2p="$(arg is_bt_2p)"/>
       </xacro:if>
     </xacro:unless>
@@ -287,15 +288,15 @@
     </xacro:if>
     <xacro:if value="$(arg ff)">
-        <xacro:finger_state_pack  prefix="$(arg prefix)" joint_prefix="FF" lf="0" is_biotac="$(arg is_biotac)"/>
-    </xacro:if>
-    <xacro:if value="$(arg mf)">
-        <xacro:finger_state_pack  prefix="$(arg prefix)" joint_prefix="MF" lf="0" is_biotac="$(arg is_biotac)"/>
-    </xacro:if>
-    <xacro:if value="$(arg rf)">
-        <xacro:finger_state_pack  prefix="$(arg prefix)" joint_prefix="RF" lf="0" is_biotac="$(arg is_biotac)"/>
-    </xacro:if>
-    <xacro:unless value="$(arg is_lite)">
-      <xacro:if value="$(arg lf)">
-          <xacro:finger_state_pack  prefix="$(arg prefix)" joint_prefix="LF" lf="1" is_biotac="$(arg is_biotac)"/>
+        <xacro:finger_state_pack  prefix="$(arg prefix)" joint_prefix="FF" lf="0" is_bt_2p="$(arg is_bt_2p)"/>
+    </xacro:if>
+    <xacro:if value="$(arg mf)">
+        <xacro:finger_state_pack  prefix="$(arg prefix)" joint_prefix="MF" lf="0" is_bt_2p="$(arg is_bt_2p)"/>
+    </xacro:if>
+    <xacro:if value="$(arg rf)">
+        <xacro:finger_state_pack  prefix="$(arg prefix)" joint_prefix="RF" lf="0" is_bt_2p="$(arg is_bt_2p)"/>
+    </xacro:if>
+    <xacro:unless value="$(arg is_lite)">
+      <xacro:if value="$(arg lf)">
+          <xacro:finger_state_pack  prefix="$(arg prefix)" joint_prefix="LF" lf="1" is_bt_2p="$(arg is_bt_2p)"/>
       </xacro:if>
     </xacro:unless>
@@ -303,5 +304,5 @@
   <group_state name="first_finger_point" group="$(arg prefix)fingers">
     <xacro:if value="$(arg th)">
-        <xacro:thumb_state_pack  prefix="$(arg prefix)" is_biotac="$(arg is_biotac)" />
+        <xacro:thumb_state_pack  prefix="$(arg prefix)" is_bt_2p="$(arg is_bt_2p)" />
     </xacro:if>
     <xacro:if value="$(arg ff)">
@@ -309,12 +310,12 @@
     </xacro:if>
     <xacro:if value="$(arg mf)">
-        <xacro:finger_state_pack  prefix="$(arg prefix)" joint_prefix="MF" lf="0" is_biotac="$(arg is_biotac)"/>
-    </xacro:if>
-    <xacro:if value="$(arg rf)">
-        <xacro:finger_state_pack  prefix="$(arg prefix)" joint_prefix="RF" lf="0" is_biotac="$(arg is_biotac)"/>
-    </xacro:if>
-    <xacro:unless value="$(arg is_lite)">
-      <xacro:if value="$(arg lf)">
-          <xacro:finger_state_pack  prefix="$(arg prefix)" joint_prefix="LF" lf="1" is_biotac="$(arg is_biotac)"/>
+        <xacro:finger_state_pack  prefix="$(arg prefix)" joint_prefix="MF" lf="0" is_bt_2p="$(arg is_bt_2p)"/>
+    </xacro:if>
+    <xacro:if value="$(arg rf)">
+        <xacro:finger_state_pack  prefix="$(arg prefix)" joint_prefix="RF" lf="0" is_bt_2p="$(arg is_bt_2p)"/>
+    </xacro:if>
+    <xacro:unless value="$(arg is_lite)">
+      <xacro:if value="$(arg lf)">
+          <xacro:finger_state_pack  prefix="$(arg prefix)" joint_prefix="LF" lf="1" is_bt_2p="$(arg is_bt_2p)"/>
       </xacro:if>
     </xacro:unless>

Commit message: Adding params

File: sr_moveit_hand_config/config/shadowhand.srdf.xacro (robot description, xacro)
@@ -41,5 +41,5 @@
     <xacro:if value="${lf}">
       <!-- Little finger special case -->
-     <joint name="${prefix}${joint_prefix}J5" />
+      <joint name="${prefix}${joint_prefix}J5" />
     </xacro:if>
     <joint name="${prefix}${joint_prefix}J4" />
@@ -55,5 +55,5 @@
     <xacro:if value="${lf}">
       <!-- Little finger special case -->
-     <link name="${prefix}${link_prefix}metacarpal" />
+      <link name="${prefix}${link_prefix}metacarpal" />
     </xacro:if>
     <link name="${prefix}${link_prefix}knuckle" />
@@ -81,38 +81,38 @@
   <!--GROUP STATES: Purpose: Define a named state for a particular group, in terms of joint values. This is useful to define states like 'folded arms'-->
   <xacro:macro name="finger_state_open" params="prefix joint_prefix lf">
-      <joint name="${prefix}${joint_prefix}J1" value="0" />
-      <joint name="${prefix}${joint_prefix}J2" value="0" />
-      <joint name="${prefix}${joint_prefix}J3" value="0" />
-      <joint name="${prefix}${joint_prefix}J4" value="0" />
-      <xacro:if value="${lf}">
-       <!-- Little finger special case -->
-       <joint name="${prefix}${joint_prefix}J5" value="0" />
-      </xacro:if>
+    <joint name="${prefix}${joint_prefix}J1" value="0" />
+    <joint name="${prefix}${joint_prefix}J2" value="0" />
+    <joint name="${prefix}${joint_prefix}J3" value="0" />
+    <joint name="${prefix}${joint_prefix}J4" value="0" />
+    <xacro:if value="${lf}">
+      <!-- Little finger special case -->
+      <joint name="${prefix}${joint_prefix}J5" value="0" />
+    </xacro:if>
   </xacro:macro>
   <xacro:macro name="thumb_state_open" params="prefix">
-      <joint name="${prefix}THJ1" value="0" />
-      <joint name="${prefix}THJ2" value="0" />
-      <xacro:unless value="$(arg is_lite)">
-        <joint name="${prefix}THJ3" value="0" />
-      </xacro:unless>
-      <joint name="${prefix}THJ4" value="0" />
-      <joint name="${prefix}THJ5" value="0" />
-  </xacro:macro>
-  <xacro:macro name="finger_state_pack" params="prefix joint_prefix lf is_bt_2p">
-  	<xacro:unless value="${is_bt_2p}">
+    <joint name="${prefix}THJ1" value="0" />
+    <joint name="${prefix}THJ2" value="0" />
+    <xacro:unless value="$(arg is_lite)">
+      <joint name="${prefix}THJ3" value="0" />
+    </xacro:unless>
+    <joint name="${prefix}THJ4" value="0" />
+    <joint name="${prefix}THJ5" value="0" />
+  </xacro:macro>
+  <xacro:macro name="finger_state_pack" params="prefix joint_prefix lf tip_sensors">
+  	<xacro:if value="${tip_sensors} == 'pst'">
       <joint name="${prefix}${joint_prefix}J1" value="1.5707" />
     </xacro:unless>
-    <xacro:if value="${is_bt_2p}">
+    <xacro:if value="${tip_sensors} == 'bt_2p'">
       <joint name="${prefix}${joint_prefix}J1" value="0.35" />
     </xacro:if>
-      <joint name="${prefix}${joint_prefix}J2" value="1.5707" />
-      <joint name="${prefix}${joint_prefix}J3" value="1.5707" />
-      <joint name="${prefix}${joint_prefix}J4" value="0" />
-      <xacro:if value="${lf}">
-       <joint name="${prefix}${joint_prefix}J5" value="0" />
-      </xacro:if>
-  </xacro:macro>
-  <xacro:macro name="thumb_state_pack" params="prefix is_bt_2p">
-    <xacro:unless value="${is_bt_2p}">
+    <joint name="${prefix}${joint_prefix}J2" value="1.5707" />
+    <joint name="${prefix}${joint_prefix}J3" value="1.5707" />
+    <joint name="${prefix}${joint_prefix}J4" value="0" />
+    <xacro:if value="${lf}">
+      <joint name="${prefix}${joint_prefix}J5" value="0" />
+    </xacro:if>
+  </xacro:macro>
+  <xacro:macro name="thumb_state_pack" params="prefix tip_sensors">
+    <xacro:if value="${tip_sensors} == 'pst'">
       <joint name="${prefix}THJ1" value="0.72" />
       <joint name="${prefix}THJ2" value="0.71" />
@@ -123,5 +123,5 @@
       <joint name="${prefix}THJ5" value="0.17" />
     </xacro:unless>
-    <xacro:if value="${is_bt_2p}">
+    <xacro:if value="${tip_sensors} == 'bt_2p'">
       <joint name="${prefix}THJ1" value="0.35" />
       <joint name="${prefix}THJ2" value="0.58" />
@@ -170,5 +170,5 @@
   </xacro:macro>
   <xacro:macro name="finger_thumb_state_open" params="prefix finger_name joint_prefix lf is_lite">
-   <group_state name="${finger_name}_thumb_open" group="${prefix}${finger_name}_thumb">
+    <group_state name="${finger_name}_thumb_open" group="${prefix}${finger_name}_thumb">
       <joint name="${prefix}${joint_prefix}J1" value="0" />
       <joint name="${prefix}${joint_prefix}J2" value="0" />
@@ -182,6 +182,6 @@
       <xacro:unless value="${is_lite}">
         <xacro:if value="${lf}">
-        <!-- Little finger special case -->
-         <joint name="${prefix}${joint_prefix}J5" value="0" />
+          <!-- Little finger special case -->
+          <joint name="${prefix}${joint_prefix}J5" value="0" />
         </xacro:if>
       </xacro:unless>
@@ -320,6 +320,6 @@
     <disable_collisions link1="${prefix}ffproximal" link2="${prefix}lfmetacarpal" reason="Never" />
   </xacro:macro>
-   <!-- finger next to other finger -->
-   <xacro:macro name="finger_closefinger_collisions" params="prefix link_prefix link_prefix2 lf" >
+  <!-- finger next to other finger -->
+  <xacro:macro name="finger_closefinger_collisions" params="prefix link_prefix link_prefix2 lf" >
     <disable_collisions link1="${prefix}${link_prefix}distal" link2="${prefix}${link_prefix2}knuckle" reason="Never" />
     <disable_collisions link1="${prefix}${link_prefix}knuckle" link2="${prefix}${link_prefix2}distal" reason="Never" />
@@ -346,6 +346,6 @@
     </xacro:if>
   </xacro:macro>
-   <!-- finger to thumb, far is 1 if at least one finger is in between -->
-   <xacro:macro name="finger_thumb_collisions" params="prefix link_prefix far lf" >
+  <!-- finger to thumb, far is 1 if at least one finger is in between -->
+  <xacro:macro name="finger_thumb_collisions" params="prefix link_prefix far lf" >
     <disable_collisions link1="${prefix}${link_prefix}distal" link2="${prefix}thbase" reason="Never" />
     <disable_collisions link1="${prefix}${link_prefix}distal" link2="${prefix}thhub" reason="Never" />

Commit message: Adding params

File: sr_moveit_hand_config/config/shadowhand.srdf.xacro (robot description, xacro)
@@ -103,4 +103,7 @@
       <joint name="${prefix}${joint_prefix}J1" value="1.5707" />
     </xacro:if>
+    <xacro:if value="${tip_sensors == 'bt_sp'}">
+      <joint name="${prefix}${joint_prefix}J1" value="1.5707" />
+    </xacro:if>
     <xacro:if value="${tip_sensors == 'bt_2p'}">
       <joint name="${prefix}${joint_prefix}J1" value="0.35" />
@@ -115,4 +118,13 @@
   <xacro:macro name="thumb_state_pack" params="prefix tip_sensors">
     <xacro:if value="${tip_sensors == 'pst'}">
+      <joint name="${prefix}THJ1" value="0.72" />
+      <joint name="${prefix}THJ2" value="0.71" />
+      <xacro:unless value="$(arg is_lite)">
+        <joint name="${prefix}THJ3" value="0.00" />
+      </xacro:unless>
+      <joint name="${prefix}THJ4" value="1.20" />
+      <joint name="${prefix}THJ5" value="0.17" />
+    </xacro:if>
+    <xacro:if value="${tip_sensors == 'bt_sp'}">
       <joint name="${prefix}THJ1" value="0.72" />
       <joint name="${prefix}THJ2" value="0.71" />

Commit message: Adding params

File: sr_moveit_hand_config/config/shadowhand.srdf.xacro (robot description, xacro)
@@ -102,13 +102,15 @@
   	<xacro:if value="${tip_sensors == 'pst'}">
       <joint name="${prefix}${joint_prefix}J1" value="1.5707" />
+      <joint name="${prefix}${joint_prefix}J3" value="1.5707" />
     </xacro:if>
     <xacro:if value="${tip_sensors == 'bt_sp'}">
-      <joint name="${prefix}${joint_prefix}J1" value="1.5707" />
+      <joint name="${prefix}${joint_prefix}J1" value="1.309" />
+      <joint name="${prefix}${joint_prefix}J3" value="1.309" />
     </xacro:if>
     <xacro:if value="${tip_sensors == 'bt_2p'}">
       <joint name="${prefix}${joint_prefix}J1" value="0.35" />
+      <joint name="${prefix}${joint_prefix}J3" value="1.5707" />
     </xacro:if>
     <joint name="${prefix}${joint_prefix}J2" value="1.5707" />
-    <joint name="${prefix}${joint_prefix}J3" value="1.5707" />
     <joint name="${prefix}${joint_prefix}J4" value="0" />
     <xacro:if value="${lf}">
@@ -127,10 +129,10 @@
     </xacro:if>
     <xacro:if value="${tip_sensors == 'bt_sp'}">
-      <joint name="${prefix}THJ1" value="0.72" />
+      <joint name="${prefix}THJ1" value="0.77" />
       <joint name="${prefix}THJ2" value="0.71" />
       <xacro:unless value="$(arg is_lite)">
         <joint name="${prefix}THJ3" value="0.00" />
       </xacro:unless>
-      <joint name="${prefix}THJ4" value="1.20" />
+      <joint name="${prefix}THJ4" value="1.00" />
       <joint name="${prefix}THJ5" value="0.17" />
     </xacro:if>

Commit message: Adding params

File: sr_moveit_hand_config/config/shadowhand.srdf.xacro (robot description, xacro)
@@ -129,11 +129,11 @@
     </xacro:if>
     <xacro:if value="${tip_sensors == 'bt_sp'}">
-      <joint name="${prefix}THJ1" value="0.77" />
-      <joint name="${prefix}THJ2" value="0.71" />
-      <xacro:unless value="$(arg is_lite)">
-        <joint name="${prefix}THJ3" value="0.00" />
+      <joint name="${prefix}THJ1" value="0.732" />
+      <joint name="${prefix}THJ2" value="0.70" />
+      <xacro:unless value="$(arg is_lite)">
+        <joint name="${prefix}THJ3" value="0.2" />
       </xacro:unless>
       <joint name="${prefix}THJ4" value="1.00" />
-      <joint name="${prefix}THJ5" value="0.17" />
+      <joint name="${prefix}THJ5" value="-0.10" />
     </xacro:if>
     <xacro:if value="${tip_sensors == 'bt_2p'}">
