Commit message: Changing load params

File: sr_moveit_hand_config/config/shadowhand.srdf.xacro (robot description, xacro)
@@ -99,50 +99,89 @@
     <joint name="${prefix}THJ5" value="0" />
   </xacro:macro>
-  <xacro:macro name="finger_state_pack" params="prefix joint_prefix lf tip_sensors">
-  	<xacro:if value="${tip_sensors == 'pst'}">
-      <joint name="${prefix}${joint_prefix}J1" value="1.5707" />
-      <joint name="${prefix}${joint_prefix}J3" value="1.5707" />
-    </xacro:if>
-    <xacro:if value="${tip_sensors == 'bt_sp'}">
-      <joint name="${prefix}${joint_prefix}J1" value="1.309" />
-      <joint name="${prefix}${joint_prefix}J3" value="1.309" />
-    </xacro:if>
-    <xacro:if value="${tip_sensors == 'bt_2p'}">
-      <joint name="${prefix}${joint_prefix}J1" value="0.35" />
-      <joint name="${prefix}${joint_prefix}J3" value="1.5707" />
-    </xacro:if>
-    <joint name="${prefix}${joint_prefix}J2" value="1.5707" />
-    <joint name="${prefix}${joint_prefix}J4" value="0" />
-    <xacro:if value="${lf}">
-      <joint name="${prefix}${joint_prefix}J5" value="0" />
-    </xacro:if>
-  </xacro:macro>
-  <xacro:macro name="thumb_state_pack" params="prefix tip_sensors">
-    <xacro:if value="${tip_sensors == 'pst'}">
-      <joint name="${prefix}THJ1" value="0.72" />
-      <joint name="${prefix}THJ2" value="0.71" />
-      <xacro:unless value="$(arg is_lite)">
+  <xacro:macro name="finger_state_pack" params="prefix joint_prefix lf tip_sensors hand_version">
+    <xacro:unless value="${hand_version == 'E4'}">
+      <xacro:if value="${tip_sensors == 'pst'}">
+        <joint name="${prefix}${joint_prefix}J1" value="1.5707" />
+        <joint name="${prefix}${joint_prefix}J3" value="1.5707" />
+      </xacro:if>
+      <xacro:if value="${tip_sensors == 'bt_sp'}">
+        <joint name="${prefix}${joint_prefix}J1" value="1.309" />
+        <joint name="${prefix}${joint_prefix}J3" value="1.309" />
+      </xacro:if>
+      <xacro:if value="${tip_sensors == 'bt_2p'}">
+        <joint name="${prefix}${joint_prefix}J1" value="0.35" />
+        <joint name="${prefix}${joint_prefix}J3" value="1.5707" />
+      </xacro:if>
+      <joint name="${prefix}${joint_prefix}J2" value="1.5707" />
+      <joint name="${prefix}${joint_prefix}J4" value="0" />
+      <xacro:if value="${lf}">
+        <joint name="${prefix}${joint_prefix}J5" value="0" />
+      </xacro:if>
+    </xacro:unless>
+    <xacro:if value="${hand_version == 'E4'}">
+      <xacro:if value="${tip_sensors == 'pst'}">
+        <joint name="${prefix}${joint_prefix}J1" value="1.5707" />
+        <joint name="${prefix}${joint_prefix}J3" value="1.309" />
+      </xacro:if>
+      <xacro:if value="${tip_sensors == 'bt_sp'}">
+        <joint name="${prefix}${joint_prefix}J1" value="1.309" />
+        <joint name="${prefix}${joint_prefix}J3" value="1.309" />
+      </xacro:if>
+      <joint name="${prefix}${joint_prefix}J2" value="1.5707" />
+      <joint name="${prefix}${joint_prefix}J4" value="0" />
+      <xacro:if value="${lf}">
+        <joint name="${prefix}${joint_prefix}J5" value="0" />
+      </xacro:if>
+    </xacro:if>
+  </xacro:macro>
+  <xacro:macro name="thumb_state_pack" params="prefix tip_sensors hand_version">
+    <xacro:unless value="${hand_version == 'E4'}">
+      <xacro:if value="${tip_sensors == 'pst'}">
+        <joint name="${prefix}THJ1" value="0.72" />
+        <joint name="${prefix}THJ2" value="0.71" />
+        <xacro:unless value="$(arg is_lite)">
+          <joint name="${prefix}THJ3" value="0.00" />
+        </xacro:unless>
+        <joint name="${prefix}THJ4" value="1.20" />
+        <joint name="${prefix}THJ5" value="0.17" />
+      </xacro:if>
+      <xacro:if value="${tip_sensors == 'bt_sp'}">
+        <joint name="${prefix}THJ1" value="0.732" />
+        <joint name="${prefix}THJ2" value="0.70" />
+        <xacro:unless value="$(arg is_lite)">
+          <joint name="${prefix}THJ3" value="0.2" />
+        </xacro:unless>
+        <joint name="${prefix}THJ4" value="1.00" />
+        <joint name="${prefix}THJ5" value="-0.10" />
+      </xacro:if>
+      <xacro:if value="${tip_sensors == 'bt_2p'}">
+        <joint name="${prefix}THJ1" value="0.35" />
+        <joint name="${prefix}THJ2" value="0.58" />
+        <xacro:unless value="$(arg is_lite)">
         <joint name="${prefix}THJ3" value="0.00" />
-      </xacro:unless>
-      <joint name="${prefix}THJ4" value="1.20" />
-      <joint name="${prefix}THJ5" value="0.17" />
-    </xacro:if>
-    <xacro:if value="${tip_sensors == 'bt_sp'}">
-      <joint name="${prefix}THJ1" value="0.732" />
-      <joint name="${prefix}THJ2" value="0.70" />
-      <xacro:unless value="$(arg is_lite)">
-        <joint name="${prefix}THJ3" value="0.2" />
-      </xacro:unless>
-      <joint name="${prefix}THJ4" value="1.00" />
-      <joint name="${prefix}THJ5" value="-0.10" />
-    </xacro:if>
-    <xacro:if value="${tip_sensors == 'bt_2p'}">
-      <joint name="${prefix}THJ1" value="0.35" />
-      <joint name="${prefix}THJ2" value="0.58" />
-      <xacro:unless value="$(arg is_lite)">
-      <joint name="${prefix}THJ3" value="0.00" />
-      </xacro:unless>
-      <joint name="${prefix}THJ4" value="0.39" />
-      <joint name="${prefix}THJ5" value="0.19" />
+        </xacro:unless>
+        <joint name="${prefix}THJ4" value="0.39" />
+        <joint name="${prefix}THJ5" value="0.19" />
+      </xacro:if>
+    </xacro:unless>
+    <xacro:if value="${hand_version == 'E4'}">
+      <xacro:if value="${tip_sensors == 'pst'}">
+        <joint name="${prefix}THJ1" value="0.72" />
+        <joint name="${prefix}THJ2" value="0.57" />
+        <xacro:unless value="$(arg is_lite)">
+          <joint name="${prefix}THJ3" value="0.00" />
+        </xacro:unless>
+        <joint name="${prefix}THJ4" value="1.20" />
+        <joint name="${prefix}THJ5" value="0.17" />
+      </xacro:if>
+      <xacro:if value="${tip_sensors == 'bt_sp'}">
+        <joint name="${prefix}THJ1" value="0.732" />
+        <joint name="${prefix}THJ2" value="0.70" />
+        <xacro:unless value="$(arg is_lite)">
+          <joint name="${prefix}THJ3" value="0.2" />
+        </xacro:unless>
+        <joint name="${prefix}THJ4" value="1.00" />
+        <joint name="${prefix}THJ5" value="-0.10" />
+      </xacro:if>
     </xacro:if>
   </xacro:macro>

File: sr_moveit_hand_config/config/shadowhands_prefix.srdf.xacro (robot description, xacro)
@@ -34,4 +34,5 @@
   <xacro:arg name="is_lite" default="0"/>
   <xacro:arg name="tip_sensors" default="pst"/>
+  <xacro:arg name="hand_version" default="E3M5"/>
   <xacro:arg name="robot_name" default="shadowhand_motor"/>
   <xacro:arg name="hand_name" default="right_hand"/>
@@ -148,18 +149,18 @@
   <group_state name="pack" group="$(arg hand_name)">
     <xacro:if value="$(arg th)">
-        <xacro:thumb_state_pack  prefix="$(arg prefix)" tip_sensors="$(arg tip_sensors)" />
-    </xacro:if>
-    <xacro:if value="$(arg ff)">
-        <xacro:finger_state_pack  prefix="$(arg prefix)" joint_prefix="FF" lf="0" tip_sensors="$(arg tip_sensors)"/>
-    </xacro:if>
-    <xacro:if value="$(arg mf)">
-        <xacro:finger_state_pack  prefix="$(arg prefix)" joint_prefix="MF" lf="0" tip_sensors="$(arg tip_sensors)"/>
-    </xacro:if>
-    <xacro:if value="$(arg rf)">
-        <xacro:finger_state_pack  prefix="$(arg prefix)" joint_prefix="RF" lf="0" tip_sensors="$(arg tip_sensors)"/>
-    </xacro:if>
-    <xacro:unless value="$(arg is_lite)">
-      <xacro:if value="$(arg lf)">
-          <xacro:finger_state_pack  prefix="$(arg prefix)" joint_prefix="LF" lf="1" tip_sensors="$(arg tip_sensors)"/>
+        <xacro:thumb_state_pack  prefix="$(arg prefix)" tip_sensors="$(arg tip_sensors)" hand_version="$(arg hand_version)"/>
+    </xacro:if>
+    <xacro:if value="$(arg ff)">
+        <xacro:finger_state_pack  prefix="$(arg prefix)" joint_prefix="FF" lf="0" tip_sensors="$(arg tip_sensors)" hand_version="$(arg hand_version)"/>
+    </xacro:if>
+    <xacro:if value="$(arg mf)">
+        <xacro:finger_state_pack  prefix="$(arg prefix)" joint_prefix="MF" lf="0" tip_sensors="$(arg tip_sensors)" hand_version="$(arg hand_version)"/>
+    </xacro:if>
+    <xacro:if value="$(arg rf)">
+        <xacro:finger_state_pack  prefix="$(arg prefix)" joint_prefix="RF" lf="0" tip_sensors="$(arg tip_sensors)" hand_version="$(arg hand_version)"/>
+    </xacro:if>
+    <xacro:unless value="$(arg is_lite)">
+      <xacro:if value="$(arg lf)">
+          <xacro:finger_state_pack  prefix="$(arg prefix)" joint_prefix="LF" lf="1" tip_sensors="$(arg tip_sensors)" hand_version="$(arg hand_version)"/>
       </xacro:if>
       <joint name="$(arg prefix)WRJ1" value="0" />
@@ -172,15 +173,15 @@
     </xacro:if>
     <xacro:if value="$(arg ff)">
-        <xacro:finger_state_pack  prefix="$(arg prefix)" joint_prefix="FF" lf="0" tip_sensors="$(arg tip_sensors)"/>
-    </xacro:if>
-    <xacro:if value="$(arg mf)">
-        <xacro:finger_state_pack  prefix="$(arg prefix)" joint_prefix="MF" lf="0" tip_sensors="$(arg tip_sensors)"/>
-    </xacro:if>
-    <xacro:if value="$(arg rf)">
-        <xacro:finger_state_pack  prefix="$(arg prefix)" joint_prefix="RF" lf="0" tip_sensors="$(arg tip_sensors)"/>
-    </xacro:if>
-    <xacro:unless value="$(arg is_lite)">
-      <xacro:if value="$(arg lf)">
-          <xacro:finger_state_pack  prefix="$(arg prefix)" joint_prefix="LF" lf="1" tip_sensors="$(arg tip_sensors)"/>
+        <xacro:finger_state_pack  prefix="$(arg prefix)" joint_prefix="FF" lf="0" tip_sensors="$(arg tip_sensors)" hand_version="$(arg hand_version)"/>
+    </xacro:if>
+    <xacro:if value="$(arg mf)">
+        <xacro:finger_state_pack  prefix="$(arg prefix)" joint_prefix="MF" lf="0" tip_sensors="$(arg tip_sensors)" hand_version="$(arg hand_version)"/>
+    </xacro:if>
+    <xacro:if value="$(arg rf)">
+        <xacro:finger_state_pack  prefix="$(arg prefix)" joint_prefix="RF" lf="0" tip_sensors="$(arg tip_sensors)" hand_version="$(arg hand_version)"/>
+    </xacro:if>
+    <xacro:unless value="$(arg is_lite)">
+      <xacro:if value="$(arg lf)">
+          <xacro:finger_state_pack  prefix="$(arg prefix)" joint_prefix="LF" lf="1" tip_sensors="$(arg tip_sensors)" hand_version="$(arg hand_version)"/>
       </xacro:if>
       <joint name="$(arg prefix)WRJ1" value="0" />
@@ -218,15 +219,15 @@
   <xacro:if value="$(arg ff)">
     <group_state name="first_finger_pack" group="$(arg prefix)first_finger">
-        <xacro:finger_state_pack  prefix="$(arg prefix)" joint_prefix="FF" lf="0" tip_sensors="$(arg tip_sensors)"/>
+        <xacro:finger_state_pack  prefix="$(arg prefix)" joint_prefix="FF" lf="0" tip_sensors="$(arg tip_sensors)" hand_version="$(arg hand_version)"/>
       </group_state>
   </xacro:if>
   <xacro:if value="$(arg mf)">
     <group_state name="middle_finger_pack" group="$(arg prefix)middle_finger">
-      <xacro:finger_state_pack  prefix="$(arg prefix)" joint_prefix="MF" lf="0" tip_sensors="$(arg tip_sensors)"/>
+      <xacro:finger_state_pack  prefix="$(arg prefix)" joint_prefix="MF" lf="0" tip_sensors="$(arg tip_sensors)" hand_version="$(arg hand_version)"/>
     </group_state>
   </xacro:if>
   <xacro:if value="$(arg rf)">
     <group_state name="ring_finger_pack" group="$(arg prefix)ring_finger">
-      <xacro:finger_state_pack  prefix="$(arg prefix)" joint_prefix="RF" lf="0" tip_sensors="$(arg tip_sensors)"/>
+      <xacro:finger_state_pack  prefix="$(arg prefix)" joint_prefix="RF" lf="0" tip_sensors="$(arg tip_sensors)" hand_version="$(arg hand_version)"/>
     </group_state>
   </xacro:if>
@@ -234,5 +235,5 @@
     <xacro:if value="$(arg lf)">
       <group_state name="little_finger_pack" group="$(arg prefix)little_finger">
-        <xacro:finger_state_pack  prefix="$(arg prefix)" joint_prefix="LF" lf="1" tip_sensors="$(arg tip_sensors)"/>
+        <xacro:finger_state_pack  prefix="$(arg prefix)" joint_prefix="LF" lf="1" tip_sensors="$(arg tip_sensors)" hand_version="$(arg hand_version)"/>
       </group_state>
     </xacro:if>
@@ -240,5 +241,5 @@
   <xacro:if value="$(arg th)">
     <group_state name="thumb_pack" group="$(arg prefix)thumb">
-        <xacro:thumb_state_pack  prefix="$(arg prefix)" tip_sensors="$(arg tip_sensors)" />
+        <xacro:thumb_state_pack  prefix="$(arg prefix)" tip_sensors="$(arg tip_sensors)" hand_version="$(arg hand_version)"/>
     </group_state>
   </xacro:if>
@@ -265,18 +266,18 @@
   <group_state name="fingers_pack" group="$(arg prefix)fingers">
     <xacro:if value="$(arg th)">
-        <xacro:thumb_state_pack  prefix="$(arg prefix)" tip_sensors="$(arg tip_sensors)" />
-    </xacro:if>
-    <xacro:if value="$(arg ff)">
-        <xacro:finger_state_pack  prefix="$(arg prefix)" joint_prefix="FF" lf="0" tip_sensors="$(arg tip_sensors)"/>
-    </xacro:if>
-    <xacro:if value="$(arg mf)">
-        <xacro:finger_state_pack  prefix="$(arg prefix)" joint_prefix="MF" lf="0" tip_sensors="$(arg tip_sensors)"/>
-    </xacro:if>
-    <xacro:if value="$(arg rf)">
-        <xacro:finger_state_pack  prefix="$(arg prefix)" joint_prefix="RF" lf="0" tip_sensors="$(arg tip_sensors)"/>
-    </xacro:if>
-    <xacro:unless value="$(arg is_lite)">
-      <xacro:if value="$(arg lf)">
-          <xacro:finger_state_pack  prefix="$(arg prefix)" joint_prefix="LF" lf="1" tip_sensors="$(arg tip_sensors)"/>
+        <xacro:thumb_state_pack  prefix="$(arg prefix)" tip_sensors="$(arg tip_sensors)" hand_version="$(arg hand_version)" />
+    </xacro:if>
+    <xacro:if value="$(arg ff)">
+        <xacro:finger_state_pack  prefix="$(arg prefix)" joint_prefix="FF" lf="0" tip_sensors="$(arg tip_sensors)" hand_version="$(arg hand_version)"/>
+    </xacro:if>
+    <xacro:if value="$(arg mf)">
+        <xacro:finger_state_pack  prefix="$(arg prefix)" joint_prefix="MF" lf="0" tip_sensors="$(arg tip_sensors)" hand_version="$(arg hand_version)"/>
+    </xacro:if>
+    <xacro:if value="$(arg rf)">
+        <xacro:finger_state_pack  prefix="$(arg prefix)" joint_prefix="RF" lf="0" tip_sensors="$(arg tip_sensors)" hand_version="$(arg hand_version)"/>
+    </xacro:if>
+    <xacro:unless value="$(arg is_lite)">
+      <xacro:if value="$(arg lf)">
+          <xacro:finger_state_pack  prefix="$(arg prefix)" joint_prefix="LF" lf="1" tip_sensors="$(arg tip_sensors)" hand_version="$(arg hand_version)"/>
       </xacro:if>
     </xacro:unless>
@@ -287,15 +288,15 @@
     </xacro:if>
     <xacro:if value="$(arg ff)">
-        <xacro:finger_state_pack  prefix="$(arg prefix)" joint_prefix="FF" lf="0" tip_sensors="$(arg tip_sensors)"/>
-    </xacro:if>
-    <xacro:if value="$(arg mf)">
-        <xacro:finger_state_pack  prefix="$(arg prefix)" joint_prefix="MF" lf="0" tip_sensors="$(arg tip_sensors)"/>
-    </xacro:if>
-    <xacro:if value="$(arg rf)">
-        <xacro:finger_state_pack  prefix="$(arg prefix)" joint_prefix="RF" lf="0" tip_sensors="$(arg tip_sensors)"/>
-    </xacro:if>
-    <xacro:unless value="$(arg is_lite)">
-      <xacro:if value="$(arg lf)">
-          <xacro:finger_state_pack  prefix="$(arg prefix)" joint_prefix="LF" lf="1" tip_sensors="$(arg tip_sensors)"/>
+        <xacro:finger_state_pack  prefix="$(arg prefix)" joint_prefix="FF" lf="0" tip_sensors="$(arg tip_sensors)" hand_version="$(arg hand_version)"/>
+    </xacro:if>
+    <xacro:if value="$(arg mf)">
+        <xacro:finger_state_pack  prefix="$(arg prefix)" joint_prefix="MF" lf="0" tip_sensors="$(arg tip_sensors)" hand_version="$(arg hand_version)"/>
+    </xacro:if>
+    <xacro:if value="$(arg rf)">
+        <xacro:finger_state_pack  prefix="$(arg prefix)" joint_prefix="RF" lf="0" tip_sensors="$(arg tip_sensors)" hand_version="$(arg hand_version)"/>
+    </xacro:if>
+    <xacro:unless value="$(arg is_lite)">
+      <xacro:if value="$(arg lf)">
+          <xacro:finger_state_pack  prefix="$(arg prefix)" joint_prefix="LF" lf="1" tip_sensors="$(arg tip_sensors)" hand_version="$(arg hand_version)"/>
       </xacro:if>
     </xacro:unless>
@@ -303,5 +304,5 @@
   <group_state name="first_finger_point" group="$(arg prefix)fingers">
     <xacro:if value="$(arg th)">
-        <xacro:thumb_state_pack  prefix="$(arg prefix)" tip_sensors="$(arg tip_sensors)" />
+        <xacro:thumb_state_pack  prefix="$(arg prefix)" tip_sensors="$(arg tip_sensors)" hand_version="$(arg hand_version)"/>
     </xacro:if>
     <xacro:if value="$(arg ff)">
@@ -309,12 +310,12 @@
     </xacro:if>
     <xacro:if value="$(arg mf)">
-        <xacro:finger_state_pack  prefix="$(arg prefix)" joint_prefix="MF" lf="0" tip_sensors="$(arg tip_sensors)"/>
-    </xacro:if>
-    <xacro:if value="$(arg rf)">
-        <xacro:finger_state_pack  prefix="$(arg prefix)" joint_prefix="RF" lf="0" tip_sensors="$(arg tip_sensors)"/>
-    </xacro:if>
-    <xacro:unless value="$(arg is_lite)">
-      <xacro:if value="$(arg lf)">
-          <xacro:finger_state_pack  prefix="$(arg prefix)" joint_prefix="LF" lf="1" tip_sensors="$(arg tip_sensors)"/>
+        <xacro:finger_state_pack  prefix="$(arg prefix)" joint_prefix="MF" lf="0" tip_sensors="$(arg tip_sensors)" hand_version="$(arg hand_version)"/>
+    </xacro:if>
+    <xacro:if value="$(arg rf)">
+        <xacro:finger_state_pack  prefix="$(arg prefix)" joint_prefix="RF" lf="0" tip_sensors="$(arg tip_sensors)" hand_version="$(arg hand_version)"/>
+    </xacro:if>
+    <xacro:unless value="$(arg is_lite)">
+      <xacro:if value="$(arg lf)">
+          <xacro:finger_state_pack  prefix="$(arg prefix)" joint_prefix="LF" lf="1" tip_sensors="$(arg tip_sensors)" hand_version="$(arg hand_version)"/>
       </xacro:if>
     </xacro:unless>

Commit message: Updating positions to fit hand lite

File: sr_moveit_hand_config/config/shadowhand.srdf.xacro (robot description, xacro)
@@ -138,20 +138,20 @@
     <xacro:unless value="${hand_version == 'E4'}">
       <xacro:if value="${tip_sensors == 'pst'}">
-        <joint name="${prefix}THJ1" value="0.72" />
-        <joint name="${prefix}THJ2" value="0.71" />
+        <joint name="${prefix}THJ1" value="0.73" />
+        <joint name="${prefix}THJ2" value="0.70" />
         <xacro:unless value="$(arg is_lite)">
           <joint name="${prefix}THJ3" value="0.00" />
         </xacro:unless>
-        <joint name="${prefix}THJ4" value="1.20" />
-        <joint name="${prefix}THJ5" value="0.17" />
+        <joint name="${prefix}THJ4" value="1.22" />
+        <joint name="${prefix}THJ5" value="0.05" />
       </xacro:if>
       <xacro:if value="${tip_sensors == 'bt_sp'}">
-        <joint name="${prefix}THJ1" value="0.732" />
-        <joint name="${prefix}THJ2" value="0.70" />
+        <joint name="${prefix}THJ1" value="0.82" />
+        <joint name="${prefix}THJ2" value="0.55" />
         <xacro:unless value="$(arg is_lite)">
           <joint name="${prefix}THJ3" value="0.2" />
         </xacro:unless>
-        <joint name="${prefix}THJ4" value="1.00" />
-        <joint name="${prefix}THJ5" value="-0.10" />
+        <joint name="${prefix}THJ4" value="1.22" />
+        <joint name="${prefix}THJ5" value="0.06" />
       </xacro:if>
       <xacro:if value="${tip_sensors == 'bt_2p'}">
