Commit message: adding new store state for pelicase

File: sr_moveit_hand_config/config/shadowhand.srdf.xacro (robot description, xacro)
@@ -213,4 +213,23 @@
     </xacro:if>
   </xacro:macro>
+  <xacro:macro name="thumb_state_store" params="prefix is_lite">
+    <joint name="${prefix}THJ1" value="0.15708" />
+    <joint name="${prefix}THJ2" value="0.541052" />
+    <xacro:unless value="$(arg is_lite)">
+      <joint name="${prefix}THJ3" value="0.122173" />
+    </xacro:unless>
+    <joint name="${prefix}THJ4" value="0.331613" />
+    <joint name="${prefix}THJ5" value="0.331613" />
+  </xacro:macro>
+  <xacro:macro name="finger_state_store" params="prefix joint_prefix lf">
+    <joint name="${prefix}${joint_prefix}J1" value="1.37881" />
+    <joint name="${prefix}${joint_prefix}J2" value="1.37881" />
+    <joint name="${prefix}${joint_prefix}J3" value="1.55334" />
+    <joint name="${prefix}${joint_prefix}J4" value="0" />
+    <xacro:if value="${lf}">
+      <!-- Little finger special case -->
+      <joint name="${prefix}${joint_prefix}J5" value="0" />
+    </xacro:if>
+  </xacro:macro>
   <xacro:macro name="thumb_state_relaxed" params="prefix">
     <joint name="${prefix}THJ1" value="0.0837" />

File: sr_moveit_hand_config/config/shadowhands_prefix.srdf.xacro (robot description, xacro)
@@ -361,4 +361,25 @@
     </xacro:unless>
   </group_state>
+  <group_state name="store" group="$(arg hand_name)">
+    <xacro:if value="$(arg th)">
+        <xacro:thumb_state_store  prefix="$(arg prefix)" is_lite="$(arg is_lite)"/>
+    </xacro:if>
+    <xacro:if value="$(arg ff)">
+        <xacro:finger_state_store  prefix="$(arg prefix)" joint_prefix="FF" lf="0"/>
+    </xacro:if>
+    <xacro:if value="$(arg mf)">
+        <xacro:finger_state_store  prefix="$(arg prefix)" joint_prefix="MF" lf="0"/>
+    </xacro:if>
+    <xacro:if value="$(arg rf)">
+        <xacro:finger_state_store  prefix="$(arg prefix)" joint_prefix="RF" lf="0"/>
+    </xacro:if>
+    <xacro:unless value="$(arg is_lite)">
+      <xacro:if value="$(arg lf)">
+          <xacro:finger_state_store  prefix="$(arg prefix)" joint_prefix="LF" lf="1"/>
+      </xacro:if>
+      <joint name="$(arg prefix)WRJ1" value="0" />
+      <joint name="$(arg prefix)WRJ2" value="0" />
+    </xacro:unless>
+  </group_state>
   <!--END EFFECTOR: Purpose: Represent information about an end effector.-->
   <!-- single finger end-effectors -->

Commit message: adding new stored state called store

File: sr_moveit_hand_config/config/shadowhand.srdf.xacro (robot description, xacro)
@@ -222,14 +222,4 @@
     <joint name="${prefix}THJ5" value="0.331613" />
   </xacro:macro>
-  <xacro:macro name="finger_state_store" params="prefix joint_prefix lf">
-    <joint name="${prefix}${joint_prefix}J1" value="1.37881" />
-    <joint name="${prefix}${joint_prefix}J2" value="1.37881" />
-    <joint name="${prefix}${joint_prefix}J3" value="1.55334" />
-    <joint name="${prefix}${joint_prefix}J4" value="0" />
-    <xacro:if value="${lf}">
-      <!-- Little finger special case -->
-      <joint name="${prefix}${joint_prefix}J5" value="0" />
-    </xacro:if>
-  </xacro:macro>
   <xacro:macro name="thumb_state_relaxed" params="prefix">
     <joint name="${prefix}THJ1" value="0.0837" />

File: sr_moveit_hand_config/config/shadowhands_prefix.srdf.xacro (robot description, xacro)
@@ -363,18 +363,23 @@
   <group_state name="store" group="$(arg hand_name)">
     <xacro:if value="$(arg th)">
+      <xacro:unless value="$(arg is_lite)">
         <xacro:thumb_state_store  prefix="$(arg prefix)" is_lite="$(arg is_lite)"/>
-    </xacro:if>
-    <xacro:if value="$(arg ff)">
-        <xacro:finger_state_store  prefix="$(arg prefix)" joint_prefix="FF" lf="0"/>
-    </xacro:if>
-    <xacro:if value="$(arg mf)">
-        <xacro:finger_state_store  prefix="$(arg prefix)" joint_prefix="MF" lf="0"/>
-    </xacro:if>
-    <xacro:if value="$(arg rf)">
-        <xacro:finger_state_store  prefix="$(arg prefix)" joint_prefix="RF" lf="0"/>
-    </xacro:if>
-    <xacro:unless value="$(arg is_lite)">
-      <xacro:if value="$(arg lf)">
-          <xacro:finger_state_store  prefix="$(arg prefix)" joint_prefix="LF" lf="1"/>
+      </xacro:unless>
+      <xacro:if value="$(arg is_lite)">
+        <xacro:thumb_state_pack  prefix="$(arg prefix)" tip_sensors="$(arg tip_sensors)" hand_version="$(arg hand_version)"/>
+      </xacro:if>
+    </xacro:if>
+    <xacro:if value="$(arg ff)">
+        <xacro:finger_state_pack  prefix="$(arg prefix)" joint_prefix="FF" lf="0" tip_sensors="$(arg tip_sensors)" hand_version="$(arg hand_version)"/>
+    </xacro:if>
+    <xacro:if value="$(arg mf)">
+        <xacro:finger_state_pack  prefix="$(arg prefix)" joint_prefix="MF" lf="0" tip_sensors="$(arg tip_sensors)" hand_version="$(arg hand_version)"/>
+    </xacro:if>
+    <xacro:if value="$(arg rf)">
+        <xacro:finger_state_pack  prefix="$(arg prefix)" joint_prefix="RF" lf="0" tip_sensors="$(arg tip_sensors)" hand_version="$(arg hand_version)"/>
+    </xacro:if>
+    <xacro:unless value="$(arg is_lite)">
+      <xacro:if value="$(arg lf)">
+          <xacro:finger_state_pack  prefix="$(arg prefix)" joint_prefix="LF" lf="1" tip_sensors="$(arg tip_sensors)" hand_version="$(arg hand_version)"/>
       </xacro:if>
       <joint name="$(arg prefix)WRJ1" value="0" />

Commit message: adapting the pack/store for new palm flesh

File: sr_moveit_hand_config/config/shadowhand.srdf.xacro (robot description, xacro)
@@ -121,9 +121,9 @@
     <xacro:if value="${hand_version == 'E4'}">
       <xacro:if value="${tip_sensors == 'pst'}">
-        <joint name="${prefix}${joint_prefix}J1" value="1.5707" />
+        <joint name="${prefix}${joint_prefix}J1" value="1.4" />
         <joint name="${prefix}${joint_prefix}J3" value="1.309" />
       </xacro:if>
       <xacro:if value="${tip_sensors == 'bt_sp'}">
-        <joint name="${prefix}${joint_prefix}J1" value="1.309" />
+        <joint name="${prefix}${joint_prefix}J1" value="1.000" />
         <joint name="${prefix}${joint_prefix}J3" value="1.309" />
       </xacro:if>

Commit message: New store saved state (#836)
* Removing UR static paths (#829)

* removed static paths to scripts

* undid change

* improved comments

* unified

* Returning at the correct line (#831)

* Removing static UR paths (#828)

* removed static paths to scripts

* undid change

* improved comments

* unified

* returning at the correct time

---------

Co-authored-by: Jesús Ferrándiz <62122095+jeferal@users.noreply.github.com>

* adding new store state for pelicase

* adding new stored state called store

* adapting the pack/store for new palm flesh

* rewriting the date

---------

Co-authored-by: Jesús Ferrándiz <62122095+jeferal@users.noreply.github.com>

File: sr_moveit_hand_config/config/shadowhand.srdf.xacro (robot description, xacro)
@@ -121,9 +121,9 @@
     <xacro:if value="${hand_version == 'E4'}">
       <xacro:if value="${tip_sensors == 'pst'}">
-        <joint name="${prefix}${joint_prefix}J1" value="1.5707" />
+        <joint name="${prefix}${joint_prefix}J1" value="1.4" />
         <joint name="${prefix}${joint_prefix}J3" value="1.309" />
       </xacro:if>
       <xacro:if value="${tip_sensors == 'bt_sp'}">
-        <joint name="${prefix}${joint_prefix}J1" value="1.309" />
+        <joint name="${prefix}${joint_prefix}J1" value="1.000" />
         <joint name="${prefix}${joint_prefix}J3" value="1.309" />
       </xacro:if>
@@ -212,4 +212,13 @@
       <joint name="${prefix}${joint_prefix}J5" value="0.3325" />
     </xacro:if>
+  </xacro:macro>
+  <xacro:macro name="thumb_state_store" params="prefix is_lite">
+    <joint name="${prefix}THJ1" value="0.15708" />
+    <joint name="${prefix}THJ2" value="0.541052" />
+    <xacro:unless value="$(arg is_lite)">
+      <joint name="${prefix}THJ3" value="0.122173" />
+    </xacro:unless>
+    <joint name="${prefix}THJ4" value="0.331613" />
+    <joint name="${prefix}THJ5" value="0.331613" />
   </xacro:macro>
   <xacro:macro name="thumb_state_relaxed" params="prefix">

File: sr_moveit_hand_config/config/shadowhands_prefix.srdf.xacro (robot description, xacro)
@@ -361,4 +361,30 @@
     </xacro:unless>
   </group_state>
+  <group_state name="store" group="$(arg hand_name)">
+    <xacro:if value="$(arg th)">
+      <xacro:unless value="$(arg is_lite)">
+        <xacro:thumb_state_store  prefix="$(arg prefix)" is_lite="$(arg is_lite)"/>
+      </xacro:unless>
+      <xacro:if value="$(arg is_lite)">
+        <xacro:thumb_state_pack  prefix="$(arg prefix)" tip_sensors="$(arg tip_sensors)" hand_version="$(arg hand_version)"/>
+      </xacro:if>
+    </xacro:if>
+    <xacro:if value="$(arg ff)">
+        <xacro:finger_state_pack  prefix="$(arg prefix)" joint_prefix="FF" lf="0" tip_sensors="$(arg tip_sensors)" hand_version="$(arg hand_version)"/>
+    </xacro:if>
+    <xacro:if value="$(arg mf)">
+        <xacro:finger_state_pack  prefix="$(arg prefix)" joint_prefix="MF" lf="0" tip_sensors="$(arg tip_sensors)" hand_version="$(arg hand_version)"/>
+    </xacro:if>
+    <xacro:if value="$(arg rf)">
+        <xacro:finger_state_pack  prefix="$(arg prefix)" joint_prefix="RF" lf="0" tip_sensors="$(arg tip_sensors)" hand_version="$(arg hand_version)"/>
+    </xacro:if>
+    <xacro:unless value="$(arg is_lite)">
+      <xacro:if value="$(arg lf)">
+          <xacro:finger_state_pack  prefix="$(arg prefix)" joint_prefix="LF" lf="1" tip_sensors="$(arg tip_sensors)" hand_version="$(arg hand_version)"/>
+      </xacro:if>
+      <joint name="$(arg prefix)WRJ1" value="0" />
+      <joint name="$(arg prefix)WRJ2" value="0" />
+    </xacro:unless>
+  </group_state>
   <!--END EFFECTOR: Purpose: Represent information about an end effector.-->
   <!-- single finger end-effectors -->

Commit message: created more grasps and adding republisher

File: sr_moveit_hand_config/config/shadowhand.srdf.xacro (robot description, xacro)
@@ -99,4 +99,13 @@
     <joint name="${prefix}THJ5" value="0" />
   </xacro:macro>
+  <xacro:macro name="thumb_state_open_ladle" params="prefix">
+    <joint name="${prefix}THJ1" value="0.021128104873725195" />
+    <joint name="${prefix}THJ2" value="-0.1960632500796953" />
+    <xacro:unless value="$(arg is_lite)">
+      <joint name="${prefix}THJ3" value="-0.012912613691254187" />
+    </xacro:unless>
+    <joint name="${prefix}THJ4" value="0.4758017440421255" />
+    <joint name="${prefix}THJ5" value="-0.832660323827618" />
+  </xacro:macro>
   <xacro:macro name="finger_state_pack" params="prefix joint_prefix lf tip_sensors hand_version">
     <xacro:unless value="${hand_version == 'E4'}">

File: sr_moveit_hand_config/config/shadowhands_prefix.srdf.xacro (robot description, xacro)
@@ -170,5 +170,5 @@
   <group_state name="fingers_pack_thumb_open" group="$(arg hand_name)">
     <xacro:if value="$(arg th)">
-        <xacro:thumb_state_open  prefix="$(arg prefix)" />
+        <xacro:thumb_state_open_ladle  prefix="$(arg prefix)" />
     </xacro:if>
     <xacro:if value="$(arg ff)">
@@ -188,4 +188,153 @@
       <joint name="$(arg prefix)WRJ2" value="0" />
     </xacro:unless>
+  </group_state>
+  <group_state name="fingers_open_wok" group="$(arg hand_name)">
+      <joint name="$(arg prefix)FFJ1" value="0.0" />
+      <joint name="$(arg prefix)FFJ2" value="0.0" />
+      <joint name="$(arg prefix)FFJ3" value="0.0" />
+      <joint name="$(arg prefix)FFJ4" value="0.0" />
+      <joint name="$(arg prefix)MFJ1" value="0.0" />
+      <joint name="$(arg prefix)MFJ2" value="0.0" />
+      <joint name="$(arg prefix)MFJ3" value="0.0" />
+      <joint name="$(arg prefix)MFJ4" value="0.0" />
+      <joint name="$(arg prefix)RFJ1" value="0.0" />
+      <joint name="$(arg prefix)RFJ2" value="0.0" />
+      <joint name="$(arg prefix)RFJ3" value="0.0" />
+      <joint name="$(arg prefix)RFJ4" value="0.0" />
+      <joint name="$(arg prefix)LFJ1" value="0.0" />
+      <joint name="$(arg prefix)LFJ2" value="0.0" />
+      <joint name="$(arg prefix)LFJ3" value="0.0" />
+      <joint name="$(arg prefix)LFJ4" value="0.0" />
+      <joint name="$(arg prefix)LFJ5" value="0.0" />
+      <joint name="$(arg prefix)THJ1" value="0.0" />
+      <joint name="$(arg prefix)THJ2" value="0.0" />
+      <joint name="$(arg prefix)THJ3" value="0.0" />
+      <joint name="$(arg prefix)THJ4" value="1.22" />
+      <joint name="$(arg prefix)THJ5" value="-1.0" />
+      <joint name="$(arg prefix)WRJ1" value="0.0" />
+      <joint name="$(arg prefix)WRJ2" value="0.0" />
+  </group_state>
+  <group_state name="fingers_pack_wok" group="$(arg hand_name)">
+      <joint name="$(arg prefix)FFJ1" value="1.57" />
+      <joint name="$(arg prefix)FFJ2" value="1.57" />
+      <joint name="$(arg prefix)FFJ3" value="1.57" />
+      <joint name="$(arg prefix)FFJ4" value="0.0" />
+      <joint name="$(arg prefix)MFJ1" value="1.57" />
+      <joint name="$(arg prefix)MFJ2" value="1.57" />
+      <joint name="$(arg prefix)MFJ3" value="1.57" />
+      <joint name="$(arg prefix)MFJ4" value="0.0" />
+      <joint name="$(arg prefix)RFJ1" value="1.57" />
+      <joint name="$(arg prefix)RFJ2" value="1.57" />
+      <joint name="$(arg prefix)RFJ3" value="1.57" />
+      <joint name="$(arg prefix)RFJ4" value="0.0" />
+      <joint name="$(arg prefix)LFJ1" value="1.57" />
+      <joint name="$(arg prefix)LFJ2" value="1.57" />
+      <joint name="$(arg prefix)LFJ3" value="1.57" />
+      <joint name="$(arg prefix)LFJ4" value="0.0" />
+      <joint name="$(arg prefix)LFJ5" value="0.0" />
+      <joint name="$(arg prefix)THJ1" value="0.67" />
+      <joint name="$(arg prefix)THJ2" value="0.55" />
+      <joint name="$(arg prefix)THJ3" value="0.0" />
+      <joint name="$(arg prefix)THJ4" value="1.1692534528173206" />
+      <joint name="$(arg prefix)THJ5" value="0.0" />
+      <joint name="$(arg prefix)WRJ1" value="0.0" />
+      <joint name="$(arg prefix)WRJ2" value="0.0" />
+  </group_state>
+    <!-- GRASPS FOR THE LADLE -->
+  <group_state name="grasp_ladle_approach" group="$(arg prefix)fingers">
+    <joint name="$(arg prefix)FFJ1" value="0" />
+    <joint name="$(arg prefix)FFJ2" value="0" />
+    <joint name="$(arg prefix)FFJ3" value="0" />
+    <joint name="$(arg prefix)FFJ4" value="0" />
+    <joint name="$(arg prefix)MFJ1" value="0" />
+    <joint name="$(arg prefix)MFJ2" value="0" />
+    <joint name="$(arg prefix)MFJ3" value="0" />
+    <joint name="$(arg prefix)MFJ4" value="0" />
+    <joint name="$(arg prefix)RFJ1" value="0" />
+    <joint name="$(arg prefix)RFJ2" value="0" />
+    <joint name="$(arg prefix)RFJ3" value="0" />
+    <joint name="$(arg prefix)RFJ4" value="0" />
+    <joint name="$(arg prefix)LFJ1" value="0" />
+    <joint name="$(arg prefix)LFJ2" value="0" />
+    <joint name="$(arg prefix)LFJ3" value="0" />
+    <joint name="$(arg prefix)LFJ4" value="0" />
+    <joint name="$(arg prefix)LFJ5" value="0" />
+    <joint name="$(arg prefix)THJ1" value="0.0" />
+    <joint name="$(arg prefix)THJ2" value="-0.17" />
+    <joint name="$(arg prefix)THJ3" value="0.0" />
+    <joint name="$(arg prefix)THJ4" value="1.03" />
+    <joint name="$(arg prefix)THJ5" value="-1.05" />
+  </group_state>
+  <group_state name="grasp_ladle_intermediate" group="$(arg prefix)fingers">
+    <joint name="$(arg prefix)FFJ1" value="0" />
+    <joint name="$(arg prefix)FFJ2" value="0" />
+    <joint name="$(arg prefix)FFJ3" value="0.95" />
+    <joint name="$(arg prefix)FFJ4" value="0" />
+    <joint name="$(arg prefix)MFJ1" value="0" />
+    <joint name="$(arg prefix)MFJ2" value="0" />
+    <joint name="$(arg prefix)MFJ3" value="1.3" />
+    <joint name="$(arg prefix)MFJ4" value="0" />
+    <joint name="$(arg prefix)RFJ1" value="0" />
+    <joint name="$(arg prefix)RFJ2" value="0" />
+    <joint name="$(arg prefix)RFJ3" value="1.57" />
+    <joint name="$(arg prefix)RFJ4" value="0" />
+    <joint name="$(arg prefix)LFJ1" value="0" />
+    <joint name="$(arg prefix)LFJ2" value="0" />
+    <joint name="$(arg prefix)LFJ3" value="1.57" />
+    <joint name="$(arg prefix)LFJ4" value="0" />
+    <joint name="$(arg prefix)LFJ5" value="0" />
+    <joint name="$(arg prefix)THJ1" value="0.0" />
+    <joint name="$(arg prefix)THJ2" value="0.0349066" />
+    <joint name="$(arg prefix)THJ3" value="0.0" />
+    <joint name="$(arg prefix)THJ4" value="0.0872665" />
+    <joint name="$(arg prefix)THJ5" value="-1.05" />
+  </group_state>
+  <group_state name="grasp_ladle_pack" group="$(arg prefix)fingers">
+    <joint name="$(arg prefix)FFJ1" value="1.57" />
+    <joint name="$(arg prefix)FFJ2" value="1.57" />
+    <joint name="$(arg prefix)FFJ3" value="0.95" />
+    <joint name="$(arg prefix)FFJ4" value="0" />
+    <joint name="$(arg prefix)MFJ1" value="1.57" />
+    <joint name="$(arg prefix)MFJ2" value="1.57" />
+    <joint name="$(arg prefix)MFJ3" value="1.3" />
+    <joint name="$(arg prefix)MFJ4" value="0" />
+    <joint name="$(arg prefix)RFJ1" value="1.57" />
+    <joint name="$(arg prefix)RFJ2" value="1.57" />
+    <joint name="$(arg prefix)RFJ3" value="1.57" />
+    <joint name="$(arg prefix)RFJ4" value="0" />
+    <joint name="$(arg prefix)LFJ1" value="1.57" />
+    <joint name="$(arg prefix)LFJ2" value="1.57" />
+    <joint name="$(arg prefix)LFJ3" value="1.57" />
+    <joint name="$(arg prefix)LFJ4" value="0.174533" />
+    <joint name="$(arg prefix)LFJ5" value="-1.0472" />
+    <joint name="$(arg prefix)THJ1" value="0.0174533" />
+    <joint name="$(arg prefix)THJ2" value="0.0349066" />
+    <joint name="$(arg prefix)THJ3" value="0.0" />
+    <joint name="$(arg prefix)THJ4" value="0.174533" />
+    <joint name="$(arg prefix)THJ5" value="0.261799" />
+  </group_state>
+  <group_state name="soy_sauce_pack" group="$(arg prefix)fingers">
+    <joint name="$(arg prefix)FFJ1" value="0.785398" />
+    <joint name="$(arg prefix)FFJ2" value="0.785398" />
+    <joint name="$(arg prefix)FFJ3" value="1.57" />
+    <joint name="$(arg prefix)FFJ4" value="0" />
+    <joint name="$(arg prefix)MFJ1" value="0.785398" />
+    <joint name="$(arg prefix)MFJ2" value="0.785398" />
+    <joint name="$(arg prefix)MFJ3" value="1.57" />
+    <joint name="$(arg prefix)MFJ4" value="0" />
+    <joint name="$(arg prefix)RFJ1" value="0.785398" />
+    <joint name="$(arg prefix)RFJ2" value="0.785398" />
+    <joint name="$(arg prefix)RFJ3" value="1.57" />
+    <joint name="$(arg prefix)RFJ4" value="0" />
+    <joint name="$(arg prefix)LFJ1" value="0.785398" />
+    <joint name="$(arg prefix)LFJ2" value="0.785398" />
+    <joint name="$(arg prefix)LFJ3" value="1.57" />
+    <joint name="$(arg prefix)LFJ4" value="0.0" />
+    <joint name="$(arg prefix)LFJ5" value="0.0" />
+    <joint name="$(arg prefix)THJ1" value="0.0" />
+    <joint name="$(arg prefix)THJ2" value="-0.17" />
+    <joint name="$(arg prefix)THJ3" value="0.0" />
+    <joint name="$(arg prefix)THJ4" value="1.03" />
+    <joint name="$(arg prefix)THJ5" value="-1.05" />
   </group_state>
   <!-- single fingers state -->
@@ -247,5 +396,5 @@
   <group_state name="fingers_open" group="$(arg prefix)fingers">
     <xacro:if value="$(arg th)">
-        <xacro:thumb_state_open  prefix="$(arg prefix)" />
+        <xacro:thumb_state_open_ladle  prefix="$(arg prefix)" />
     </xacro:if>
     <xacro:if value="$(arg ff)">
@@ -285,5 +434,5 @@
   <group_state name="fingers_pack_thumb_open" group="$(arg prefix)fingers">
     <xacro:if value="$(arg th)">
-        <xacro:thumb_state_open  prefix="$(arg prefix)" />
+        <xacro:thumb_state_open_ladle  prefix="$(arg prefix)" />
     </xacro:if>
     <xacro:if value="$(arg ff)">
