Commit message: Fixed printing

File: sr_moveit_hand_config/config/shadowhands_prefix.srdf.xacro (robot description, xacro)
@@ -8,9 +8,4 @@
   <xacro:arg name="lf" default="1"/>
   <xacro:arg name="th" default="1"/>
-  <xacro:arg name="ff_bio" default="0"/>
-  <xacro:arg name="mf_bio" default="0"/>
-  <xacro:arg name="rf_bio" default="0"/>
-  <xacro:arg name="lf_bio" default="0"/>
-  <xacro:arg name="th_bio" default="0"/>
   <xacro:arg name="is_lite" default="0"/>
   <xacro:arg name="robot_name" default="shadowhand_motor"/>
@@ -18,55 +13,26 @@
   <group name="$(arg hand_name)">
     <xacro:if value="$(arg th)">
-      <xacro:if value="$(arg th_bio)">
-        <xacro:property name="distal" value="biotac"/>
-      </xacro:if>
-      <xacro:unless value="$(arg th_bio)">
-        <xacro:property name="distal" value="distal"/>
-      </xacro:unless>
+      <xacro:property name="distal" value="distal"/>
       <xacro:thumbjoints prefix="$(arg prefix)"/>
     </xacro:if>
     <xacro:if value="$(arg ff)">
-      <xacro:if value="$(arg ff_bio)">
-        <xacro:property name="" value="biotac"/>
-        <xacro:property name="middle" value="adapter"/>
-      </xacro:if>
-      <xacro:unless value="$(arg ff_bio)">
+      <xacro:property name="distal" value="distal"/>
+      <xacro:property name="middle" value="middle"/>
+      <xacro:fingerjoints prefix="$(arg prefix)" joint_prefix="FF" lf="0"/>
+    </xacro:if>
+    <xacro:if value="$(arg mf)">
+      <xacro:property name="distal" value="distal"/>
+      <xacro:property name="middle" value="middle"/>
+      <xacro:fingerjoints prefix="$(arg prefix)" joint_prefix="MF" lf="0"/>
+    </xacro:if>
+    <xacro:if value="$(arg rf)">
+      <xacro:property name="distal" value="distal"/>
+      <xacro:property name="middle" value="middle"/>
+      <xacro:fingerjoints prefix="$(arg prefix)" joint_prefix="RF" lf="0"/>
+    </xacro:if>
+    <xacro:unless value="$(arg is_lite)">
+      <xacro:if value="$(arg lf)">
         <xacro:property name="distal" value="distal"/>
         <xacro:property name="middle" value="middle"/>
-      </xacro:unless>
-      <xacro:fingerjoints prefix="$(arg prefix)" joint_prefix="FF" lf="0"/>
-    </xacro:if>
-    <xacro:if value="$(arg mf)">
-      <xacro:if value="$(arg mf_bio)">
-        <xacro:property name="distal" value="biotac"/>
-        <xacro:property name="middle" value="adapter"/>
-      </xacro:if>
-      <xacro:unless value="$(arg mf_bio)">
-        <xacro:property name="distal" value="distal"/>
-        <xacro:property name="middle" value="middle"/>
-      </xacro:unless>
-      <xacro:fingerjoints prefix="$(arg prefix)" joint_prefix="MF" lf="0"/>
-    </xacro:if>
-    <xacro:if value="$(arg rf)">
-      <xacro:if value="$(arg rf_bio)">
-        <xacro:property name="distal" value="biotac"/>
-        <xacro:property name="middle" value="adapter"/>
-      </xacro:if>
-      <xacro:unless value="$(arg rf_bio)">
-        <xacro:property name="distal" value="distal"/>
-        <xacro:property name="middle" value="middle"/>
-      </xacro:unless>
-      <xacro:fingerjoints prefix="$(arg prefix)" joint_prefix="RF" lf="0"/>
-    </xacro:if>
-    <xacro:unless value="$(arg is_lite)">
-      <xacro:if value="$(arg lf)">
-        <xacro:if value="$(arg lf_bio)">
-          <xacro:property name="distal" value="biotac"/>
-          <xacro:property name="middle" value="adapter"/>
-        </xacro:if>
-        <xacro:unless value="$(arg lf_bio)">
-          <xacro:property name="distal" value="distal"/>
-          <xacro:property name="middle" value="middle"/>
-        </xacro:unless>
         <xacro:fingerjoints prefix="$(arg prefix)" joint_prefix="LF" lf="1"/>
       </xacro:if>
@@ -290,5 +256,5 @@
   </xacro:if>
   <xacro:unless value="$(arg is_lite)">
-    <end_effector name="$(arg hand_name)_ee" parent_link="$(arg prefix)wrist" group="$(arg hand_name)" />
+    <end_effector name="$(arg hand_name)_ee" parent_link="$(arg prefix)palm" group="$(arg hand_name)"/>
   </xacro:unless>
   <xacro:virtual_joints prefix="$(arg prefix)" />
@@ -297,236 +263,106 @@
   <!-- single fingers collision -->
   <xacro:if value="$(arg ff)">
-    <xacro:if value="$(arg ff_bio)">
-      <xacro:property name="distal" value="biotac"/>
-      <xacro:property name="middle" value="adapter"/>
-    </xacro:if>
-    <xacro:unless value="$(arg ff_bio)">
-      <xacro:property name="distal" value="distal"/>
-      <xacro:property name="middle" value="middle"/>
-    </xacro:unless>
+    <xacro:property name="distal" value="distal"/>
+    <xacro:property name="middle" value="middle"/>
     <xacro:finger_collisions prefix="$(arg prefix)" link_prefix="ff" lf="0" />
   </xacro:if>
   <xacro:if value="$(arg mf)">
-    <xacro:if value="$(arg mf_bio)">
-      <xacro:property name="distal" value="biotac"/>
-      <xacro:property name="middle" value="adapter"/>
-    </xacro:if>
-    <xacro:unless value="$(arg mf_bio)">
-      <xacro:property name="distal" value="distal"/>
-      <xacro:property name="middle" value="middle"/>
-    </xacro:unless>
+    <xacro:property name="distal" value="distal"/>
+    <xacro:property name="middle" value="middle"/>
     <xacro:finger_collisions prefix="$(arg prefix)" link_prefix="mf" lf="0" />
   </xacro:if>
   <xacro:if value="$(arg rf)">
-    <xacro:if value="$(arg rf_bio)">
-      <xacro:property name="distal" value="biotac"/>
-      <xacro:property name="middle" value="adapter"/>
-    </xacro:if>
-    <xacro:unless value="$(arg rf_bio)">
-      <xacro:property name="distal" value="distal"/>
-      <xacro:property name="middle" value="middle"/>
-    </xacro:unless>
+    <xacro:property name="distal" value="distal"/>
+    <xacro:property name="middle" value="middle"/>
     <xacro:finger_collisions prefix="$(arg prefix)" link_prefix="rf" lf="0" />
   </xacro:if>
   <xacro:unless value="$(arg is_lite)">
     <xacro:if value="$(arg lf)">
-      <xacro:if value="$(arg lf_bio)">
-        <xacro:property name="distal" value="biotac"/>
-        <xacro:property name="middle" value="adapter"/>
-      </xacro:if>
-      <xacro:unless value="$(arg lf_bio)">
+      <xacro:property name="distal" value="distal"/>
+      <xacro:property name="middle" value="middle"/>
+      <xacro:finger_collisions prefix="$(arg prefix)" link_prefix="lf" lf="1" />
+    </xacro:if>
+  </xacro:unless>
+  <xacro:if value="$(arg th)">
+    <xacro:property name="distal" value="distal"/>
+    <xacro:thumb_collisions prefix="$(arg prefix)" />
+  </xacro:if>
+  <!-- pairs with thumb for collision-->
+  <xacro:if value="$(arg th)">
+    <xacro:property name="thdistal" value="thdistal"/>
+    <xacro:if value="$(arg ff)">
+      <xacro:property name="distal" value="distal"/>
+      <xacro:property name="middle" value="middle"/>
+      <xacro:finger_thumb_collisions  prefix="$(arg prefix)" link_prefix="ff" far="0" lf="0" />
+    </xacro:if>
+    <xacro:if value="$(arg mf)">
+      <xacro:property name="distal" value="distal"/>
+      <xacro:property name="middle" value="middle"/>
+      <xacro:finger_thumb_collisions  prefix="$(arg prefix)" link_prefix="mf" far="1" lf="0" />
+    </xacro:if>
+    <xacro:if value="$(arg rf)">
+      <xacro:property name="distal" value="distal"/>
+      <xacro:property name="middle" value="middle"/>
+      <xacro:finger_thumb_collisions  prefix="$(arg prefix)" link_prefix="rf" far="1" lf="0" />
+    </xacro:if>
+    <xacro:unless value="$(arg is_lite)">
+      <xacro:if value="$(arg lf)">
+       <xacro:property name="distal" value="distal"/>
+       <xacro:property name="middle" value="middle"/>
+       <xacro:finger_thumb_collisions  prefix="$(arg prefix)" link_prefix="lf" far="1" lf="1" />
+      </xacro:if>
+    </xacro:unless>
+  </xacro:if>
+  <!-- pairs with other fingers for collision-->
+  <xacro:if value="$(arg ff)">
+    <xacro:if value="$(arg mf)">
+      <xacro:property name="distal" value="distal"/>
+      <xacro:property name="middle" value="middle"/>
+      <xacro:property name="distal2" value="distal"/>
+      <xacro:property name="middle2" value="middle"/>
+      <xacro:finger_closefinger_collisions prefix="$(arg prefix)" link_prefix="ff" link_prefix2="mf"  lf="0"/>
+    </xacro:if>
+    <xacro:if value="$(arg rf)">
+      <xacro:property name="distal" value="distal"/>
+      <xacro:property name="middle" value="middle"/>
+      <xacro:property name="distal2" value="distal"/>
+      <xacro:property name="middle2" value="middle"/>
+      <xacro:finger_farfinger_collisions prefix="$(arg prefix)" link_prefix="ff" link_prefix2="rf"  lf="0" />
+    </xacro:if>
+    <xacro:unless value="$(arg is_lite)">
+      <xacro:if value="$(arg lf)">
         <xacro:property name="distal" value="distal"/>
         <xacro:property name="middle" value="middle"/>
-      </xacro:unless>
-       <xacro:finger_collisions prefix="$(arg prefix)" link_prefix="lf" lf="1" />
-    </xacro:if>
-  </xacro:unless>
-  <xacro:if value="$(arg th)">
-    <xacro:if value="$(arg th_bio)">
-      <xacro:property name="distal" value="biotac"/>
-    </xacro:if>
-    <xacro:unless value="$(arg th_bio)">
-      <xacro:property name="distal" value="distal"/>
-    </xacro:unless>
-    <xacro:thumb_collisions prefix="$(arg prefix)" />
-  </xacro:if>
-  <!-- pairs with thumb for collision-->
-  <xacro:if value="$(arg th)">
-    <xacro:if value="$(arg th_bio)">
-      <xacro:property name="thdistal" value="thbiotac"/>
-    </xacro:if>
-    <xacro:unless value="$(arg th_bio)">
-      <xacro:property name="thdistal" value="thdistal"/>
-    </xacro:unless>
-    <xacro:if value="$(arg ff)">
-      <xacro:if value="$(arg ff_bio)">
-        <xacro:property name="distal" value="biotac"/>
-        <xacro:property name="middle" value="adapter"/>
-      </xacro:if>
-      <xacro:unless value="$(arg ff_bio)">
+        <xacro:property name="distal2" value="distal"/>
+        <xacro:property name="middle2" value="middle"/>
+        <xacro:first_little_collisions prefix="$(arg prefix)" />
+      </xacro:if>
+    </xacro:unless>
+  </xacro:if>
+  <xacro:if value="$(arg mf)">
+    <xacro:if value="$(arg rf)">
+      <xacro:property name="distal" value="distal"/>
+      <xacro:property name="middle" value="middle"/>
+      <xacro:property name="distal2" value="distal"/>
+      <xacro:property name="middle2" value="middle"/>
+      <xacro:finger_closefinger_collisions prefix="$(arg prefix)" link_prefix="mf" link_prefix2="rf"  lf="0" />
+    </xacro:if>
+    <xacro:unless value="$(arg is_lite)">
+      <xacro:if value="$(arg lf)">
         <xacro:property name="distal" value="distal"/>
         <xacro:property name="middle" value="middle"/>
-      </xacro:unless>
-      <xacro:finger_thumb_collisions  prefix="$(arg prefix)" link_prefix="ff" far="0" lf="0" />
-    </xacro:if>
-    <xacro:if value="$(arg mf)">
-      <xacro:if value="$(arg mf_bio)">
-        <xacro:property name="distal" value="biotac"/>
-        <xacro:property name="middle" value="adapter"/>
-      </xacro:if>
-      <xacro:unless value="$(arg mf_bio)">
+        <xacro:property name="distal2" value="distal"/>
+        <xacro:property name="middle2" value="middle"/>
+        <xacro:finger_farfinger_collisions prefix="$(arg prefix)" link_prefix="mf" link_prefix2="lf"  lf="1" />
+      </xacro:if>
+    </xacro:unless>
+  </xacro:if>
+  <xacro:if value="$(arg rf)">
+    <xacro:unless value="$(arg is_lite)">
+      <xacro:if value="$(arg lf)">
         <xacro:property name="distal" value="distal"/>
         <xacro:property name="middle" value="middle"/>
-      </xacro:unless>
-      <xacro:finger_thumb_collisions  prefix="$(arg prefix)" link_prefix="mf" far="1" lf="0" />
-    </xacro:if>
-    <xacro:if value="$(arg rf)">
-      <xacro:if value="$(arg rf_bio)">
-        <xacro:property name="distal" value="biotac"/>
-        <xacro:property name="middle" value="adapter"/>
-      </xacro:if>
-      <xacro:unless value="$(arg rf_bio)">
-        <xacro:property name="distal" value="distal"/>
-        <xacro:property name="middle" value="middle"/>
-      </xacro:unless>
-      <xacro:finger_thumb_collisions  prefix="$(arg prefix)" link_prefix="rf" far="1" lf="0" />
-    </xacro:if>
-    <xacro:unless value="$(arg is_lite)">
-      <xacro:if value="$(arg lf)">
-          <xacro:if value="$(arg lf_bio)">
-            <xacro:property name="distal" value="biotac"/>
-            <xacro:property name="middle" value="adapter"/>
-          </xacro:if>
-          <xacro:unless value="$(arg lf_bio)">
-            <xacro:property name="distal" value="distal"/>
-            <xacro:property name="middle" value="middle"/>
-          </xacro:unless>
-          <xacro:finger_thumb_collisions  prefix="$(arg prefix)" link_prefix="lf" far="1" lf="1" />
-      </xacro:if>
-    </xacro:unless>
-  </xacro:if>
-  <!-- pairs with other fingers for collision-->
-  <xacro:if value="$(arg ff)">
-    <xacro:if value="$(arg mf)">
-      <xacro:if value="$(arg ff_bio)">
-        <xacro:property name="distal" value="biotac"/>
-        <xacro:property name="middle" value="adapter"/>
-      </xacro:if>
-      <xacro:unless value="$(arg ff_bio)">
-        <xacro:property name="distal" value="distal"/>
-        <xacro:property name="middle" value="middle"/>
-      </xacro:unless>
-      <xacro:if value="$(arg mf_bio)">
-        <xacro:property name="distal2" value="biotac"/>
-        <xacro:property name="middle2" value="adapter"/>
-        </xacro:if>
-      <xacro:unless value="$(arg mf_bio)">
         <xacro:property name="distal2" value="distal"/>
         <xacro:property name="middle2" value="middle"/>
-      </xacro:unless>
-      <xacro:finger_closefinger_collisions prefix="$(arg prefix)" link_prefix="ff" link_prefix2="mf"  lf="0"/>
-    </xacro:if>
-    <xacro:if value="$(arg rf)">
-      <xacro:if value="$(arg ff_bio)">
-        <xacro:property name="distal" value="biotac"/>
-        <xacro:property name="middle" value="adapter"/>
-      </xacro:if>
-      <xacro:unless value="$(arg ff_bio)">
-        <xacro:property name="distal" value="distal"/>
-        <xacro:property name="middle" value="middle"/>
-      </xacro:unless>
-      <xacro:if value="$(arg rf_bio)">
-        <xacro:property name="distal2" value="biotac"/>
-        <xacro:property name="middle2" value="adapter"/>
-        </xacro:if>
-      <xacro:unless value="$(arg rf_bio)">
-        <xacro:property name="distal2" value="distal"/>
-        <xacro:property name="middle2" value="middle"/>
-      </xacro:unless>
-      <xacro:finger_farfinger_collisions prefix="$(arg prefix)" link_prefix="ff" link_prefix2="rf"  lf="0" />
-    </xacro:if>
-    <xacro:unless value="$(arg is_lite)">
-      <xacro:if value="$(arg lf)">
-        <xacro:if value="$(arg ff_bio)">
-          <xacro:property name="distal" value="biotac"/>
-          <xacro:property name="middle" value="adapter"/>
-        </xacro:if>
-        <xacro:unless value="$(arg ff_bio)">
-          <xacro:property name="distal" value="distal"/>
-          <xacro:property name="middle" value="middle"/>
-        </xacro:unless>
-        <xacro:if value="$(arg lf_bio)">
-          <xacro:property name="distal2" value="biotac"/>
-          <xacro:property name="middle2" value="adapter"/>
-          </xacro:if>
-        <xacro:unless value="$(arg lf_bio)">
-          <xacro:property name="distal2" value="distal"/>
-          <xacro:property name="middle2" value="middle"/>
-        </xacro:unless>
-        <xacro:first_little_collisions prefix="$(arg prefix)" />
-      </xacro:if>
-    </xacro:unless>
-  </xacro:if>
-  <xacro:if value="$(arg mf)">
-    <xacro:if value="$(arg rf)">
-      <xacro:if value="$(arg mf_bio)">
-        <xacro:property name="distal" value="biotac"/>
-        <xacro:property name="middle" value="adapter"/>
-      </xacro:if>
-      <xacro:unless value="$(arg mf_bio)">
-        <xacro:property name="distal" value="distal"/>
-        <xacro:property name="middle" value="middle"/>
-      </xacro:unless>
-      <xacro:if value="$(arg rf_bio)">
-        <xacro:property name="distal2" value="biotac"/>
-        <xacro:property name="middle2" value="adapter"/>
-        </xacro:if>
-      <xacro:unless value="$(arg rf_bio)">
-        <xacro:property name="distal2" value="distal"/>
-        <xacro:property name="middle2" value="middle"/>
-      </xacro:unless>
-      <xacro:finger_closefinger_collisions prefix="$(arg prefix)" link_prefix="mf" link_prefix2="rf"  lf="0" />
-    </xacro:if>
-    <xacro:unless value="$(arg is_lite)">
-      <xacro:if value="$(arg lf)">
-        <xacro:if value="$(arg mf_bio)">
-          <xacro:property name="distal" value="biotac"/>
-          <xacro:property name="middle" value="adapter"/>
-        </xacro:if>
-        <xacro:unless value="$(arg mf_bio)">
-          <xacro:property name="distal" value="distal"/>
-          <xacro:property name="middle" value="middle"/>
-        </xacro:unless>
-        <xacro:if value="$(arg lf_bio)">
-          <xacro:property name="distal2" value="biotac"/>
-          <xacro:property name="middle2" value="adapter"/>
-          </xacro:if>
-        <xacro:unless value="$(arg lf_bio)">
-          <xacro:property name="distal2" value="distal"/>
-          <xacro:property name="middle2" value="middle"/>
-        </xacro:unless>
-        <xacro:finger_farfinger_collisions prefix="$(arg prefix)" link_prefix="mf" link_prefix2="lf"  lf="1" />
-      </xacro:if>
-    </xacro:unless>
-  </xacro:if>
-  <xacro:if value="$(arg rf)">
-    <xacro:unless value="$(arg is_lite)">
-      <xacro:if value="$(arg lf)">
-        <xacro:if value="$(arg rf_bio)">
-          <xacro:property name="distal" value="biotac"/>
-          <xacro:property name="middle" value="adapter"/>
-        </xacro:if>
-        <xacro:unless value="$(arg rf_bio)">
-          <xacro:property name="distal" value="distal"/>
-          <xacro:property name="middle" value="middle"/>
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
Commit message: Removed groups with thumb and fingers and the one of the fingertips

File: sr_moveit_hand_config/config/shadowhands_prefix.srdf.xacro (robot description, xacro)
@@ -67,22 +67,4 @@
     </group>
   </xacro:if>
-  <!-- all fingerstips -->
-  <group name="$(arg prefix)fingertips">
-    <xacro:if value="$(arg ff)">
-      <link name="$(arg prefix)fftip" />
-    </xacro:if>
-    <xacro:if value="$(arg mf)">
-      <link name="$(arg prefix)mftip" />
-    </xacro:if>
-    <xacro:if value="$(arg rf)">
-      <link name="$(arg prefix)rftip" />
-    </xacro:if>
-    <xacro:if value="$(arg lf)">
-      <link name="$(arg prefix)lftip" />
-    </xacro:if>
-    <xacro:if value="$(arg th)">
-      <link name="$(arg prefix)thtip" />
-    </xacro:if>
-  </group>
   <!-- all fingers group -->
   <group name="$(arg prefix)fingers">
@@ -110,33 +92,4 @@
     </xacro:unless>
   </group>
-   <!-- pairs with thumb for groups -->
-  <xacro:if value="$(arg th)">
-    <xacro:if value="$(arg ff)">
-      <group name="$(arg prefix)first_finger_thumb">
-        <xacro:thumbjoints prefix="$(arg prefix)" />
-        <xacro:fingerjoints prefix="$(arg prefix)" joint_prefix="FF" lf="0"/>
-      </group>
-    </xacro:if>
-    <xacro:if value="$(arg mf)">
-      <group name="$(arg prefix)middle_finger_thumb">
-        <xacro:thumbjoints prefix="$(arg prefix)"/>
-        <xacro:fingerjoints prefix="$(arg prefix)" joint_prefix="MF" lf="0"/>
-      </group>
-    </xacro:if>
-    <xacro:if value="$(arg rf)">
-      <group name="$(arg prefix)ring_finger_thumb">
-        <xacro:thumbjoints prefix="$(arg prefix)"/>
-        <xacro:fingerjoints prefix="$(arg prefix)" joint_prefix="RF" lf="0"/>
-      </group>
-    </xacro:if>
-    <xacro:unless value="$(arg is_lite)">
-      <xacro:if value="$(arg lf)">
-        <group name="$(arg prefix)little_finger_thumb">
-          <xacro:thumbjoints prefix="$(arg prefix)"/>
-          <xacro:fingerjoints prefix="$(arg prefix)" joint_prefix="LF" lf="1"/>
-        </group>
-      </xacro:if>
-    </xacro:unless>
-  </xacro:if>
   <!--GROUP STATES: Purpose: Define a named state for a particular group, in terms of joint values. This is useful to define states like 'folded arms'-->
   <!-- hand state -->
@@ -210,21 +163,4 @@
     </xacro:unless>
   </group_state>
-  <!-- pairs with thumb for state -->
-  <xacro:if value="$(arg th)">
-    <xacro:if value="$(arg ff)">
-      <xacro:finger_thumb_state_open  prefix="$(arg prefix)" finger_name="first_finger" joint_prefix="FF" lf="0"  is_lite="$(arg is_lite)" />
-    </xacro:if>
-    <xacro:if value="$(arg mf)">
-      <xacro:finger_thumb_state_open  prefix="$(arg prefix)" finger_name="middle_finger" joint_prefix="MF" lf="0"  is_lite="$(arg is_lite)" />
-    </xacro:if>
-    <xacro:if value="$(arg rf)">
-      <xacro:finger_thumb_state_open  prefix="$(arg prefix)" finger_name="ring_finger" joint_prefix="RF" lf="0"  is_lite="$(arg is_lite)" />
-    </xacro:if>
-    <xacro:unless value="$(arg is_lite)">
-      <xacro:if value="$(arg lf)">
-          <xacro:finger_thumb_state_open  prefix="$(arg prefix)" finger_name="little_finger" joint_prefix="LF" lf="1"  is_lite="$(arg is_lite)" />
-      </xacro:if>
-    </xacro:unless>
-  </xacro:if>
   <!--END EFFECTOR: Purpose: Represent information about an end effector.-->
   <!-- single finger end-effectors -->

Commit message: Added wrist group and fixed ee

File: sr_moveit_hand_config/config/shadowhands_prefix.srdf.xacro (robot description, xacro)
@@ -34,4 +34,10 @@
     <group name="$(arg prefix)fingers" />
   </group>
+  <xacro:unless value="$(arg is_lite)">
+    <group name="$(arg prefix)wrist">
+ 	  <joint name="$(arg prefix)WRJ2" />
+      <joint name="$(arg prefix)WRJ1" />
+    </group>
+  </xacro:unless>
   <!-- single finger groups -->
   <xacro:if value="$(arg ff)">
@@ -250,5 +256,5 @@
   </xacro:if>
   <xacro:unless value="$(arg is_lite)">
-    <end_effector name="$(arg hand_name)_ee" parent_link="$(arg prefix)palm" group="$(arg hand_name)"/>
+    <end_effector group="$(arg prefix)wrist" name="$(arg prefix)wrist_ee" parent_link="$(arg prefix)palm" parent_group="$(arg hand_name)"/>
   </xacro:unless>
   <xacro:virtual_joints prefix="$(arg prefix)" />
